File: LT1763IDE-1.8.kicad_sch (KiCad schematic)
At the start: 6 parts, among them U3201 LT1763IDE-1.8PBF

Commit message: fields
Parts:
- C3201: gfootprint 1206 -> (none)
- C3202, C3203, C3204: gfootprint 0603 -> (none)
- FB3201: gfootprint 0805 -> (none)
- U3201: MPN LT1763IDE-1.8#PBF -> (none); PACKAGE DFN-12 -> (none); Vendor digikey:LT1763IDE-1.8#PBF-ND -> (none)
Changed lines of the file:
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@@
-			)
-		)
-		(property "gfootprint" "0805"
-			(at 179.07 179.07 0)
-			(effects
-				(font
-					(size 1.27 1.27)
-				)
-				(hide yes)
 			)
 		)
@@
 			)
 		)
-		(property "PACKAGE" "DFN-12"
-			(at 153.67 87.63 0)
-			(effects
-				(font
-					(size 1.27 1.27)
-				)
-				(justify bottom)
-				(hide yes)
-			)
-		)
-		(property "MPN" "LT1763IDE-1.8#PBF"
-			(at 153.67 87.63 0)
-			(effects
-				(font
-					(size 1.27 1.27)
-				)
-				(justify bottom)
-				(hide yes)
-			)
-		)
-		(property "Vendor" "digikey:LT1763IDE-1.8#PBF-ND"
-			(at 153.67 87.63 0)
-			(effects
-				(font
-					(size 1.27 1.27)
-				)
-				(hide yes)
-			)
-		)
 		(pin "6"
 		)
@@
 			)
 		)
-		(property "gfootprint" "1206"
-			(at 223.52 0 0)
-			(effects
-				(font
-					(size 1.27 1.27)
-				)
-				(hide yes)
-			)
-		)
 		(pin "2"
 		)
@@
 			)
 		)
-		(property "gfootprint" "0603"
-			(at 0 165.1 0)
-			(effects
-				(font
-					(size 1.27 1.27)
-				)
-				(hide yes)
-			)
-		)
 		(pin "2"
 		)
@@
 			)
 		)
-		(property "gfootprint" "0603"
-			(at 233.68 0 0)
-			(effects
-				(font
-					(size 1.27 1.27)
-				)
-				(hide yes)
-			)
-		)
 		(pin "2"
 		)
@@
 			(effects
 				(font
-					(size 1.27 1.27)
-				)
-				(hide yes)
-			)
-		)
-		(property "gfootprint" "0603"
-			(at 212.09 212.09 0)
-			(effects
-				(font

Commit message: vendor info
Parts:
- C3201: Vendor (none) -> digikey:490-5528-1-ND
- C3202: Vendor (none) -> digikey:490-3897-1-ND
- C3203: Vendor (none) -> digikey:445-2664-1-ND
- C3204: Vendor (none) -> digikey:445-6853-1-ND
- FB3201: Vendor (none) -> digikey:732-1620-1-ND
- U3201: Vendor (none) -> digikey:LT1763IDE-1.8#PBF-ND
Changed lines of the file:
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@@
+			)
+		)
+		(property "Vendor" "digikey:732-1620-1-ND"
+			(at 179.07 179.07 0)
+			(effects
+				(font
+					(size 1.27 1.27)
+				)
+				(hide yes)
 			)
 		)
@@
 			)
 		)
+		(property "Vendor" "digikey:LT1763IDE-1.8#PBF-ND"
+			(at 0 175.26 0)
+			(effects
+				(font
+					(size 1.27 1.27)
+				)
+				(hide yes)
+			)
+		)
 		(pin "6"
 		)
@@
 			)
 		)
+		(property "Vendor" "digikey:490-5528-1-ND"
+			(at 223.52 0 0)
+			(effects
+				(font
+					(size 1.27 1.27)
+				)
+				(hide yes)
+			)
+		)
 		(pin "2"
 		)
@@
 			)
 		)
+		(property "Vendor" "digikey:445-6853-1-ND"
+			(at 0 165.1 0)
+			(effects
+				(font
+					(size 1.27 1.27)
+				)
+				(hide yes)
+			)
+		)
 		(pin "2"
 		)
@@
 			)
 		)
+		(property "Vendor" "digikey:490-3897-1-ND"
+			(at 233.68 0 0)
+			(effects
+				(font
+					(size 1.27 1.27)
+				)
+				(hide yes)
+			)
+		)
 		(pin "2"
 		)
@@
 			(effects
 				(font
+					(size 1.27 1.27)
+				)
+				(hide yes)
+			)
+		)
+		(property "Vendor" "digikey:445-2664-1-ND"
+			(at 212.09 212.09 0)
+			(effects
+				(font

Commit message: update value
Parts:
- C3201: value C -> 47UF
- C3202: value C -> 1UF
- C3203: value C -> 10000PF
- C3204: value C -> 10UF
- FB3201: value FerriteBead -> 742792040
- U3201: value LT1763IDE-1.8PBF -> LT1763IDE-1.8#PBF
Changed lines of the file:
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@@
 			)
 		)
-		(property "Value" "FerriteBead"
+		(property "Value" "742792040"
 			(at 104.0892 69.85 90)
 			(effects
@@
 			)
 		)
-		(property "Value" "LT1763IDE-1.8PBF"
+		(property "Value" "LT1763IDE-1.8#PBF"
 			(at 153.67 67.31 0)
 			(effects
@@
 			)
 		)
-		(property "Value" "C"
+		(property "Value" "47UF"
 			(at 115.57 83.8199 0)
 			(effects
@@
 			)
 		)
-		(property "Value" "C"
+		(property "Value" "10UF"
 			(at 184.15 83.8199 0)
 			(effects
@@
 			)
 		)
-		(property "Value" "C"
+		(property "Value" "1UF"
 			(at 120.65 92.7099 0)
 			(effects
@@
 			)
 		)
-		(property "Value" "C"
+		(property "Value" "10000PF"
 			(at 129.54 77.47 90)
 			(effects
