File: adl5501.kicad_sch (KiCad schematic)
At the start: 7 parts, among them U1801 ADL5501AKSZ-R7

Commit message: fields
Parts:
- C1801, C1802, C1803, C1804, FB1801, R1801: gfootprint 0603 -> (none)
Changed lines of the file:
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@@
-			)
-		)
-		(property "gfootprint" "0603"
-			(at 383.54 0 0)
-			(effects
-				(font
-					(size 1.27 1.27)
-				)
-				(hide yes)
 			)
 		)
@@
 			)
 		)
-		(property "gfootprint" "0603"
-			(at 355.6 0 0)
-			(effects
-				(font
-					(size 1.27 1.27)
-				)
-				(hide yes)
-			)
-		)
 		(pin "2"
 		)
@@
 			)
 		)
-		(property "gfootprint" "0603"
-			(at 200.66 0 0)
-			(effects
-				(font
-					(size 1.27 1.27)
-				)
-				(hide yes)
-			)
-		)
 		(pin "1"
 		)
@@
 			)
 		)
-		(property "gfootprint" "0603"
-			(at 262.89 262.89 0)
-			(effects
-				(font
-					(size 1.27 1.27)
-				)
-				(hide yes)
-			)
-		)
 		(pin "1"
 		)
@@
 			)
 		)
-		(property "gfootprint" "0603"
-			(at 34.29 -34.29 0)
-			(effects
-				(font
-					(size 1.27 1.27)
-				)
-				(hide yes)
-			)
-		)
 		(pin "2"
 		)
@@
 			(effects
 				(font
-					(size 1.27 1.27)
-				)
-				(hide yes)
-			)
-		)
-		(property "gfootprint" "0603"
-			(at 35.56 -35.56 0)
-			(effects
-				(font

Commit message: vendor info
Parts:
- C1801, C1802, C1803, C1804: Vendor (none) -> digikey:445-2664-1-ND
- FB1801: Vendor (none) -> digikey:490-1011-1-ND
- R1801: Vendor (none) -> digikey:311-221HRCT-ND
- U1801: Vendor (none) -> digikey:ADL5501AKSZ-R7CT-ND
Changed lines of the file:
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@@
+			)
+		)
+		(property "Vendor" "digikey:445-2664-1-ND"
+			(at 383.54 0 0)
+			(effects
+				(font
+					(size 1.27 1.27)
+				)
+				(hide yes)
 			)
 		)
@@
 			)
 		)
+		(property "Vendor" "digikey:445-2664-1-ND"
+			(at 355.6 0 0)
+			(effects
+				(font
+					(size 1.27 1.27)
+				)
+				(hide yes)
+			)
+		)
 		(pin "2"
 		)
@@
 			)
 		)
+		(property "Vendor" "digikey:445-2664-1-ND"
+			(at 200.66 0 0)
+			(effects
+				(font
+					(size 1.27 1.27)
+				)
+				(hide yes)
+			)
+		)
 		(pin "1"
 		)
@@
 			)
 		)
+		(property "Vendor" "digikey:311-221HRCT-ND"
+			(at 262.89 262.89 0)
+			(effects
+				(font
+					(size 1.27 1.27)
+				)
+				(hide yes)
+			)
+		)
 		(pin "1"
 		)
@@
 			)
 		)
+		(property "Vendor" "digikey:490-1011-1-ND"
+			(at 34.29 -34.29 0)
+			(effects
+				(font
+					(size 1.27 1.27)
+				)
+				(hide yes)
+			)
+		)
 		(pin "2"
 		)
@@
 			)
 		)
+		(property "Vendor" "digikey:ADL5501AKSZ-R7CT-ND"
+			(at 0 157.48 0)
+			(effects
+				(font
+					(size 1.27 1.27)
+				)
+				(hide yes)
+			)
+		)
 		(pin "5"
 		)
@@
 			(effects
 				(font
+					(size 1.27 1.27)
+				)
+				(hide yes)
+			)
+		)
+		(property "Vendor" "digikey:445-2664-1-ND"
+			(at 35.56 -35.56 0)
+			(effects
+				(font

Commit message: update value
Parts:
- C1801, C1802, C1803, C1804: value C -> 10000PF
- FB1801: value FerriteBead -> BLM18AG121SN1D
- R1801: value R -> 221
Changed lines of the file:
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@@
 			)
 		)
-		(property "Value" "C"
+		(property "Value" "10000PF"
 			(at 195.58 85.0899 0)
 			(effects
@@
 			)
 		)
-		(property "Value" "C"
+		(property "Value" "10000PF"
 			(at 181.61 85.0899 0)
 			(effects
@@
 			)
 		)
-		(property "Value" "C"
+		(property "Value" "10000PF"
 			(at 104.14 67.3099 0)
 			(effects
@@
 			)
 		)
-		(property "Value" "R"
+		(property "Value" "221"
 			(at 184.15 74.93 90)
 			(effects
@@
 			)
 		)
-		(property "Value" "FerriteBead"
+		(property "Value" "BLM18AG121SN1D"
 			(at 96.5708 57.15 90)
 			(effects
@@
 			)
 		)
-		(property "Value" "C"
+		(property "Value" "10000PF"
 			(at 116.84 76.2 90)
 			(effects
