File: diff_se.kicad_sch (KiCad schematic)
At the start: 7 parts

Commit message: fields
Parts:
- C2501, C2502, C2503, C2504, L2501, R2501: gfootprint 0603 -> (none)
Changed lines of the file:
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@@
-			)
-		)
-		(property "gfootprint" "0603"
-			(at 203.2 0 0)
-			(effects
-				(font
-					(size 1.27 1.27)
-				)
-				(hide yes)
 			)
 		)
@@
 			)
 		)
-		(property "gfootprint" "0603"
-			(at 115.57 293.37 0)
-			(effects
-				(font
-					(size 1.27 1.27)
-				)
-				(hide yes)
-			)
-		)
 		(pin "2"
 		)
@@
 			)
 		)
-		(property "gfootprint" "0603"
-			(at 180.34 0 0)
-			(effects
-				(font
-					(size 1.27 1.27)
-				)
-				(hide yes)
-			)
-		)
 		(pin "2"
 		)
@@
 			)
 		)
-		(property "gfootprint" "0603"
-			(at 120.65 -120.65 0)
-			(effects
-				(font
-					(size 1.27 1.27)
-				)
-				(hide yes)
-			)
-		)
 		(pin "2"
 		)
@@
 			)
 		)
-		(property "gfootprint" "0603"
-			(at 180.34 0 0)
-			(effects
-				(font
-					(size 1.27 1.27)
-				)
-				(hide yes)
-			)
-		)
 		(pin "2"
 		)
@@
 			(effects
 				(font
-					(size 1.27 1.27)
-				)
-				(hide yes)
-			)
-		)
-		(property "gfootprint" "0603"
-			(at 149.86 0 0)
-			(effects
-				(font

Commit message: vendor info
Parts:
- C2501: Vendor (none) -> digikey:1276-1089-1-ND
- C2502: Vendor (none) -> digikey:490-1437-1-ND
- C2503, C2504: Vendor (none) -> digikey:490-1451-1-ND
- L2501: Vendor (none) -> digikey:445-1000-1-ND
- R2501: Vendor (none) -> digikey:RR08P200DCT-ND
- XMER2501: Vendor (none) -> digikey:TCM4-19+
Changed lines of the file:
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@@
+			)
+		)
+		(property "Vendor" "digikey:RR08P200DCT-ND"
+			(at 203.2 0 0)
+			(effects
+				(font
+					(size 1.27 1.27)
+				)
+				(hide yes)
 			)
 		)
@@
 			)
 		)
+		(property "Vendor" "digikey:490-1451-1-ND"
+			(at 115.57 293.37 0)
+			(effects
+				(font
+					(size 1.27 1.27)
+				)
+				(hide yes)
+			)
+		)
 		(pin "2"
 		)
@@
 			)
 		)
+		(property "Vendor" "digikey:445-1000-1-ND"
+			(at 180.34 0 0)
+			(effects
+				(font
+					(size 1.27 1.27)
+				)
+				(hide yes)
+			)
+		)
 		(pin "2"
 		)
@@
 			)
 		)
+		(property "Vendor" "digikey:490-1451-1-ND"
+			(at 120.65 -120.65 0)
+			(effects
+				(font
+					(size 1.27 1.27)
+				)
+				(hide yes)
+			)
+		)
 		(pin "2"
 		)
@@
 			)
 		)
+		(property "Vendor" "digikey:490-1437-1-ND"
+			(at 180.34 0 0)
+			(effects
+				(font
+					(size 1.27 1.27)
+				)
+				(hide yes)
+			)
+		)
 		(pin "2"
 		)
@@
 			)
 		)
+		(property "Vendor" "digikey:1276-1089-1-ND"
+			(at 149.86 0 0)
+			(effects
+				(font
+					(size 1.27 1.27)
+				)
+				(hide yes)
+			)
+		)
 		(pin "2"
 		)
@@
 			(effects
 				(font
+					(size 1.27 1.27)
+				)
+				(hide yes)
+			)
+		)
+		(property "Vendor" "digikey:TCM4-19+"
+			(at 0 167.64 0)
+			(effects
+				(font

Commit message: update value
Parts:
- C2501: value C -> 18PF
- C2502: value C -> 270PF
- C2503, C2504: value C -> 1000PF
- L2501: value L -> MLF1608D47NMTA00
- R2501: value R -> 200
Changed lines of the file:
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@@
 			)
 		)
-		(property "Value" "R"
+		(property "Value" "200"
 			(at 104.14 87.6299 0)
 			(effects
@@
 			)
 		)
-		(property "Value" "C"
+		(property "Value" "1000PF"
 			(at 204.47 83.82 90)
 			(effects
@@
 			)
 		)
-		(property "Value" "L"
+		(property "Value" "MLF1608D47NMTA00"
 			(at 91.44 81.2799 0)
 			(effects
@@
 			)
 		)
-		(property "Value" "C"
+		(property "Value" "1000PF"
 			(at 204.47 78.74 90)
 			(effects
@@
 			)
 		)
-		(property "Value" "C"
+		(property "Value" "270PF"
 			(at 93.98 92.7099 0)
 			(effects
@@
 			)
 		)
-		(property "Value" "C"
+		(property "Value" "18PF"
 			(at 78.74 87.6299 0)
 			(effects
