File: LTC6655.kicad_sch (KiCad schematic)
At the start: 5 parts, among them U2801 LTC6655CHLS8-2.5-PBF

Commit message: fields
Parts:
- C2801: gfootprint 0603 -> (none)
- C2802: gfootprint 1206 -> (none)
- C2803: gfootprint 2917 -> (none)
- FB2801: gfootprint 0805 -> (none)
Changed lines of the file:
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@@
-			)
-		)
-		(property "gfootprint" "2917"
-			(at 0 185.42 0)
-			(effects
-				(font
-					(size 1.27 1.27)
-				)
-				(hide yes)
 			)
 		)
@@
 			)
 		)
-		(property "gfootprint" "0805"
-			(at -16.51 16.51 0)
-			(effects
-				(font
-					(size 1.27 1.27)
-				)
-				(hide yes)
-			)
-		)
 		(pin "1"
 		)
@@
 			)
 		)
-		(property "gfootprint" "0603"
-			(at 154.94 0 0)
-			(effects
-				(font
-					(size 1.27 1.27)
-				)
-				(hide yes)
-			)
-		)
 		(pin "2"
 		)
@@
 			(effects
 				(font
-					(size 1.27 1.27)
-				)
-				(hide yes)
-			)
-		)
-		(property "gfootprint" "1206"
-			(at 180.34 0 0)
-			(effects
-				(font

Commit message: vendor info
Parts:
- C2801: Vendor (none) -> digikey:490-3897-1-ND
- C2802: Vendor (none) -> digikey:490-5528-1-ND
- C2803: footprint 001_download:CAP_EEF_CD_PAN -> 001_download:CAP_EEF_CD_PAN_GH; Vendor (none) -> digikey:PCE3168CT-ND
- FB2801: Vendor (none) -> digikey:732-1620-1-ND
- U2801: Vendor (none) -> digikey:LTC6655CHLS8-2.5#PBF-ND
Changed lines of the file:
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@@
 			)
 		)
-		(property "Footprint" "001_download:CAP_EEF_CD_PAN"
+		(property "Footprint" "001_download:CAP_EEF_CD_PAN_GH"
 			(at 169.8752 96.52 0)
 			(effects
@@
 			)
 		)
+		(property "Vendor" "digikey:PCE3168CT-ND"
+			(at 0 185.42 0)
+			(effects
+				(font
+					(size 1.27 1.27)
+				)
+				(hide yes)
+			)
+		)
 		(pin "2"
 		)
@@
 			)
 		)
+		(property "Vendor" "digikey:732-1620-1-ND"
+			(at -16.51 16.51 0)
+			(effects
+				(font
+					(size 1.27 1.27)
+				)
+				(hide yes)
+			)
+		)
 		(pin "1"
 		)
@@
 			)
 		)
+		(property "Vendor" "digikey:LTC6655CHLS8-2.5#PBF-ND"
+			(at 0 167.64 0)
+			(effects
+				(font
+					(size 1.27 1.27)
+				)
+				(hide yes)
+			)
+		)
 		(pin "5"
 		)
@@
 			)
 		)
+		(property "Vendor" "digikey:490-3897-1-ND"
+			(at 154.94 0 0)
+			(effects
+				(font
+					(size 1.27 1.27)
+				)
+				(hide yes)
+			)
+		)
 		(pin "2"
 		)
@@
 			(effects
 				(font
+					(size 1.27 1.27)
+				)
+				(hide yes)
+			)
+		)
+		(property "Vendor" "digikey:490-5528-1-ND"
+			(at 180.34 0 0)
+			(effects
+				(font

Commit message: update value
Parts:
- C2801: value C -> 1UF
- C2802: value C -> 47UF
- C2803: value C -> EEF-CD1B220R
- FB2801: value FerriteBead -> 742792040
- U2801: value LTC6655CHLS8-2.5-PBF -> LTC6655CHLS8-2.5#PBF
Changed lines of the file:
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@@
 			)
 		)
-		(property "Value" "C"
+		(property "Value" "EEF-CD1B220R"
 			(at 172.72 93.9799 0)
 			(effects
@@
 			)
 		)
-		(property "Value" "FerriteBead"
+		(property "Value" "742792040"
 			(at 64.8208 76.2 90)
 			(effects
@@
 			)
 		)
-		(property "Value" "LTC6655CHLS8-2.5-PBF"
+		(property "Value" "LTC6655CHLS8-2.5#PBF"
 			(at 132.08 76.2 0)
 			(effects
@@
 			)
 		)
-		(property "Value" "C"
+		(property "Value" "1UF"
 			(at 81.28 90.1699 0)
 			(effects
@@
 			)
 		)
-		(property "Value" "C"
+		(property "Value" "47UF"
 			(at 93.98 90.1699 0)
 			(effects

Commit message: value
Parts:
- C2803: value EEF-CD1B220R -> 22UF
Changed lines of the file:
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@@
 			)
 		)
-		(property "Value" "EEF-CD1B220R"
+		(property "Value" "22UF"
 			(at 172.72 93.9799 0)
 			(effects
@@
 			)
 		)
-		(property "Description" "Unpolarized capacitor"
+		(property "Description" "Al-Poly"
 			(at 168.91 92.71 0)
 			(effects
