File: thermo_bridge.kicad_sch (KiCad schematic)
At the start: 4 parts

Commit message: Schematic Changes
Added Manufacturer/MPN/Description Fields to parts
Added libraries to project
Modified FMC schematic to use new symbol
Parts:
- R3601, R3604: Manufacturer (none) -> Murata; Manufacturer Part Number (none) -> NCP18XH103F03RB
- R3602, R3603: Manufacturer (none) -> Vishay; Manufacturer Part Number (none) -> MCT0603MD1002DP500
Changed lines of the file:
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@@
 			)
 		)
-		(property "Description" "Resistor"
+		(property "Description" "RES 10K OHM 0.5% 1/10W 0603"
 			(at 90.17 93.98 0)
 			(effects
@@
 		(property "Vendor" "digikey:MCT0603-10K-MDCT-ND"
 			(at 184.15 3.81 0)
+			(effects
+				(font
+					(size 1.27 1.27)
+				)
+				(hide yes)
+			)
+		)
+		(property "Manufacturer" "Vishay"
+			(at 90.17 93.98 0)
+			(effects
+				(font
+					(size 1.27 1.27)
+				)
+				(hide yes)
+			)
+		)
+		(property "Manufacturer Part Number" "MCT0603MD1002DP500 "
+			(at 90.17 93.98 0)
 			(effects
 				(font
@@
 			)
 		)
-		(property "Description" "Resistor"
+		(property "Description" "THERMISTOR NTC 10KOHM 3380K 0603"
 			(at 90.17 87.63 0)
 			(effects
@@
 		(property "Vendor" "digikey:490-4800-1-ND"
 			(at 177.8 177.8 0)
+			(effects
+				(font
+					(size 1.27 1.27)
+				)
+				(hide yes)
+			)
+		)
+		(property "Manufacturer" "Murata"
+			(at 90.17 87.63 0)
+			(effects
+				(font
+					(size 1.27 1.27)
+				)
+				(hide yes)
+			)
+		)
+		(property "Manufacturer Part Number" "NCP18XH103F03RB "
+			(at 90.17 87.63 0)
 			(effects
 				(font
@@
 			)
 		)
-		(property "Description" "Resistor"
+		(property "Description" "RES 10K OHM 0.5% 1/10W 0603"
 			(at 97.79 87.63 0)
 			(effects
@@
 		(property "Vendor" "digikey:MCT0603-10K-MDCT-ND"
 			(at 185.42 185.42 0)
+			(effects
+				(font
+					(size 1.27 1.27)
+				)
+				(hide yes)
+			)
+		)
+		(property "Manufacturer" "Vishay"
+			(at 97.79 87.63 0)
+			(effects
+				(font
+					(size 1.27 1.27)
+				)
+				(hide yes)
+			)
+		)
+		(property "Manufacturer Part Number" "MCT0603MD1002DP500 "
+			(at 97.79 87.63 0)
 			(effects
 				(font
@@
 			)
 		)
-		(property "Description" "Resistor"
+		(property "Description" "THERMISTOR NTC 10KOHM 3380K 0603"
 			(at 97.79 93.98 0)
 			(effects
@@
 			(effects
 				(font
+					(size 1.27 1.27)
+				)
+				(hide yes)
+			)
+		)
+		(property "Manufacturer" "Murata"
+			(at 97.79 93.98 0)
+			(effects
+				(font
+					(size 1.27 1.27)
+				)
+				(hide yes)
+			)
+		)
+		(property "Manufacturer Part Number" "NCP18XH103F03RB "
+			(at 97.79 93.98 0)
+			(effects
+				(font
