File: PowerSupply.kicad_sch (KiCad schematic)
At the start: 32 parts, among them J901 U.FL-R-SMT10, J902 U.FL-R-SMT10, J903 U.FL-R-SMT10, J904 U.FL-R-SMT10, J905 U.FL-R-SMT10, J906 U.FL-R-SMT10, U901 BAT54W-7-F, U902 ZXCT1009FTA, U903 LT6233CS6TRMPBF

Commit message: fields
Parts:
- C901, R905, TP33: gfootprint 1206 -> (none)
- C902: gfootprint 2917 -> (none)
- R901, R902, R903, R904, R906, R907, R908, R909, R910, R911, R912, R913, R914, TP32, TP34, TP35: gfootprint 0603 -> (none)
- U903: Availability In Stock -> (none); COPYRIGHT Copyright C 2016 Accelerated Designs. All rights reserved -> (none); Check_prices https://www.snapeda.com/parts/LT6233CS6%23TRMPBF/Analog+Dev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 -> (none); DIGIKEY_PART_NUMBER LT6233CS6#TRMPBFTRND -> (none); Description_1 General Purpose Amplifier 1 Circuit Rail-to-Rail TSOT-23-6 -> (none); MANUFACTURER_PART_NUMBER LT6233CS6#TRMPBF -> (none); MF Analog Devices -> (none); MP LT6233CS6#TRMPBF -> (none); Package SOT-23-6 Linear Technology -> (none); Price None -> (none); Purchase-URL https://www.snapeda.com/api/url_track_click_mouser/?unipart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 -> (none); SnapEDA_Link https://www.snapeda.com/parts/LT6233CS6%23TRMPBF/Analog+Dev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 -> (none); VENDOR Linear Technology -> (none)

Commit message: vendor info
Parts:
- C901: Vendor (none) -> digikey:490-5527-1-ND
- C902: footprint 001_download:CAP_EEF_CD_PAN -> 001_download:CAP_EEF_CD_PAN_GH; Vendor (none) -> digikey:PCE3168CT-ND
- D901, D902, D903: Vendor (none) -> digikey:754-1116-1-ND
- J901, J902, J903, J904, J905, J906: Vendor (none) -> digikey:H9161CT-ND
- R901, R902, R903: Vendor (none) -> digikey:P0.0GCT-ND
- R904, R906: Vendor (none) -> digikey:311-1.00KHRCT-ND
- R905: Vendor (none) -> digikey:1276-6187-1-ND
- R907, R908, R911, R912: Vendor (none) -> digikey:311-4.75KHRCT-ND
- R909, R910: Vendor (none) -> digikey:MCT0603-10K-MDCT-ND
- R913, R914: Vendor (none) -> digikey:311-150HRCT-ND
- U901: Vendor (none) -> digikey:BAT54W-FDICT-ND
- U902: Vendor (none) -> digikey:ZXCT1009QFTADICT-ND
- U903: Vendor (none) -> digikey:LT6233CS6#TRMPBFCT-ND

Commit message: update value
Parts:
- C901: value C -> 22UF
- C902: value C -> EEF-CD1B220R
- D901, D902, D903: value D -> APT1608CGCK
- J901, J902, J903, J904, J905, J906: value U.FL-R-SMT10 -> U.FL-R-SMT(10)
- R901, R902, R903: value R -> 0
- R904, R906: value R -> 1K
- R905: value R -> 0.1
- R907, R908, R911, R912: value R -> 4.75K
- R909, R910: value R -> 10K
- R913, R914: value R -> 150
- U902: value ZXCT1009FTA -> ZXCT1009QFTA
- U903: value LT6233CS6TRMPBF -> LT6233CS6#TRMPBF
Changed lines of the file:
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@@
 			)
 		)
-		(property "Value" "R"
+		(property "Value" "4.75K"
 			(at 223.52 199.136 90)
 			(effects
@@
 			)
 		)
-		(property "Value" "R"
+		(property "Value" "0.1"
 			(at 137.414 104.14 90)
 			(effects
@@
 			)
 		)
-		(property "Value" "U.FL-R-SMT10"
+		(property "Value" "U.FL-R-SMT(10)"
 			(at 295.91 204.4699 0)
 			(effects
@@
 			)
 		)
-		(property "Value" "D"
+		(property "Value" "APT1608CGCK"
 			(at 168.91 90.17 0)
 			(effects
@@
 			)
 		)
-		(property "Value" "R"
+		(property "Value" "150"
 			(at 289.306 170.18 90)
 			(effects
@@
 			)
 		)
-		(property "Value" "U.FL-R-SMT10"
+		(property "Value" "U.FL-R-SMT(10)"
 			(at 183.642 186.436 0)
 			(effects
@@
 			)
 		)
-		(property "Value" "U.FL-R-SMT10"
+		(property "Value" "U.FL-R-SMT(10)"
 			(at 220.98 91.948 0)
 			(effects
@@
 			)
 		)
-		(property "Value" "U.FL-R-SMT10"
+		(property "Value" "U.FL-R-SMT(10)"
 			(at 221.742 100.076 0)
 			(effects
@@
 			)
 		)
-		(property "Value" "R"
+		(property "Value" "150"
 			(at 309.626 69.85 90)
 			(effects
@@
 			)
 		)
-		(property "Value" "R"
+		(property "Value" "4.75K"
 			(at 282.956 119.38 90)
 			(effects
@@
 			)
 		)
-		(property "Value" "R"
+		(property "Value" "1K"
 			(at 163.576 91.44 90)
 			(effects
@@
 			)
 		)
-		(property "Value" "U.FL-R-SMT10"
+		(property "Value" "U.FL-R-SMT(10)"
 			(at 293.37 152.3999 0)
 			(effects
@@
 			)
 		)
-		(property "Value" "R"
+		(property "Value" "4.75K"
 			(at 216.916 182.88 90)
 			(effects
@@
 			)
 		)
-		(property "Value" "C"
+		(property "Value" "EEF-CD1B220R"
 			(at 260.35 102.8699 0)
 			(effects
@@
 			)
 		)
-		(property "Value" "D"
+		(property "Value" "APT1608CGCK"
 			(at 314.96 68.58 0)
 			(effects
@@
 			)
 		)
-		(property "Value" "R"
+		(property "Value" "0"
 			(at 97.282 78.994 90)
 			(effects
@@
 			)
 		)
-		(property "Value" "R"
+		(property "Value" "4.75K"
 			(at 289.56 128.016 90)
 			(effects
@@
 			)
 		)
-		(property "Value" "U.FL-R-SMT10"
+		(property "Value" "U.FL-R-SMT(10)"
 			(at 221.742 107.696 0)
 			(effects
@@
 			)
 		)
-		(property "Value" "ZXCT1009FTA"
+		(property "Value" "ZXCT1009QFTA"
 			(at 132.08 133.3499 90)
 			(effects
@@
 			)
 		)
-		(property "Value" "R"
+		(property "Value" "0"
 			(at 96.774 104.14 90)
 			(effects
@@
 			)
 		)
-		(property "Value" "C"
+		(property "Value" "22UF"
 			(at 158.75 106.6799 0)
 			(effects
@@
 			)
 		)
-		(property "Value" "R"
+		(property "Value" "1K"
 			(at 111.76 186.436 90)
 			(effects
@@
 			)
 		)
-		(property "Value" "R"
+		(property "Value" "0"
 			(at 97.028 94.234 90)
 			(effects
@@
 			)
 		)
-		(property "Value" "D"
+		(property "Value" "APT1608CGCK"
 			(at 294.64 168.91 0)
 			(effects
@@
 			)
 		)
-		(property "Value" "R"
+		(property "Value" "10K"
 			(at 276.86 102.616 90)
 			(effects
@@
 			)
 		)
-		(property "Value" "R"
+		(property "Value" "10K"
 			(at 276.86 94.996 90)
 			(effects
@@
 			)
 		)
-		(property "Value" "LT6233CS6TRMPBF"
+		(property "Value" "LT6233CS6#TRMPBF"
 			(at 312.42 83.82 0)
 			(effects

Commit message: value
Parts:
- C902: value EEF-CD1B220R -> 22UF
Changed lines of the file:
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@@
 			)
 		)
-		(property "Value" "EEF-CD1B220R"
+		(property "Value" "22UF"
 			(at 260.35 102.8699 0)
 			(effects
@@
 			)
 		)
-		(property "Description" "Unpolarized capacitor"
+		(property "Description" "Al-Poly"
 			(at 264.16 101.6 0)
 			(effects

Commit message: lots small updates
Parts:
- TP32, TP33, TP34, TP35: now left out of the parts list
Changed lines of the file:
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@@
 		(unit 1)
 		(exclude_from_sim no)
-		(in_bom yes)
+		(in_bom no)
 		(on_board yes)
 		(dnp no)
@@
 		(unit 1)
 		(exclude_from_sim no)
-		(in_bom yes)
+		(in_bom no)
 		(on_board yes)
 		(dnp no)
@@
 		(unit 1)
 		(exclude_from_sim no)
-		(in_bom yes)
+		(in_bom no)
 		(on_board yes)
 		(dnp no)
@@
 		(unit 1)
 		(exclude_from_sim no)
-		(in_bom yes)
-		(on_board yes)
-		(dnp no)
+		(in_bom no)
+		(on_board yes)
+		(dnp no)
