File: ad7794.kicad_sch (KiCad schematic)
At the start: 4 parts, among them U1101 AD7794BRUZ

Commit message: fields
Parts:
- C1101, R1101, R1102: gfootprint 0603 -> (none)
Changed lines of the file:
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@@
-			)
-		)
-		(property "gfootprint" "0603"
-			(at 165.1 0 0)
-			(effects
-				(font
-					(size 1.27 1.27)
-				)
-				(hide yes)
 			)
 		)
@@
 			)
 		)
-		(property "gfootprint" "0603"
-			(at 172.72 0 0)
-			(effects
-				(font
-					(size 1.27 1.27)
-				)
-				(hide yes)
-			)
-		)
 		(pin "2"
 		)
@@
 			(effects
 				(font
-					(size 1.27 1.27)
-				)
-				(hide yes)
-			)
-		)
-		(property "gfootprint" "0603"
-			(at 0 132.08 0)
-			(effects
-				(font

Commit message: vendor info
Parts:
- C1101: Vendor (none) -> digikey:490-3897-1-ND
- R1101, R1102: Vendor (none) -> digikey:P0.0GCT-ND
- U1101: Vendor (none) -> digikey:AD7794BRUZ-ND
Changed lines of the file:
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@@
+			)
+		)
+		(property "Vendor" "digikey:AD7794BRUZ-ND"
+			(at 0 154.94 0)
+			(effects
+				(font
+					(size 1.27 1.27)
+				)
+				(hide yes)
 			)
 		)
@@
 			)
 		)
+		(property "Vendor" "digikey:P0.0GCT-ND"
+			(at 165.1 0 0)
+			(effects
+				(font
+					(size 1.27 1.27)
+				)
+				(hide yes)
+			)
+		)
 		(pin "2"
 		)
@@
 			)
 		)
+		(property "Vendor" "digikey:P0.0GCT-ND"
+			(at 172.72 0 0)
+			(effects
+				(font
+					(size 1.27 1.27)
+				)
+				(hide yes)
+			)
+		)
 		(pin "2"
 		)
@@
 			(effects
 				(font
+					(size 1.27 1.27)
+				)
+				(hide yes)
+			)
+		)
+		(property "Vendor" "digikey:490-3897-1-ND"
+			(at 0 132.08 0)
+			(effects
+				(font

Commit message: update value
Parts:
- C1101: value C -> 1UF
- R1101, R1102: value R -> 0
Changed lines of the file:
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@@
 			)
 		)
-		(property "Value" "R"
+		(property "Value" "0"
 			(at 85.09 73.6599 0)
 			(effects
@@
 			)
 		)
-		(property "Value" "R"
+		(property "Value" "0"
 			(at 88.9 133.3499 0)
 			(effects
@@
 			)
 		)
-		(property "Value" "C"
+		(property "Value" "1UF"
 			(at 115.57 67.3099 0)
 			(effects

Commit message: lots small updates
Parts:
- U1101: footprint 001_download:RU_24_ADI -> 001_download:RU_24_ADI_GH
Changed lines of the file:
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@@
 			)
 		)
-		(property "Footprint" "001_download:RU_24_ADI"
+		(property "Footprint" "001_download:RU_24_ADI_GH"
 			(at 147.32 77.47 0)
 			(effects
