File: ad9653_adc0.kicad_sch (KiCad schematic)
At the start: 20 parts, among them J201 142-0701-201, J202 142-0701-201, J203 142-0701-201, J204 142-0701-201, U201 AD9653BCPZ-125

Commit message: fields
Parts:
- C201, C203, C205, C206, C210, C211, C212, C213, R201, R202: gfootprint 0603 -> (none)
- C202, C204, C207, C208, C209: gfootprint 0402 -> (none)
Changed lines of the file:
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@@
-			)
-		)
-		(property "gfootprint" "0603"
-			(at 115.57 -115.57 0)
-			(effects
-				(font
-					(size 1.27 1.27)
-				)
-				(hide yes)
 			)
 		)
@@
 			)
 		)
-		(property "gfootprint" "0603"
-			(at 0 139.7 0)
-			(effects
-				(font
-					(size 1.27 1.27)
-				)
-				(hide yes)
-			)
-		)
 		(pin "2"
 		)
@@
 		(property "Description" "Resistor"
 			(at 76.2 134.62 0)
-			(effects
-				(font
-					(size 1.27 1.27)
-				)
-				(hide yes)
-			)
-		)
-		(property "gfootprint" "0603"
-			(at 0 269.24 0)
 			(effects
 				(font
@@
 			)
 		)
-		(property "gfootprint" "0603"
-			(at 0 86.36 0)
-			(effects
-				(font
-					(size 1.27 1.27)
-				)
-				(hide yes)
-			)
-		)
 		(pin "2"
 		)
@@
 		(property "Description" "Unpolarized capacitor"
 			(at 54.61 60.96 0)
-			(effects
-				(font
-					(size 1.27 1.27)
-				)
-				(hide yes)
-			)
-		)
-		(property "gfootprint" "0603"
-			(at 0 121.92 0)
 			(effects
 				(font
@@
 			)
 		)
-		(property "gfootprint" "0402"
-			(at 0 86.36 0)
-			(effects
-				(font
-					(size 1.27 1.27)
-				)
-				(hide yes)
-			)
-		)
 		(pin "2"
 		)
@@
 		(property "Description" "Unpolarized capacitor"
 			(at 74.93 43.18 0)
-			(effects
-				(font
-					(size 1.27 1.27)
-				)
-				(hide yes)
-			)
-		)
-		(property "gfootprint" "0402"
-			(at 0 86.36 0)
 			(effects
 				(font
@@
 			)
 		)
-		(property "gfootprint" "0603"
-			(at 0 121.92 0)
-			(effects
-				(font
-					(size 1.27 1.27)
-				)
-				(hide yes)
-			)
-		)
 		(pin "2"
 		)
@@
 			)
 		)
-		(property "gfootprint" "0603"
-			(at 0 55.88 0)
-			(effects
-				(font
-					(size 1.27 1.27)
-				)
-				(hide yes)
-			)
-		)
 		(pin "2"
 		)
@@
 		(property "Description" "Unpolarized capacitor"
 			(at 207.01 69.85 0)
-			(effects
-				(font
-					(size 1.27 1.27)
-				)
-				(hide yes)
-			)
-		)
-		(property "gfootprint" "0603"
-			(at 0 139.7 0)
 			(effects
 				(font
@@
 			)
 		)
-		(property "gfootprint" "0402"
-			(at 0 86.36 0)
-			(effects
-				(font
-					(size 1.27 1.27)
-				)
-				(hide yes)
-			)
-		)
 		(pin "2"
 		)
@@
 			)
 		)
-		(property "gfootprint" "0402"
-			(at 0 55.88 0)
-			(effects
-				(font
-					(size 1.27 1.27)
-				)
-				(hide yes)
-			)
-		)
 		(pin "2"
 		)
@@
 		(property "Description" "Unpolarized capacitor"
 			(at 46.99 43.18 0)
-			(effects
-				(font
-					(size 1.27 1.27)
-				)
-				(hide yes)
-			)
-		)
-		(property "gfootprint" "0402"
-			(at 0 86.36 0)
 			(effects
 				(font
@@
 			)
 		)
-		(property "gfootprint" "0603"
-			(at 113.03 306.07 0)
-			(effects
-				(font
-					(size 1.27 1.27)
-				)
-				(hide yes)
-			)
-		)
 		(pin "1"
 		)
@@
 			(effects
 				(font
-					(size 1.27 1.27)
-				)
-				(hide yes)
-			)
-		)
-		(property "gfootprint" "0603"
-			(at 0 190.5 0)
-			(effects
-				(font

Commit message: vendor info
Parts:
- C201, C205: Vendor (none) -> digikey:445-6853-1-ND
- C202, C204, C207, C208, C209: Vendor (none) -> digikey:490-1318-1-ND
- C203, C211, C212, C213: Vendor (none) -> digikey:445-2664-1-ND
- C206: Vendor (none) -> digikey:478-8725-1-ND
- J201, J202, J203, J204: Vendor (none) -> digikey:J500-ND
- R201: Vendor (none) -> digikey:MCT0603-10K-MDCT-ND
- R202: Vendor (none) -> digikey:311-100HRCT-ND
- U201: Vendor (none) -> digikey:AD9653BCPZ-125-ND
Changed lines of the file:
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@@
+			)
+		)
+		(property "Vendor" "digikey:445-2664-1-ND"
+			(at 115.57 -115.57 0)
+			(effects
+				(font
+					(size 1.27 1.27)
+				)
+				(hide yes)
 			)
 		)
@@
 		(property "Description" ""
 			(at 256.54 83.82 0)
+			(effects
+				(font
+					(size 1.27 1.27)
+				)
+				(hide yes)
+			)
+		)
+		(property "Vendor" "digikey:J500-ND"
+			(at 0 167.64 0)
 			(effects
 				(font
@@
 			)
 		)
+		(property "Vendor" "digikey:445-2664-1-ND"
+			(at 0 139.7 0)
+			(effects
+				(font
+					(size 1.27 1.27)
+				)
+				(hide yes)
+			)
+		)
 		(pin "2"
 		)
@@
 		(property "Description" "Resistor"
 			(at 76.2 134.62 0)
+			(effects
+				(font
+					(size 1.27 1.27)
+				)
+				(hide yes)
+			)
+		)
+		(property "Vendor" "digikey:MCT0603-10K-MDCT-ND"
+			(at 0 269.24 0)
 			(effects
 				(font
@@
 			)
 		)
+		(property "Vendor" "digikey:445-6853-1-ND"
+			(at 0 86.36 0)
+			(effects
+				(font
+					(size 1.27 1.27)
+				)
+				(hide yes)
+			)
+		)
 		(pin "2"
 		)
@@
 		(property "Description" "Unpolarized capacitor"
 			(at 54.61 60.96 0)
+			(effects
+				(font
+					(size 1.27 1.27)
+				)
+				(hide yes)
+			)
+		)
+		(property "Vendor" "digikey:478-8725-1-ND"
+			(at 0 121.92 0)
 			(effects
 				(font
@@
 			)
 		)
+		(property "Vendor" "digikey:J500-ND"
+			(at 91.44 228.6 0)
+			(effects
+				(font
+					(size 1.27 1.27)
+				)
+				(hide yes)
+			)
+		)
 		(pin "1"
 		)
@@
 			)
 		)
+		(property "Vendor" "digikey:490-1318-1-ND"
+			(at 0 86.36 0)
+			(effects
+				(font
+					(size 1.27 1.27)
+				)
+				(hide yes)
+			)
+		)
 		(pin "2"
 		)
@@
 		(property "Description" "Unpolarized capacitor"
 			(at 74.93 43.18 0)
+			(effects
+				(font
+					(size 1.27 1.27)
+				)
+				(hide yes)
+			)
+		)
+		(property "Vendor" "digikey:490-1318-1-ND"
+			(at 0 86.36 0)
 			(effects
 				(font
@@
 			)
 		)
+		(property "Vendor" "digikey:J500-ND"
+			(at 91.44 203.2 0)
+			(effects
+				(font
+					(size 1.27 1.27)
+				)
+				(hide yes)
+			)
+		)
 		(pin "1"
 		)
@@
 		(property "Description" "Unpolarized capacitor"
 			(at 48.26 60.96 0)
+			(effects
+				(font
+					(size 1.27 1.27)
+				)
+				(hide yes)
+			)
+		)
+		(property "Vendor" "digikey:445-2664-1-ND"
+			(at 0 121.92 0)
 			(effects
 				(font
@@
 			)
 		)
+		(property "Vendor" "digikey:J500-ND"
+			(at 91.44 167.64 0)
+			(effects
+				(font
+					(size 1.27 1.27)
+				)
+				(hide yes)
+			)
+		)
 		(pin "1"
 		)
@@
 		(property "Description" "Unpolarized capacitor"
 			(at 46.99 27.94 0)
+			(effects
+				(font
+					(size 1.27 1.27)
+				)
+				(hide yes)
+			)
+		)
+		(property "Vendor" "digikey:445-6853-1-ND"
+			(at 0 55.88 0)
 			(effects
 				(font
@@
 			)
 		)
+		(property "Vendor" "digikey:490-1318-1-ND"
+			(at 0 86.36 0)
+			(effects
+				(font
+					(size 1.27 1.27)
+				)
+				(hide yes)
+			)
+		)
 		(pin "2"
 		)
@@
 			)
 		)
+		(property "Vendor" "digikey:490-1318-1-ND"
+			(at 0 55.88 0)
+			(effects
+				(font
+					(size 1.27 1.27)
+				)
+				(hide yes)
+			)
+		)
 		(pin "2"
 		)
@@
 		(property "Description" "Unpolarized capacitor"
 			(at 46.99 43.18 0)
+			(effects
+				(font
+					(size 1.27 1.27)
+				)
+				(hide yes)
+			)
+		)
+		(property "Vendor" "digikey:490-1318-1-ND"
+			(at 0 86.36 0)
 			(effects
 				(font
@@
 			)
 		)
+		(property "Vendor" "digikey:AD9653BCPZ-125-ND"
+			(at 398.78 167.64 0)
+			(effects
+				(font
+					(size 1.27 1.27)
+				)
+				(hide yes)
+			)
+		)
 		(pin "18"
 		)
@@
 			)
 		)
+		(property "Vendor" "digikey:445-2664-1-ND"
+			(at 113.03 306.07 0)
+			(effects
+				(font
+					(size 1.27 1.27)
+				)
+				(hide yes)
+			)
+		)
 		(pin "1"
 		)
@@
 			(effects
 				(font
+					(size 1.27 1.27)
+				)
+				(hide yes)
+			)
+		)
+		(property "Vendor" "digikey:311-100HRCT-ND"
+			(at 0 190.5 0)
+			(effects
+				(font

Commit message: update value
Parts:
- C201, C205: value C -> 10UF
- C202, C204, C207, C208, C209: value C -> 0.1UF
- C203, C211, C212, C213: value C -> 10000PF
- C206: value C -> F381A225MMA
- R201: value R -> 10K
- R202: value R -> 100
Changed lines of the file:
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@@
 			)
 		)
-		(property "Value" "C"
+		(property "Value" "10000PF"
 			(at 209.55 99.06 90)
 			(effects
@@
 			)
 		)
-		(property "Value" "C"
+		(property "Value" "10000PF"
 			(at 223.52 71.1199 0)
 			(effects
@@
 			)
 		)
-		(property "Value" "R"
+		(property "Value" "10K"
 			(at 78.74 135.8899 0)
 			(effects
@@
 			)
 		)
-		(property "Value" "C"
+		(property "Value" "10UF"
 			(at 58.42 44.4499 0)
 			(effects
@@
 			)
 		)
-		(property "Value" "C"
+		(property "Value" "F381A225MMA"
 			(at 58.42 62.2299 0)
 			(effects
@@
 			)
 		)
-		(property "Value" "C"
+		(property "Value" "0.1UF"
 			(at 64.77 44.4499 0)
 			(effects
@@
 			)
 		)
-		(property "Value" "C"
+		(property "Value" "0.1UF"
 			(at 78.74 44.4499 0)
 			(effects
@@
 			)
 		)
-		(property "Value" "C"
+		(property "Value" "10000PF"
 			(at 52.07 62.2299 0)
 			(effects
@@
 			)
 		)
-		(property "Value" "C"
+		(property "Value" "10UF"
 			(at 50.8 29.2099 0)
 			(effects
@@
 			)
 		)
-		(property "Value" "C"
+		(property "Value" "0.1UF"
 			(at 71.12 44.4499 0)
 			(effects
@@
 			)
 		)
-		(property "Value" "C"
+		(property "Value" "0.1UF"
 			(at 57.15 29.2099 0)
 			(effects
@@
 			)
 		)
-		(property "Value" "C"
+		(property "Value" "0.1UF"
 			(at 50.8 44.4499 0)
 			(effects
@@
 			)
 		)
-		(property "Value" "C"
+		(property "Value" "10000PF"
 			(at 209.55 91.44 90)
 			(effects
@@
 			)
 		)
-		(property "Value" "R"
+		(property "Value" "100"
 			(at 222.25 96.5199 0)
 			(effects

Commit message: value
Parts:
- C206: value F381A225MMA -> 2.2UF
Changed lines of the file:
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@@
 			)
 		)
-		(property "Value" "F381A225MMA"
+		(property "Value" "2.2UF"
 			(at 58.42 62.2299 0)
 			(effects
@@
 			)
 		)
-		(property "Description" "Unpolarized capacitor"
+		(property "Description" "Tant_poly"
 			(at 54.61 60.96 0)
 			(effects

Commit message: lots small updates
Parts:
- C210: value C -> DNP
- J201, J202, J203, J204: footprint 001_download:CONN_142-0701-201_CIN -> CONN_142-0701-201_CIN; symbol 001_symbol:142-0701-201 -> 001_symbol:142-0701-201_GH
Connections:
- net GND: now also J201.2, J201.3, J201.4, J201.5, J202.2, J202.3, J202.4, J202.5, J203.2, J203.3, J203.4, J203.5, J204.2, J204.3, J204.4, J204.5
