File: ad9653_adc1.kicad_sch (KiCad schematic)
At the start: 20 parts, among them J701 142-0701-201, J702 142-0701-201, J703 142-0701-201, J704 142-0701-201, U701 AD9653BCPZ-125

Commit message: fields
Parts:
- C701, C703, C705, C706, C710, C711, C712, C713, R701, R702: gfootprint 0603 -> (none)
- C702, C704, C707, C708, C709: gfootprint 0402 -> (none)
Changed lines of the file:
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@@
-			)
-		)
-		(property "gfootprint" "0603"
-			(at 0 59.69 0)
-			(effects
-				(font
-					(size 1.27 1.27)
-				)
-				(hide yes)
 			)
 		)
@@
 			)
 		)
-		(property "gfootprint" "0603"
-			(at 0 143.51 0)
-			(effects
-				(font
-					(size 1.27 1.27)
-				)
-				(hide yes)
-			)
-		)
 		(pin "1"
 		)
@@
 			)
 		)
-		(property "gfootprint" "0603"
-			(at 0 273.05 0)
-			(effects
-				(font
-					(size 1.27 1.27)
-				)
-				(hide yes)
-			)
-		)
 		(pin "2"
 		)
@@
 		(property "Description" "Unpolarized capacitor"
 			(at 74.93 46.99 0)
-			(effects
-				(font
-					(size 1.27 1.27)
-				)
-				(hide yes)
-			)
-		)
-		(property "gfootprint" "0402"
-			(at 0 90.17 0)
 			(effects
 				(font
@@
 			)
 		)
-		(property "gfootprint" "0603"
-			(at 0 143.51 0)
-			(effects
-				(font
-					(size 1.27 1.27)
-				)
-				(hide yes)
-			)
-		)
 		(pin "2"
 		)
@@
 			)
 		)
-		(property "gfootprint" "0603"
-			(at 0 90.17 0)
-			(effects
-				(font
-					(size 1.27 1.27)
-				)
-				(hide yes)
-			)
-		)
 		(pin "2"
 		)
@@
 			)
 		)
-		(property "gfootprint" "0402"
-			(at 0 59.69 0)
-			(effects
-				(font
-					(size 1.27 1.27)
-				)
-				(hide yes)
-			)
-		)
 		(pin "2"
 		)
@@
 		(property "Description" "Resistor"
 			(at 219.71 99.06 0)
-			(effects
-				(font
-					(size 1.27 1.27)
-				)
-				(hide yes)
-			)
-		)
-		(property "gfootprint" "0603"
-			(at 0 194.31 0)
 			(effects
 				(font
@@
 			)
 		)
-		(property "gfootprint" "0402"
-			(at 0 90.17 0)
-			(effects
-				(font
-					(size 1.27 1.27)
-				)
-				(hide yes)
-			)
-		)
 		(pin "2"
 		)
@@
 			)
 		)
-		(property "gfootprint" "0603"
-			(at 113.03 309.88 0)
-			(effects
-				(font
-					(size 1.27 1.27)
-				)
-				(hide yes)
-			)
-		)
 		(pin "1"
 		)
@@
 			)
 		)
-		(property "gfootprint" "0603"
-			(at 0 125.73 0)
-			(effects
-				(font
-					(size 1.27 1.27)
-				)
-				(hide yes)
-			)
-		)
 		(pin "2"
 		)
@@
 		(property "Description" "Unpolarized capacitor"
 			(at 67.31 46.99 0)
-			(effects
-				(font
-					(size 1.27 1.27)
-				)
-				(hide yes)
-			)
-		)
-		(property "gfootprint" "0402"
-			(at 0 90.17 0)
 			(effects
 				(font
@@
 			)
 		)
-		(property "gfootprint" "0402"
-			(at 0 90.17 0)
-			(effects
-				(font
-					(size 1.27 1.27)
-				)
-				(hide yes)
-			)
-		)
 		(pin "2"
 		)
@@
 			)
 		)
-		(property "gfootprint" "0603"
-			(at 115.57 -111.76 0)
-			(effects
-				(font
-					(size 1.27 1.27)
-				)
-				(hide yes)
-			)
-		)
 		(pin "1"
 		)
@@
 			(effects
 				(font
-					(size 1.27 1.27)
-				)
-				(hide yes)
-			)
-		)
-		(property "gfootprint" "0603"
-			(at 0 125.73 0)
-			(effects
-				(font

Commit message: vendor info
Parts:
- C701, C705: Vendor (none) -> digikey:445-6853-1-ND
- C702, C704, C707, C708, C709: Vendor (none) -> digikey:490-1318-1-ND
- C703, C711, C712, C713: Vendor (none) -> digikey:445-2664-1-ND
- C706: Vendor (none) -> digikey:478-8725-1-ND
- J701, J702, J703, J704: Vendor (none) -> digikey:J500-ND
- R701: Vendor (none) -> digikey:MCT0603-10K-MDCT-ND
- R702: Vendor (none) -> digikey:311-100HRCT-ND
- U701: Vendor (none) -> digikey:AD9653BCPZ-125-ND
Changed lines of the file:
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@@
+			)
+		)
+		(property "Vendor" "digikey:J500-ND"
+			(at 0 175.26 0)
+			(effects
+				(font
+					(size 1.27 1.27)
+				)
+				(hide yes)
 			)
 		)
@@
 			)
 		)
+		(property "Vendor" "digikey:J500-ND"
+			(at 91.44 175.26 0)
+			(effects
+				(font
+					(size 1.27 1.27)
+				)
+				(hide yes)
+			)
+		)
 		(pin "1"
 		)
@@
 			)
 		)
+		(property "Vendor" "digikey:445-6853-1-ND"
+			(at 0 63.5 0)
+			(effects
+				(font
+					(size 1.27 1.27)
+				)
+				(hide yes)
+			)
+		)
 		(pin "2"
 		)
@@
 			)
 		)
+		(property "Vendor" "digikey:MCT0603-10K-MDCT-ND"
+			(at 0 276.86 0)
+			(effects
+				(font
+					(size 1.27 1.27)
+				)
+				(hide yes)
+			)
+		)
 		(pin "2"
 		)
@@
 		(property "Description" "Unpolarized capacitor"
 			(at 74.93 46.99 0)
+			(effects
+				(font
+					(size 1.27 1.27)
+				)
+				(hide yes)
+			)
+		)
+		(property "Vendor" "digikey:490-1318-1-ND"
+			(at 0 93.98 0)
 			(effects
 				(font
@@
 			)
 		)
+		(property "Vendor" "digikey:J500-ND"
+			(at 91.44 210.82 0)
+			(effects
+				(font
+					(size 1.27 1.27)
+				)
+				(hide yes)
+			)
+		)
 		(pin "1"
 		)
@@
 		(property "Description" "Unpolarized capacitor"
 			(at 219.71 73.66 0)
+			(effects
+				(font
+					(size 1.27 1.27)
+				)
+				(hide yes)
+			)
+		)
+		(property "Vendor" "digikey:445-2664-1-ND"
+			(at 0 147.32 0)
 			(effects
 				(font
@@
 			)
 		)
+		(property "Vendor" "digikey:J500-ND"
+			(at 91.44 236.22 0)
+			(effects
+				(font
+					(size 1.27 1.27)
+				)
+				(hide yes)
+			)
+		)
 		(pin "1"
 		)
@@
 			)
 		)
+		(property "Vendor" "digikey:445-6853-1-ND"
+			(at 0 93.98 0)
+			(effects
+				(font
+					(size 1.27 1.27)
+				)
+				(hide yes)
+			)
+		)
 		(pin "2"
 		)
@@
 			)
 		)
+		(property "Vendor" "digikey:490-1318-1-ND"
+			(at 0 63.5 0)
+			(effects
+				(font
+					(size 1.27 1.27)
+				)
+				(hide yes)
+			)
+		)
 		(pin "2"
 		)
@@
 		(property "Description" "Resistor"
 			(at 219.71 99.06 0)
+			(effects
+				(font
+					(size 1.27 1.27)
+				)
+				(hide yes)
+			)
+		)
+		(property "Vendor" "digikey:311-100HRCT-ND"
+			(at 0 198.12 0)
 			(effects
 				(font
@@
 			)
 		)
+		(property "Vendor" "digikey:AD9653BCPZ-125-ND"
+			(at 398.78 175.26 0)
+			(effects
+				(font
+					(size 1.27 1.27)
+				)
+				(hide yes)
+			)
+		)
 		(pin "18"
 		)
@@
 			)
 		)
+		(property "Vendor" "digikey:490-1318-1-ND"
+			(at 0 93.98 0)
+			(effects
+				(font
+					(size 1.27 1.27)
+				)
+				(hide yes)
+			)
+		)
 		(pin "2"
 		)
@@
 			)
 		)
+		(property "Vendor" "digikey:445-2664-1-ND"
+			(at 109.22 309.88 0)
+			(effects
+				(font
+					(size 1.27 1.27)
+				)
+				(hide yes)
+			)
+		)
 		(pin "1"
 		)
@@
 			)
 		)
+		(property "Vendor" "digikey:478-8725-1-ND"
+			(at 0 129.54 0)
+			(effects
+				(font
+					(size 1.27 1.27)
+				)
+				(hide yes)
+			)
+		)
 		(pin "2"
 		)
@@
 		(property "Description" "Unpolarized capacitor"
 			(at 67.31 46.99 0)
+			(effects
+				(font
+					(size 1.27 1.27)
+				)
+				(hide yes)
+			)
+		)
+		(property "Vendor" "digikey:490-1318-1-ND"
+			(at 0 93.98 0)
 			(effects
 				(font
@@
 			)
 		)
+		(property "Vendor" "digikey:490-1318-1-ND"
+			(at 0 93.98 0)
+			(effects
+				(font
+					(size 1.27 1.27)
+				)
+				(hide yes)
+			)
+		)
 		(pin "2"
 		)
@@
 			)
 		)
+		(property "Vendor" "digikey:445-2664-1-ND"
+			(at 111.76 -111.76 0)
+			(effects
+				(font
+					(size 1.27 1.27)
+				)
+				(hide yes)
+			)
+		)
 		(pin "1"
 		)
@@
 			(effects
 				(font
+					(size 1.27 1.27)
+				)
+				(hide yes)
+			)
+		)
+		(property "Vendor" "digikey:445-2664-1-ND"
+			(at 0 129.54 0)
+			(effects
+				(font

Commit message: update value
Parts:
- C701, C705: value C -> 10UF
- C702, C704, C707, C708, C709: value C -> 0.1UF
- C703, C711, C712, C713: value C -> 10000PF
- C706: value C -> F381A225MMA
- R701: value R -> 10K
- R702: value R -> 100
Changed lines of the file:
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@@
 			)
 		)
-		(property "Value" "C"
+		(property "Value" "10UF"
 			(at 50.8 33.0199 0)
 			(effects
@@
 			)
 		)
-		(property "Value" "R"
+		(property "Value" "10K"
 			(at 78.74 139.6999 0)
 			(effects
@@
 			)
 		)
-		(property "Value" "C"
+		(property "Value" "0.1UF"
 			(at 78.74 48.2599 0)
 			(effects
@@
 			)
 		)
-		(property "Value" "C"
+		(property "Value" "10000PF"
 			(at 223.52 74.9299 0)
 			(effects
@@
 			)
 		)
-		(property "Value" "C"
+		(property "Value" "10UF"
 			(at 58.42 48.2599 0)
 			(effects
@@
 			)
 		)
-		(property "Value" "C"
+		(property "Value" "0.1UF"
 			(at 57.15 33.0199 0)
 			(effects
@@
 			)
 		)
-		(property "Value" "R"
+		(property "Value" "100"
 			(at 222.25 100.3299 0)
 			(effects
@@
 			)
 		)
-		(property "Value" "C"
+		(property "Value" "0.1UF"
 			(at 64.77 48.2599 0)
 			(effects
@@
 			)
 		)
-		(property "Value" "C"
+		(property "Value" "10000PF"
 			(at 209.55 95.25 90)
 			(effects
@@
 			)
 		)
-		(property "Value" "C"
+		(property "Value" "F381A225MMA"
 			(at 58.42 66.0399 0)
 			(effects
@@
 			)
 		)
-		(property "Value" "C"
+		(property "Value" "0.1UF"
 			(at 71.12 48.2599 0)
 			(effects
@@
 			)
 		)
-		(property "Value" "C"
+		(property "Value" "0.1UF"
 			(at 50.8 48.2599 0)
 			(effects
@@
 			)
 		)
-		(property "Value" "C"
+		(property "Value" "10000PF"
 			(at 209.55 102.87 90)
 			(effects
@@
 			)
 		)
-		(property "Value" "C"
+		(property "Value" "10000PF"
 			(at 52.07 66.0399 0)
 			(effects

Commit message: value
Parts:
- C706: value F381A225MMA -> 2.2UF
Changed lines of the file:
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@@
 			)
 		)
-		(property "Value" "F381A225MMA"
+		(property "Value" "2.2UF"
 			(at 58.42 66.0399 0)
 			(effects
@@
 			)
 		)
-		(property "Description" "Unpolarized capacitor"
+		(property "Description" "Tant_poly"
 			(at 54.61 64.77 0)
 			(effects

Commit message: lots small updates
Parts:
- C710: value C -> DNP
- J701, J702, J703, J704: footprint 001_download:CONN_142-0701-201_CIN -> CONN_142-0701-201_CIN; symbol 001_symbol:142-0701-201 -> 001_symbol:142-0701-201_GH
Connections:
- net GND: now also J701.2, J701.3, J701.4, J701.5, J702.2, J702.3, J702.4, J702.5, J703.2, J703.3, J703.4, J703.5, J704.2, J704.3, J704.4, J704.5
