File: ad9781.kicad_sch (KiCad schematic)
At the start: 20 parts, among them J1201 142-0701-201, J1202 142-0701-201, U1201 AD9781BCPZ

Commit message: fields
Parts:
- C1201, C1205, C1207, C1210, C1212: gfootprint 0402 -> (none)
- C1202, C1203, C1204, C1206, C1208, C1209, C1211, R1201, R1202, R1203, R1204, R1205: gfootprint 0603 -> (none)
Changed lines of the file:
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@@
-			)
-		)
-		(property "gfootprint" "0603"
-			(at 0 96.52 0)
-			(effects
-				(font
-					(size 1.27 1.27)
-				)
-				(hide yes)
 			)
 		)
@@
 			)
 		)
-		(property "gfootprint" "0603"
-			(at 490.22 0 0)
-			(effects
-				(font
-					(size 1.27 1.27)
-				)
-				(hide yes)
-			)
-		)
 		(pin "1"
 		)
@@
 		(property "Description" "Unpolarized capacitor"
 			(at 46.99 80.01 0)
-			(effects
-				(font
-					(size 1.27 1.27)
-				)
-				(hide yes)
-			)
-		)
-		(property "gfootprint" "0603"
-			(at 127 127 0)
 			(effects
 				(font
@@
 			)
 		)
-		(property "gfootprint" "0603"
-			(at 167.64 187.96 0)
-			(effects
-				(font
-					(size 1.27 1.27)
-				)
-				(hide yes)
-			)
-		)
 		(pin "2"
 		)
@@
 			)
 		)
-		(property "gfootprint" "0603"
-			(at 0 0 0)
-			(effects
-				(font
-					(size 1.27 1.27)
-				)
-				(hide yes)
-			)
-		)
 		(pin "1"
 		)
@@
 			)
 		)
-		(property "gfootprint" "0603"
-			(at 0 96.52 0)
-			(effects
-				(font
-					(size 1.27 1.27)
-				)
-				(hide yes)
-			)
-		)
 		(pin "2"
 		)
@@
 			)
 		)
-		(property "gfootprint" "0402"
-			(at 0 96.52 0)
-			(effects
-				(font
-					(size 1.27 1.27)
-				)
-				(hide yes)
-			)
-		)
 		(pin "2"
 		)
@@
 			)
 		)
-		(property "gfootprint" "0603"
-			(at 0 147.32 0)
-			(effects
-				(font
-					(size 1.27 1.27)
-				)
-				(hide yes)
-			)
-		)
 		(pin "1"
 		)
@@
 			)
 		)
-		(property "gfootprint" "0402"
-			(at 505.46 0 0)
-			(effects
-				(font
-					(size 1.27 1.27)
-				)
-				(hide yes)
-			)
-		)
 		(pin "2"
 		)
@@
 			)
 		)
-		(property "gfootprint" "0402"
-			(at 0 96.52 0)
-			(effects
-				(font
-					(size 1.27 1.27)
-				)
-				(hide yes)
-			)
-		)
 		(pin "2"
 		)
@@
 			)
 		)
-		(property "gfootprint" "0402"
-			(at 0 96.52 0)
-			(effects
-				(font
-					(size 1.27 1.27)
-				)
-				(hide yes)
-			)
-		)
 		(pin "2"
 		)
@@
 			)
 		)
-		(property "gfootprint" "0603"
-			(at 0 96.52 0)
-			(effects
-				(font
-					(size 1.27 1.27)
-				)
-				(hide yes)
-			)
-		)
 		(pin "2"
 		)
@@
 			)
 		)
-		(property "gfootprint" "0402"
-			(at 0 96.52 0)
-			(effects
-				(font
-					(size 1.27 1.27)
-				)
-				(hide yes)
-			)
-		)
 		(pin "2"
 		)
@@
 		(property "Description" "Unpolarized capacitor"
 			(at 87.63 48.26 0)
-			(effects
-				(font
-					(size 1.27 1.27)
-				)
-				(hide yes)
-			)
-		)
-		(property "gfootprint" "0603"
-			(at 0 96.52 0)
 			(effects
 				(font
@@
 			)
 		)
-		(property "gfootprint" "0603"
-			(at 148.59 54.61 0)
-			(effects
-				(font
-					(size 1.27 1.27)
-				)
-				(hide yes)
-			)
-		)
 		(pin "2"
 		)
@@
 			)
 		)
-		(property "gfootprint" "0603"
-			(at 0 0 0)
-			(effects
-				(font
-					(size 1.27 1.27)
-				)
-				(hide yes)
-			)
-		)
 		(pin "1"
 		)
@@
 			(effects
 				(font
-					(size 1.27 1.27)
-				)
-				(hide yes)
-			)
-		)
-		(property "gfootprint" "0603"
-			(at 139.7 190.5 0)
-			(effects
-				(font

Commit message: vendor info
Parts:
- C1201, C1205, C1207, C1210, C1212: Vendor (none) -> digikey:490-1318-1-ND
- C1202, C1203, C1208: Vendor (none) -> digikey:490-1451-1-ND
- C1204, C1206, C1209, C1211: Vendor (none) -> digikey:445-6853-1-ND
- J1201, J1202: Vendor (none) -> digikey:J500-ND
- R1201, R1202: Vendor (none) -> digikey:311-49.9HRCT-ND
- R1203: Vendor (none) -> digikey:311-1.00KHRCT-ND
- R1204: Vendor (none) -> digikey:311-287HRCT-ND
- R1205: Vendor (none) -> digikey:MCT0603-10K-MDCT-ND
- U1201: Vendor (none) -> digikey:AD9781BCPZ-ND
Changed lines of the file:
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@@
+			)
+		)
+		(property "Vendor" "digikey:445-6853-1-ND"
+			(at 0 96.52 0)
+			(effects
+				(font
+					(size 1.27 1.27)
+				)
+				(hide yes)
 			)
 		)
@@
 			)
 		)
+		(property "Vendor" "digikey:MCT0603-10K-MDCT-ND"
+			(at 490.22 0 0)
+			(effects
+				(font
+					(size 1.27 1.27)
+				)
+				(hide yes)
+			)
+		)
 		(pin "1"
 		)
@@
 		(property "Description" "Unpolarized capacitor"
 			(at 46.99 80.01 0)
+			(effects
+				(font
+					(size 1.27 1.27)
+				)
+				(hide yes)
+			)
+		)
+		(property "Vendor" "digikey:490-1451-1-ND"
+			(at 127 127 0)
 			(effects
 				(font
@@
 			)
 		)
+		(property "Vendor" "digikey:490-1451-1-ND"
+			(at 167.64 187.96 0)
+			(effects
+				(font
+					(size 1.27 1.27)
+				)
+				(hide yes)
+			)
+		)
 		(pin "2"
 		)
@@
 			)
 		)
+		(property "Vendor" "digikey:311-287HRCT-ND"
+			(at 0 0 0)
+			(effects
+				(font
+					(size 1.27 1.27)
+				)
+				(hide yes)
+			)
+		)
 		(pin "1"
 		)
@@
 			)
 		)
+		(property "Vendor" "digikey:445-6853-1-ND"
+			(at 0 96.52 0)
+			(effects
+				(font
+					(size 1.27 1.27)
+				)
+				(hide yes)
+			)
+		)
 		(pin "2"
 		)
@@
 			)
 		)
+		(property "Vendor" "digikey:490-1318-1-ND"
+			(at 0 96.52 0)
+			(effects
+				(font
+					(size 1.27 1.27)
+				)
+				(hide yes)
+			)
+		)
 		(pin "2"
 		)
@@
 			)
 		)
+		(property "Vendor" "digikey:311-1.00KHRCT-ND"
+			(at 0 147.32 0)
+			(effects
+				(font
+					(size 1.27 1.27)
+				)
+				(hide yes)
+			)
+		)
 		(pin "1"
 		)
@@
 			)
 		)
+		(property "Vendor" "digikey:490-1318-1-ND"
+			(at 505.46 0 0)
+			(effects
+				(font
+					(size 1.27 1.27)
+				)
+				(hide yes)
+			)
+		)
 		(pin "2"
 		)
@@
 			)
 		)
+		(property "Vendor" "digikey:490-1318-1-ND"
+			(at 0 96.52 0)
+			(effects
+				(font
+					(size 1.27 1.27)
+				)
+				(hide yes)
+			)
+		)
 		(pin "2"
 		)
@@
 			)
 		)
+		(property "Vendor" "digikey:J500-ND"
+			(at 0 147.32 0)
+			(effects
+				(font
+					(size 1.27 1.27)
+				)
+				(hide yes)
+			)
+		)
 		(pin "1"
 		)
@@
 			)
 		)
+		(property "Vendor" "digikey:490-1318-1-ND"
+			(at 0 96.52 0)
+			(effects
+				(font
+					(size 1.27 1.27)
+				)
+				(hide yes)
+			)
+		)
 		(pin "2"
 		)
@@
 			)
 		)
+		(property "Vendor" "digikey:AD9781BCPZ-ND"
+			(at 0 127 0)
+			(effects
+				(font
+					(size 1.27 1.27)
+				)
+				(hide yes)
+			)
+		)
 		(pin "37"
 		)
@@
 			)
 		)
+		(property "Vendor" "digikey:445-6853-1-ND"
+			(at 0 96.52 0)
+			(effects
+				(font
+					(size 1.27 1.27)
+				)
+				(hide yes)
+			)
+		)
 		(pin "2"
 		)
@@
 			)
 		)
+		(property "Vendor" "digikey:490-1318-1-ND"
+			(at 0 96.52 0)
+			(effects
+				(font
+					(size 1.27 1.27)
+				)
+				(hide yes)
+			)
+		)
 		(pin "2"
 		)
@@
 		(property "Description" "Unpolarized capacitor"
 			(at 87.63 48.26 0)
+			(effects
+				(font
+					(size 1.27 1.27)
+				)
+				(hide yes)
+			)
+		)
+		(property "Vendor" "digikey:445-6853-1-ND"
+			(at 0 96.52 0)
 			(effects
 				(font
@@
 			)
 		)
+		(property "Vendor" "digikey:J500-ND"
+			(at 0 0 0)
+			(effects
+				(font
+					(size 1.27 1.27)
+				)
+				(hide yes)
+			)
+		)
 		(pin "1"
 		)
@@
 			)
 		)
+		(property "Vendor" "digikey:490-1451-1-ND"
+			(at 148.59 54.61 0)
+			(effects
+				(font
+					(size 1.27 1.27)
+				)
+				(hide yes)
+			)
+		)
 		(pin "2"
 		)
@@
 			)
 		)
+		(property "Vendor" "digikey:311-49.9HRCT-ND"
+			(at 0 0 0)
+			(effects
+				(font
+					(size 1.27 1.27)
+				)
+				(hide yes)
+			)
+		)
 		(pin "1"
 		)
@@
 			(effects
 				(font
+					(size 1.27 1.27)
+				)
+				(hide yes)
+			)
+		)
+		(property "Vendor" "digikey:311-49.9HRCT-ND"
+			(at 139.7 190.5 0)
+			(effects
+				(font

Commit message: update value
Parts:
- C1201, C1205, C1207, C1210, C1212: value C -> 0.1UF
- C1202, C1203, C1208: value C -> 1000PF
- C1204, C1206, C1209, C1211: value C -> 10UF
- R1201, R1202: value R -> 49.9
- R1203: value R -> 1K
- R1204: value R -> 287
- R1205: value R -> 10K
Changed lines of the file:
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@@
 			)
 		)
-		(property "Value" "C"
+		(property "Value" "10UF"
 			(at 69.85 49.5299 0)
 			(effects
@@
 			)
 		)
-		(property "Value" "R"
+		(property "Value" "10K"
 			(at 247.65 118.1099 0)
 			(effects
@@
 			)
 		)
-		(property "Value" "C"
+		(property "Value" "1000PF"
 			(at 46.99 74.93 90)
 			(effects
@@
 			)
 		)
-		(property "Value" "C"
+		(property "Value" "1000PF"
 			(at 80.01 95.2499 0)
 			(effects
@@
 			)
 		)
-		(property "Value" "R"
+		(property "Value" "287"
 			(at 77.47 109.2199 0)
 			(effects
@@
 			)
 		)
-		(property "Value" "C"
+		(property "Value" "10UF"
 			(at 54.61 49.5299 0)
 			(effects
@@
 			)
 		)
-		(property "Value" "C"
+		(property "Value" "0.1UF"
 			(at 48.26 49.5299 0)
 			(effects
@@
 			)
 		)
-		(property "Value" "R"
+		(property "Value" "1K"
 			(at 82.55 74.9299 0)
 			(effects
@@
 			)
 		)
-		(property "Value" "C"
+		(property "Value" "0.1UF"
 			(at 256.54 115.5699 0)
 			(effects
@@
 			)
 		)
-		(property "Value" "C"
+		(property "Value" "0.1UF"
 			(at 77.47 49.5299 0)
 			(effects
@@
 			)
 		)
-		(property "Value" "C"
+		(property "Value" "0.1UF"
 			(at 99.06 49.5299 0)
 			(effects
@@
 			)
 		)
-		(property "Value" "C"
+		(property "Value" "10UF"
 			(at 105.41 49.5299 0)
 			(effects
@@
 			)
 		)
-		(property "Value" "C"
+		(property "Value" "0.1UF"
 			(at 63.5 49.5299 0)
 			(effects
@@
 			)
 		)
-		(property "Value" "C"
+		(property "Value" "10UF"
 			(at 91.44 49.5299 0)
 			(effects
@@
 			)
 		)
-		(property "Value" "C"
+		(property "Value" "1000PF"
 			(at 46.99 96.52 90)
 			(effects
@@
 			)
 		)
-		(property "Value" "R"
+		(property "Value" "49.9"
 			(at 67.31 87.6299 0)
 			(effects
@@
 			)
 		)
-		(property "Value" "R"
+		(property "Value" "49.9"
 			(at 67.31 96.5199 0)
 			(effects

Commit message: lots small updates
Parts:
- J1201, J1202: footprint 001_download:CONN_142-0701-201_CIN -> CONN_142-0701-201_CIN; symbol 001_symbol:142-0701-201 -> 001_symbol:142-0701-201_GH
Connections:
- net GND: now also J1201.2, J1201.3, J1201.4, J1201.5, J1202.2, J1202.3, J1202.4, J1202.5
Changed lines of the file:
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@@
 	)
 	(junction
+		(at 260.35 96.52)
+		(diameter 0)
+		(color 0 0 0 0)
+	)
+	(junction
 		(at 50.8 39.37)
 		(diameter 0)
@@
 	)
 	(junction
+		(at 260.35 76.2)
+		(diameter 0)
+		(color 0 0 0 0)
+	)
+	(junction
 		(at 80.01 31.75)
 		(diameter 0)
@@
 	(wire
 		(pts
-			(xy 248.92 96.52) (xy 248.92 95.25)
+			(xy 265.43 96.52) (xy 265.43 93.98)
 		)
 		(stroke
@@
 	(wire
 		(pts
-			(xy 245.11 76.2) (xy 248.92 76.2)
+			(xy 245.11 76.2) (xy 260.35 76.2)
 		)
 		(stroke
@@
 	(wire
 		(pts
+			(xy 260.35 76.2) (xy 265.43 76.2)
+		)
+		(stroke
+			(width 0)
+			(type default)
+		)
+	)
+	(wire
+		(pts
 			(xy 80.01 104.14) (xy 80.01 90.17)
 		)
@@
 		)
 	)
+	(wire
+		(pts
+			(xy 260.35 73.66) (xy 260.35 76.2)
+		)
+		(stroke
+			(width 0)
+			(type default)
+		)
+	)
 	(bus
 		(pts
@@
 	(wire
 		(pts
+			(xy 260.35 96.52) (xy 265.43 96.52)
+		)
+		(stroke
+			(width 0)
+			(type default)
+		)
+	)
+	(wire
+		(pts
 			(xy 124.46 119.38) (xy 151.13 119.38)
 		)
@@
 	(wire
 		(pts
-			(xy 248.92 76.2) (xy 248.92 77.47)
-		)
-		(stroke
-			(width 0)
-			(type default)
-		)
-	)
-	(wire
-		(pts
 			(xy 69.85 90.17) (xy 69.85 91.44)
 		)
@@
 	(wire
 		(pts
+			(xy 260.35 96.52) (xy 260.35 99.06)
+		)
+		(stroke
+			(width 0)
+			(type default)
+		)
+	)
+	(wire
+		(pts
 			(xy 201.93 127) (xy 208.28 127)
 		)
@@
 	(wire
 		(pts
-			(xy 245.11 96.52) (xy 248.92 96.52)
+			(xy 245.11 96.52) (xy 260.35 96.52)
 		)
 		(stroke
@@
 	(symbol
 		(lib_id "power:GND")
-		(at 248.92 95.25 0)
+		(at 265.43 93.98 0)
 		(mirror x)
 		(unit 1)
@@
 		(fields_autoplaced yes)
 		(property "Reference" "#PWR01214"
-			(at 248.92 88.9 0)
+			(at 265.43 87.63 0)
 			(effects
 				(font
@@
 		)
 		(property "Value" "GND"
-			(at 248.92 90.17 0)
+			(at 265.43 88.9 0)
 			(effects
 				(font
@@
 		)
 		(property "Footprint" ""
-			(at 248.92 95.25 0)
+			(at 265.43 93.98 0)
 			(effects
 				(font
@@
 		)
 		(property "Datasheet" ""
-			(at 248.92 95.25 0)
+			(at 265.43 93.98 0)
 			(effects
 				(font
@@
 		)
 		(property "Description" "Power symbol creates a global label with name \"GND\" , ground"
-			(at 248.92 95.25 0)
+			(at 265.43 93.98 0)
 			(effects
 				(font
@@
 	(symbol
 		(lib_id "power:GND")
-		(at 248.92 77.47 0)
+		(at 265.43 76.2 0)
 		(unit 1)
 		(exclude_from_sim no)
@@
 		(fields_autoplaced yes)
 		(property "Reference" "#PWR01213"
-			(at 248.92 83.82 0)
+			(at 265.43 82.55 0)
 			(effects
 				(font
@@
 		)
 		(property "Value" "GND"
-			(at 248.92 82.55 0)
+			(at 265.43 81.28 0)
 			(effects
 				(font
@@
 		)
 		(property "Footprint" ""
-			(at 248.92 77.47 0)
+			(at 265.43 76.2 0)
 			(effects
 				(font
@@
 		)
 		(property "Datasheet" ""
-			(at 248.92 77.47 0)
+			(at 265.43 76.2 0)
 			(effects
 				(font
@@
 		)
 		(property "Description" "Power symbol creates a global label with name \"GND\" , ground"
-			(at 248.92 77.47 0)
+			(at 265.43 76.2 0)
 			(effects
 				(font
@@
 	)
 	(symbol
-		(lib_id "001_symbol:142-0701-201")
+		(lib_id "001_symbol:142-0701-201_GH")
 		(at 245.11 73.66 0)
 		(unit 1)
@@
 		(fields_autoplaced yes)
 		(property "Reference" "J1201"
-			(at 259.08 72.3899 0)
+			(at 254 66.04 0)
 			(effects
 				(font
 					(size 1.524 1.524)
 				)
-				(justify left)
 			)
 		)
 		(property "Value" "142-0701-201"
-			(at 259.08 74.9299 0)
+			(at 254 68.58 0)
 			(effects
 				(font
 					(size 1.524 1.524)
 				)
-				(justify left)
 			)
 		)
-		(property "Footprint" "001_download:CONN_142-0701-201_CIN"
+		(property "Footprint" "CONN_142-0701-201_CIN"
 			(at 245.11 73.66 0)
 			(effects
@@
 		(pin "1"
 		)
+		(pin "2"
+		)
+		(pin "3"
+		)
+		(pin "4"
+		)
+		(pin "5"
+		)
 		(instances
 			(project "kdigitizer"
@@
 	)
 	(symbol
-		(lib_id "001_symbol:142-0701-201")
+		(lib_id "001_symbol:142-0701-201_GH")
 		(at 245.11 99.06 0)
 		(mirror x)
@@
 		(fields_autoplaced yes)
 		(property "Reference" "J1202"
-			(at 259.08 100.3301 0)
+			(at 254 91.44 0)
 			(effects
 				(font
 					(size 1.524 1.524)
 				)
-				(justify left)
 			)
 		)
 		(property "Value" "142-0701-201"
-			(at 259.08 97.7901 0)
+			(at 254 93.98 0)
 			(effects
 				(font
 					(size 1.524 1.524)
 				)
-				(justify left)
 			)
 		)
-		(property "Footprint" "001_download:CONN_142-0701-201_CIN"
+		(property "Footprint" "CONN_142-0701-201_CIN"
 			(at 245.11 99.06 0)
 			(effects
@@
 		(pin "1"
 		)
+		(pin "3"
+		)
+		(pin "2"
+		)
+		(pin "4"
+		)
+		(pin "5"
+		)
 		(instances
