File: at24c32d.kicad_sch (KiCad schematic)
At the start: 10 parts, among them J1901 961102-6404-AR, U1901 AT24C64D-SSHM-T

Commit message: fields
Parts:
- C1901, R1901, R1902, R1903, R1904, R1905, TP30, TP31: gfootprint 0603 -> (none)
- J1901: AVAILABILITY In Stock -> (none); MF 3M -> (none); MP 961102-6404-AR -> (none); PACKAGE None -> (none); PRICE None -> (none); PURCHASE-URL https://pricing.snapeda.com/search/part/961102-6404-AR/?ref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 -> (none)
Changed lines of the file:
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@@
-			)
-		)
-		(property "gfootprint" "0603"
-			(at 386.08 0 0)
-			(effects
-				(font
-					(size 1.27 1.27)
-				)
-				(hide yes)
 			)
 		)
@@
 			)
 		)
-		(property "gfootprint" "0603"
-			(at 408.94 26.67 0)
-			(effects
-				(font
-					(size 1.27 1.27)
-				)
-				(hide yes)
-			)
-		)
 		(pin "1"
 		)
@@
 			)
 		)
-		(property "gfootprint" "0603"
-			(at 0 137.16 0)
-			(effects
-				(font
-					(size 1.27 1.27)
-				)
-				(hide yes)
-			)
-		)
 		(pin "2"
 		)
@@
 			)
 		)
-		(property "gfootprint" "0603"
-			(at 467.36 0 0)
-			(effects
-				(font
-					(size 1.27 1.27)
-				)
-				(hide yes)
-			)
-		)
 		(pin "2"
 		)
@@
 			)
 		)
-		(property "MF" "3M"
-			(at 200.66 78.74 0)
-			(effects
-				(font
-					(size 1.27 1.27)
-				)
-				(justify bottom)
-				(hide yes)
-			)
-		)
-		(property "PACKAGE" "None"
-			(at 200.66 78.74 0)
-			(effects
-				(font
-					(size 1.27 1.27)
-				)
-				(justify bottom)
-				(hide yes)
-			)
-		)
-		(property "PRICE" "None"
-			(at 200.66 78.74 0)
-			(effects
-				(font
-					(size 1.27 1.27)
-				)
-				(justify bottom)
-				(hide yes)
-			)
-		)
-		(property "MP" "961102-6404-AR"
-			(at 200.66 78.74 0)
-			(effects
-				(font
-					(size 1.27 1.27)
-				)
-				(justify bottom)
-				(hide yes)
-			)
-		)
-		(property "AVAILABILITY" "In Stock"
-			(at 200.66 78.74 0)
-			(effects
-				(font
-					(size 1.27 1.27)
-				)
-				(justify bottom)
-				(hide yes)
-			)
-		)
-		(property "PURCHASE-URL" "https://pricing.snapeda.com/search/part/961102-6404-AR/?ref=eda"
-			(at 200.66 78.74 0)
-			(effects
-				(font
-					(size 1.27 1.27)
-				)
-				(justify bottom)
-				(hide yes)
-			)
-		)
 		(pin "2"
 		)
@@
 			)
 		)
-		(property "gfootprint" "0603"
-			(at 201.93 201.93 0)
-			(effects
-				(font
-					(size 1.27 1.27)
-				)
-				(hide yes)
-			)
-		)
 		(pin "2"
 		)
@@
 		(property "Description" "Resistor"
 			(at 227.33 74.93 0)
-			(effects
-				(font
-					(size 1.27 1.27)
-				)
-				(hide yes)
-			)
-		)
-		(property "gfootprint" "0603"
-			(at 454.66 0 0)
 			(effects
 				(font
@@
 			)
 		)
-		(property "gfootprint" "0603"
-			(at 204.47 -41.91 0)
-			(effects
-				(font
-					(size 1.27 1.27)
-				)
-				(hide yes)
-			)
-		)
 		(pin "2"
 		)
@@
 			(effects
 				(font
-					(size 1.27 1.27)
-				)
-				(hide yes)
-			)
-		)
-		(property "gfootprint" "0603"
-			(at 151.13 -123.19 0)
-			(effects
-				(font

Commit message: vendor info
Parts:
- C1901: Vendor (none) -> digikey:490-3897-1-ND
- J1901: Vendor (none) -> digikey:3M9447-ND
- R1901, R1902: Vendor (none) -> digikey:P0.0GCT-ND
- R1903: Vendor (none) -> digikey:311-11.5KHRCT-ND
- R1904, R1905: Vendor (none) -> digikey:311-4.75KHRCT-ND
- U1901: Vendor (none) -> digikey:AT24C64D-SSHM-TCT-ND
Changed lines of the file:
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@@
+			)
+		)
+		(property "Vendor" "digikey:311-11.5KHRCT-ND"
+			(at 386.08 0 0)
+			(effects
+				(font
+					(size 1.27 1.27)
+				)
+				(hide yes)
 			)
 		)
@@
 			)
 		)
+		(property "Vendor" "digikey:490-3897-1-ND"
+			(at 0 137.16 0)
+			(effects
+				(font
+					(size 1.27 1.27)
+				)
+				(hide yes)
+			)
+		)
 		(pin "2"
 		)
@@
 			)
 		)
+		(property "Vendor" "digikey:AT24C64D-SSHM-TCT-ND"
+			(at 0 157.48 0)
+			(effects
+				(font
+					(size 1.27 1.27)
+				)
+				(hide yes)
+			)
+		)
 		(pin "8"
 		)
@@
 			)
 		)
+		(property "Vendor" "digikey:311-4.75KHRCT-ND"
+			(at 467.36 0 0)
+			(effects
+				(font
+					(size 1.27 1.27)
+				)
+				(hide yes)
+			)
+		)
 		(pin "2"
 		)
@@
 			)
 		)
+		(property "Vendor" "digikey:3M9447-ND"
+			(at 0 157.48 0)
+			(effects
+				(font
+					(size 1.27 1.27)
+				)
+				(hide yes)
+			)
+		)
 		(pin "2"
 		)
@@
 			)
 		)
+		(property "Vendor" "digikey:P0.0GCT-ND"
+			(at 201.93 201.93 0)
+			(effects
+				(font
+					(size 1.27 1.27)
+				)
+				(hide yes)
+			)
+		)
 		(pin "2"
 		)
@@
 		(property "Description" "Resistor"
 			(at 227.33 74.93 0)
+			(effects
+				(font
+					(size 1.27 1.27)
+				)
+				(hide yes)
+			)
+		)
+		(property "Vendor" "digikey:311-4.75KHRCT-ND"
+			(at 454.66 0 0)
 			(effects
 				(font
@@
 			(effects
 				(font
+					(size 1.27 1.27)
+				)
+				(hide yes)
+			)
+		)
+		(property "Vendor" "digikey:P0.0GCT-ND"
+			(at 204.47 -41.91 0)
+			(effects
+				(font

Commit message: update value
Parts:
- C1901: value C -> 1UF
- R1901, R1902: value R -> 0
- R1903: value R -> 11.5K
- R1904, R1905: value R -> 4.75K
Changed lines of the file:
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@@
 			)
 		)
-		(property "Value" "R"
+		(property "Value" "11.5K"
 			(at 195.58 105.4099 0)
 			(effects
@@
 			)
 		)
-		(property "Value" "C"
+		(property "Value" "1UF"
 			(at 217.17 69.8499 0)
 			(effects
@@
 			)
 		)
-		(property "Value" "R"
+		(property "Value" "4.75K"
 			(at 236.22 76.1999 0)
 			(effects
@@
 			)
 		)
-		(property "Value" "R"
+		(property "Value" "0"
 			(at 123.19 74.93 90)
 			(effects
@@
 			)
 		)
-		(property "Value" "R"
+		(property "Value" "4.75K"
 			(at 229.87 76.1999 0)
 			(effects
@@
 			)
 		)
-		(property "Value" "R"
+		(property "Value" "0"
 			(at 123.19 85.09 90)
 			(effects

Commit message: lots small updates
Parts:
- TP30, TP31: now left out of the parts list
- U1901: footprint 001_download:8S1_ATM -> 001_download:8S1_ATM_GH
Changed lines of the file:
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@@
 		(unit 1)
 		(exclude_from_sim no)
-		(in_bom yes)
+		(in_bom no)
 		(on_board yes)
 		(dnp no)
@@
 			)
 		)
-		(property "Footprint" "001_download:8S1_ATM"
+		(property "Footprint" "001_download:8S1_ATM_GH"
 			(at 129.54 78.74 0)
 			(effects
@@
 		(unit 1)
 		(exclude_from_sim no)
-		(in_bom yes)
-		(on_board yes)
-		(dnp no)
+		(in_bom no)
+		(on_board yes)
+		(dnp no)
