File: fmc_misc.kicad_sch (KiCad schematic)
At the start: 14 parts, among them J1501 10029449-111RLF, J1502 Conn_02x07_Odd_Even, J1503 Conn_02x07_Odd_Even, Q1501 FDN335N, Q1502 FDN335N

Commit message: fields
Parts:
- Q1501, Q1502: Availability In Stock -> (none); Check_prices https://www.snapeda.com/parts/FDN335N/Onsemi/view-part/?ref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 -> (none); Description_1 N-Channel 20 V 0.07 Ohm 2.5 V Specified PowerTrench Mosfet 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 -> (none); MF ON Semiconductor -> (none); MP FDN335N -> (none); Package TO-236-3 ON -> (none); Price None -> (none); SnapEDA_Link https://www.snapeda.com/parts/FDN335N/Onsemi/view-part/?ref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 -> (none)
- R1501, R1502, R1503, R1504, R1505, R1506, R1507: gfootprint 0603 -> (none)

Commit message: vendor info
Parts:
- D1501, D1502: Vendor (none) -> digikey:754-1116-1-ND
- J1501: Vendor (none) -> digikey:609-4614-1-ND
- J1502, J1503: Vendor (none) -> digikey:S5560-ND
- Q1501, Q1502: Vendor (none) -> digikey:FDN335NCT-ND
- R1501, R1502, R1503, R1504: Vendor (none) -> digikey:P0.0GCT-ND
- R1505, R1506: Vendor (none) -> digikey:RR08P200DCT-ND
Changed lines of the file:
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@@
+			)
+		)
+		(property "Vendor" "digikey:P0.0GCT-ND"
+			(at 0 195.58 0)
+			(effects
+				(font
+					(size 1.27 1.27)
+				)
+				(hide yes)
 			)
 		)
@@
 			)
 		)
+		(property "Vendor" "digikey:P0.0GCT-ND"
+			(at 119.38 195.58 0)
+			(effects
+				(font
+					(size 1.27 1.27)
+				)
+				(hide yes)
+			)
+		)
 		(pin "1"
 		)
@@
 			)
 		)
+		(property "Vendor" "digikey:FDN335NCT-ND"
+			(at 0 134.62 0)
+			(effects
+				(font
+					(size 1.27 1.27)
+				)
+				(hide yes)
+			)
+		)
 		(pin "3"
 		)
@@
 			)
 		)
+		(property "Vendor" "digikey:609-4614-1-ND"
+			(at 0 83.82 0)
+			(effects
+				(font
+					(size 1.27 1.27)
+				)
+				(hide yes)
+			)
+		)
 		(pin "18"
 		)
@@
 			)
 		)
+		(property "Vendor" "digikey:754-1116-1-ND"
+			(at 142.24 142.24 0)
+			(effects
+				(font
+					(size 1.27 1.27)
+				)
+				(hide yes)
+			)
+		)
 		(pin "2"
 		)
@@
 			)
 		)
+		(property "Vendor" "digikey:P0.0GCT-ND"
+			(at 129.54 58.42 0)
+			(effects
+				(font
+					(size 1.27 1.27)
+				)
+				(hide yes)
+			)
+		)
 		(pin "1"
 		)
@@
 			)
 		)
+		(property "Vendor" "digikey:S5560-ND"
+			(at 0 0 0)
+			(effects
+				(font
+					(size 1.27 1.27)
+				)
+				(hide yes)
+			)
+		)
 		(pin "7"
 		)
@@
 			)
 		)
+		(property "Vendor" "digikey:P0.0GCT-ND"
+			(at 140.97 46.99 0)
+			(effects
+				(font
+					(size 1.27 1.27)
+				)
+				(hide yes)
+			)
+		)
 		(pin "1"
 		)
@@
 			)
 		)
+		(property "Vendor" "digikey:754-1116-1-ND"
+			(at 166.37 166.37 0)
+			(effects
+				(font
+					(size 1.27 1.27)
+				)
+				(hide yes)
+			)
+		)
 		(pin "2"
 		)
@@
 			)
 		)
+		(property "Vendor" "digikey:RR08P200DCT-ND"
+			(at 215.9 0 0)
+			(effects
+				(font
+					(size 1.27 1.27)
+				)
+				(hide yes)
+			)
+		)
 		(pin "1"
 		)
@@
 			)
 		)
+		(property "Vendor" "digikey:S5560-ND"
+			(at 0 0 0)
+			(effects
+				(font
+					(size 1.27 1.27)
+				)
+				(hide yes)
+			)
+		)
 		(pin "7"
 		)
@@
 			)
 		)
+		(property "Vendor" "digikey:RR08P200DCT-ND"
+			(at 167.64 0 0)
+			(effects
+				(font
+					(size 1.27 1.27)
+				)
+				(hide yes)
+			)
+		)
 		(pin "1"
 		)
@@
 			(effects
 				(font
+					(size 1.27 1.27)
+				)
+				(hide yes)
+			)
+		)
+		(property "Vendor" "digikey:FDN335NCT-ND"
+			(at 215.9 134.62 0)
+			(effects
+				(font

Commit message: update value
Parts:
- D1501, D1502: value D -> APT1608CGCK
- J1502, J1503: value Conn_02x07_Odd_Even -> PPPC072LJBN-RC
- R1501, R1502, R1503, R1504: value R -> 0
- R1505, R1506: value R -> 200
Changed lines of the file:
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@@
 			)
 		)
-		(property "Value" "R"
+		(property "Value" "0"
 			(at 67.31 97.79 90)
 			(effects
@@
 			)
 		)
-		(property "Value" "R"
+		(property "Value" "0"
 			(at 55.88 97.79 90)
 			(effects
@@
 			)
 		)
-		(property "Value" "D"
+		(property "Value" "APT1608CGCK"
 			(at 80.01 58.42 0)
 			(effects
@@
 			)
 		)
-		(property "Value" "R"
+		(property "Value" "0"
 			(at 35.56 97.79 90)
 			(effects
@@
 			)
 		)
-		(property "Value" "Conn_02x07_Odd_Even"
+		(property "Value" "PPPC072LJBN-RC"
 			(at 160.02 166.37 0)
 			(effects
@@
 			)
 		)
-		(property "Value" "R"
+		(property "Value" "0"
 			(at 46.99 97.79 90)
 			(effects
@@
 			)
 		)
-		(property "Value" "D"
+		(property "Value" "APT1608CGCK"
 			(at 104.14 58.42 0)
 			(effects
@@
 			)
 		)
-		(property "Value" "R"
+		(property "Value" "200"
 			(at 110.49 52.0699 0)
 			(effects
@@
 			)
 		)
-		(property "Value" "Conn_02x07_Odd_Even"
+		(property "Value" "PPPC072LJBN-RC"
 			(at 158.75 134.62 0)
 			(effects
@@
 			)
 		)
-		(property "Value" "R"
+		(property "Value" "200"
 			(at 86.36 52.0699 0)
 			(effects

Commit message: lots small updates
Parts:
- J1501: footprint 001_download:CONN_10029449111_AMP -> CONN_10029449111_AMP; symbol 001_symbol:10029449-111RLF -> 001_symbol:10029449-111RLF_GH
- R1507: value R -> DNP
Connections:
- no-connect marks 1 -> 5
Changed lines of the file:
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@@
+	)
+	(no_connect
+		(at 165.1 87.63)
+	)
+	(no_connect
+		(at 165.1 85.09)
+	)
+	(no_connect
+		(at 165.1 82.55)
+	)
+	(no_connect
+		(at 165.1 80.01)
 	)
 	(no_connect
@@
 	)
 	(symbol
-		(lib_id "001_symbol:10029449-111RLF")
+		(lib_id "001_symbol:10029449-111RLF_GH")
 		(at 149.86 41.91 0)
 		(unit 1)
@@
 			)
 		)
-		(property "Footprint" "001_download:CONN_10029449111_AMP"
+		(property "Footprint" "CONN_10029449111_AMP"
 			(at 149.86 41.91 0)
 			(effects
@@
 		)
 		(pin "15"
+		)
+		(pin "21"
+		)
+		(pin "20"
+		)
+		(pin "23"
+		)
+		(pin "22"
 		)
 		(instances
@@
 			)
 		)
-		(property "Value" "R"
+		(property "Value" "DNP"
 			(at 121.92 80.01 90)
 			(effects
