File: kdigitizer.kicad_sch (KiCad schematic)
At the start: 7 parts

Commit message: fields
Parts:
- H102, H103, H105: gfootprint 0603 -> (none)
- H104: gfootprint 0402 -> (none)
- H107: gfootprint 1206 -> (none)
Changed lines of the file:
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@@
-			)
-		)
-		(property "gfootprint" "0603"
-			(at -15.24 283.21 0)
-			(effects
-				(font
-					(size 1.27 1.27)
-				)
-				(hide yes)
 			)
 		)
@@
 			)
 		)
-		(property "gfootprint" "1206"
-			(at -15.24 283.21 0)
-			(effects
-				(font
-					(size 1.27 1.27)
-				)
-				(hide yes)
-			)
-		)
 		(instances
 			(project "kdigitizer"
@@
 			)
 		)
-		(property "gfootprint" "0603"
-			(at -15.24 283.21 0)
-			(effects
-				(font
-					(size 1.27 1.27)
-				)
-				(hide yes)
-			)
-		)
 		(instances
 			(project "kdigitizer"
@@
 			)
 		)
-		(property "gfootprint" "0603"
-			(at -15.24 283.21 0)
-			(effects
-				(font
-					(size 1.27 1.27)
-				)
-				(hide yes)
-			)
-		)
 		(instances
 			(project "kdigitizer"
@@
 			(effects
 				(font
-					(size 1.27 1.27)
-				)
-				(hide yes)
-			)
-		)
-		(property "gfootprint" "0402"
-			(at -15.24 283.21 0)
-			(effects
-				(font

Commit message: lots small updates
Parts:
- H101, H102, H103, H104, H105, H106, H107: symbol Mechanical:MountingHole -> 001_symbol:MountingHole_GH
Connections:
- no-connect marks 0 -> 7
Changed lines of the file:
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@@
 		(color 0 0 0 0)
+	)
+	(no_connect
+		(at 69.85 144.78)
+	)
+	(no_connect
+		(at 62.23 144.78)
+	)
+	(no_connect
+		(at 85.09 144.78)
+	)
+	(no_connect
+		(at 54.61 144.78)
+	)
+	(no_connect
+		(at 38.1 144.78)
+	)
+	(no_connect
+		(at 77.47 144.78)
+	)
+	(no_connect
+		(at 45.72 144.78)
 	)
 	(bus_entry
@@
 	)
 	(symbol
-		(lib_id "Mechanical:MountingHole")
+		(lib_id "001_symbol:MountingHole_GH")
 		(at 45.72 142.24 0)
 		(unit 1)
@@
 			)
 		)
+		(pin "1"
+		)
 		(instances
 			(project "kdigitizer"
@@
 	)
 	(symbol
-		(lib_id "Mechanical:MountingHole")
+		(lib_id "001_symbol:MountingHole_GH")
 		(at 38.1 142.24 0)
 		(unit 1)
@@
 			)
 		)
+		(pin "1"
+		)
 		(instances
 			(project "kdigitizer"
@@
 	)
 	(symbol
-		(lib_id "Mechanical:MountingHole")
+		(lib_id "001_symbol:MountingHole_GH")
 		(at 85.09 142.24 0)
 		(unit 1)
@@
 			)
 		)
+		(pin "1"
+		)
 		(instances
 			(project "kdigitizer"
@@
 	)
 	(symbol
-		(lib_id "Mechanical:MountingHole")
+		(lib_id "001_symbol:MountingHole_GH")
 		(at 69.85 142.24 0)
 		(unit 1)
@@
 			)
 		)
+		(pin "1"
+		)
 		(instances
 			(project "kdigitizer"
@@
 	)
 	(symbol
-		(lib_id "Mechanical:MountingHole")
+		(lib_id "001_symbol:MountingHole_GH")
 		(at 77.47 142.24 0)
 		(unit 1)
@@
 			)
 		)
+		(pin "1"
+		)
 		(instances
 			(project "kdigitizer"
@@
 	)
 	(symbol
-		(lib_id "Mechanical:MountingHole")
+		(lib_id "001_symbol:MountingHole_GH")
 		(at 54.61 142.24 0)
 		(unit 1)
@@
 			)
 		)
+		(pin "1"
+		)
 		(instances
 			(project "kdigitizer"
@@
 	)
 	(symbol
-		(lib_id "Mechanical:MountingHole")
+		(lib_id "001_symbol:MountingHole_GH")
 		(at 62.23 142.24 0)
 		(unit 1)
@@
 			)
 		)
+		(pin "1"
+		)
 		(instances
