File: kx023.kicad_sch (KiCad schematic)
At the start: 5 parts, among them U2001 KX023-1025

Commit message: fields
Parts:
- R2001, R2002, TP28, TP29: gfootprint 0603 -> (none)
Changed lines of the file:
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@@
-			)
-		)
-		(property "gfootprint" "0603"
-			(at 248.92 0 0)
-			(effects
-				(font
-					(size 1.27 1.27)
-				)
-				(hide yes)
 			)
 		)
@@
 			)
 		)
-		(property "gfootprint" "0603"
-			(at 238.76 0 0)
-			(effects
-				(font
-					(size 1.27 1.27)
-				)
-				(hide yes)
-			)
-		)
 		(pin "1"
 		)
@@
 			)
 		)
-		(property "gfootprint" "0603"
-			(at 316.23 24.13 0)
-			(effects
-				(font
-					(size 1.27 1.27)
-				)
-				(hide yes)
-			)
-		)
 		(pin "1"
 		)
@@
 			(effects
 				(font
-					(size 1.27 1.27)
-				)
-				(hide yes)
-			)
-		)
-		(property "gfootprint" "0603"
-			(at -97.79 140.97 0)
-			(effects
-				(font

Commit message: vendor info
Parts:
- R2001, R2002: Vendor (none) -> digikey:311-4.75KHRCT-ND
- U2001: Vendor (none) -> digikey:1191-1039-1-ND
Changed lines of the file:
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@@
+			)
+		)
+		(property "Vendor" "digikey:311-4.75KHRCT-ND"
+			(at 248.92 0 0)
+			(effects
+				(font
+					(size 1.27 1.27)
+				)
+				(hide yes)
 			)
 		)
@@
 			)
 		)
+		(property "Vendor" "digikey:311-4.75KHRCT-ND"
+			(at 238.76 0 0)
+			(effects
+				(font
+					(size 1.27 1.27)
+				)
+				(hide yes)
+			)
+		)
 		(pin "1"
 		)
@@
 			(effects
 				(font
+					(size 1.27 1.27)
+				)
+				(hide yes)
+			)
+		)
+		(property "Vendor" "digikey:1191-1039-1-ND"
+			(at 0 165.1 0)
+			(effects
+				(font

Commit message: update value
Parts:
- R2001, R2002: value R -> 4.75K
- U2001: value KX023-1025 -> KX023-1025-FR
Changed lines of the file:
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@@
 			)
 		)
-		(property "Value" "R"
+		(property "Value" "4.75K"
 			(at 127 74.9299 0)
 			(effects
@@
 			)
 		)
-		(property "Value" "R"
+		(property "Value" "4.75K"
 			(at 121.92 74.9299 0)
 			(effects
@@
 			)
 		)
-		(property "Value" "KX023-1025"
+		(property "Value" "KX023-1025-FR"
 			(at 144.4341 69.85 0)
 			(effects

Commit message: lots small updates
Parts:
- TP28, TP29: now left out of the parts list
Changed lines of the file:
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@@
 		(unit 1)
 		(exclude_from_sim no)
-		(in_bom yes)
+		(in_bom no)
 		(on_board yes)
 		(dnp no)
@@
 		(unit 1)
 		(exclude_from_sim no)
-		(in_bom yes)
+		(in_bom no)
 		(on_board yes)
 		(dnp no)
