File: lmk01801.kicad_sch (KiCad schematic)
At the start: 41 parts, among them J1001 142-0701-201, J1002 U.FL-R-SMT10, J1003 U.FL-R-SMT10, J1004 142-0701-201, J1005 U.FL-R-SMT10, T1001 TCM2-43X+, T1002 TCM2-43X+, U1001 TCP-2-33W+, U1002 LMK01801BISQE/NOPB

Commit message: fields
Parts:
- C1001, C1002, C1003, C1004, C1005, C1006, C1007, C1011, C1012, C1013, FB1002, FB1003, FB1004, R1001, R1002, R1003, R1004, R1005, R1006, R1007, R1008, R1009, R1010: gfootprint 0603 -> (none)
- C1008, C1009, C1010, C1014, C1015, C1016, C1017, C1018: gfootprint 0402 -> (none)
- FB1001: gfootprint 0805 -> (none)

Commit message: vendor info
Parts:
- C1001, C1006, C1007, C1011, C1012: Vendor (none) -> digikey:490-1451-1-ND
- C1002, C1003, C1004, C1005: Vendor (none) -> digikey:445-6853-1-ND
- C1008, C1009, C1010, C1014, C1015, C1016, C1017, C1018: Vendor (none) -> digikey:490-1318-1-ND
- C1013: Vendor (none) -> digikey:490-3897-1-ND
- FB1001: Vendor (none) -> digikey:732-1620-1-ND
- FB1002, FB1003, FB1004: Vendor (none) -> digikey:490-1011-1-ND
- J1001, J1004: Vendor (none) -> digikey:J500-ND
- J1002, J1003, J1005: Vendor (none) -> digikey:H9161CT-ND
- R1001: Vendor (none) -> digikey:311-475HRCT-ND
- R1002: Vendor (none) -> digikey:311-100HRCT-ND
- R1003, R1004, R1005, R1006, R1007, R1008, R1009, R1010: Vendor (none) -> digikey:RR08P200DCT-ND
- T1001, T1002: Vendor (none) -> digikey:TCM2-43X+
- U1001: Vendor (none) -> digikey:TCP-2-33W+
- U1002: Vendor (none) -> digikey:296-40276-1-ND

Commit message: update value
Parts:
- C1001, C1006, C1007, C1011, C1012: value C -> 1000PF
- C1002, C1003, C1004, C1005: value C -> 10UF
- C1008, C1009, C1010, C1014, C1015, C1016, C1017, C1018: value C -> 0.1UF
- C1013: value C -> 1UF
- FB1001: value FerriteBead -> 742792040
- FB1002, FB1003, FB1004: value FerriteBead -> BLM18AG121SN1D
- J1002, J1003, J1005: value U.FL-R-SMT10 -> U.FL-R-SMT(10)
- R1001: value R -> 475
- R1002: value R -> 100
- R1003, R1004, R1005, R1006, R1007, R1008, R1009, R1010: value R -> 200
Changed lines of the file:
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@@
 			)
 		)
-		(property "Value" "C"
+		(property "Value" "0.1UF"
 			(at 265.43 48.26 90)
 			(effects
@@
 			)
 		)
-		(property "Value" "C"
+		(property "Value" "0.1UF"
 			(at 116.84 20.32 90)
 			(effects
@@
 			)
 		)
-		(property "Value" "C"
+		(property "Value" "1UF"
 			(at 248.92 114.3 90)
 			(effects
@@
 			)
 		)
-		(property "Value" "U.FL-R-SMT10"
+		(property "Value" "U.FL-R-SMT(10)"
 			(at 135.89 74.93 0)
 			(effects
@@
 			)
 		)
-		(property "Value" "C"
+		(property "Value" "1000PF"
 			(at 97.79 153.67 90)
 			(effects
@@
 			)
 		)
-		(property "Value" "R"
+		(property "Value" "475"
 			(at 67.31 132.08 90)
 			(effects
@@
 			)
 		)
-		(property "Value" "C"
+		(property "Value" "1000PF"
 			(at 176.53 144.78 90)
 			(effects
@@
 			)
 		)
-		(property "Value" "FerriteBead"
+		(property "Value" "BLM18AG121SN1D"
 			(at 55.8292 49.53 90)
 			(effects
@@
 			)
 		)
-		(property "Value" "U.FL-R-SMT10"
+		(property "Value" "U.FL-R-SMT(10)"
 			(at 134.62 114.3 0)
 			(effects
@@
 			)
 		)
-		(property "Value" "U.FL-R-SMT10"
+		(property "Value" "U.FL-R-SMT(10)"
 			(at 267.97 78.74 0)
 			(effects
@@
 			)
 		)
-		(property "Value" "R"
+		(property "Value" "200"
 			(at 116.84 111.76 90)
 			(effects
@@
 			)
 		)
-		(property "Value" "C"
+		(property "Value" "10UF"
 			(at 68.58 68.5799 0)
 			(effects
@@
 			)
 		)
-		(property "Value" "C"
+		(property "Value" "1000PF"
 			(at 39.37 115.5699 0)
 			(effects
@@
 			)
 		)
-		(property "Value" "FerriteBead"
+		(property "Value" "BLM18AG121SN1D"
 			(at 55.8292 39.37 90)
 			(effects
@@
 			)
 		)
-		(property "Value" "C"
+		(property "Value" "0.1UF"
 			(at 270.51 38.1 90)
 			(effects
@@
 			)
 		)
-		(property "Value" "R"
+		(property "Value" "200"
 			(at 121.92 71.12 90)
 			(effects
@@
 			)
 		)
-		(property "Value" "C"
+		(property "Value" "10UF"
 			(at 78.74 68.5799 0)
 			(effects
@@
 			)
 		)
-		(property "Value" "C"
+		(property "Value" "0.1UF"
 			(at 119.38 25.4 90)
 			(effects
@@
 			)
 		)
-		(property "Value" "R"
+		(property "Value" "100"
 			(at 85.09 156.2099 0)
 			(effects
@@
 			)
 		)
-		(property "Value" "R"
+		(property "Value" "200"
 			(at 114.3 66.04 90)
 			(effects
@@
 			)
 		)
-		(property "Value" "R"
+		(property "Value" "200"
 			(at 121.92 114.3 90)
 			(effects
@@
 			)
 		)
-		(property "Value" "FerriteBead"
+		(property "Value" "BLM18AG121SN1D"
 			(at 55.8292 27.94 90)
 			(effects
@@
 			)
 		)
-		(property "Value" "R"
+		(property "Value" "200"
 			(at 261.62 92.71 90)
 			(effects
@@
 			)
 		)
-		(property "Value" "C"
+		(property "Value" "0.1UF"
 			(at 260.35 35.56 90)
 			(effects
@@
 			)
 		)
-		(property "Value" "C"
+		(property "Value" "0.1UF"
 			(at 265.43 121.92 90)
 			(effects
@@
 			)
 		)
-		(property "Value" "R"
+		(property "Value" "200"
 			(at 110.49 63.5 90)
 			(effects
@@
 			)
 		)
-		(property "Value" "C"
+		(property "Value" "0.1UF"
 			(at 264.16 30.48 90)
 			(effects
@@
 			)
 		)
-		(property "Value" "C"
+		(property "Value" "1000PF"
 			(at 176.53 147.32 90)
 			(effects
@@
 			)
 		)
-		(property "Value" "R"
+		(property "Value" "200"
 			(at 259.08 90.17 90)
 			(effects
@@
 			)
 		)
-		(property "Value" "C"
+		(property "Value" "0.1UF"
 			(at 125.73 27.94 90)
 			(effects
@@
 			)
 		)
-		(property "Value" "FerriteBead"
+		(property "Value" "742792040"
 			(at 34.2392 39.37 90)
 			(effects
@@
 			)
 		)
-		(property "Value" "R"
+		(property "Value" "200"
 			(at 125.73 73.66 90)
 			(effects
@@
 			)
 		)
-		(property "Value" "C"
+		(property "Value" "1000PF"
 			(at 97.79 146.05 90)
 			(effects
@@
 			)
 		)
-		(property "Value" "C"
+		(property "Value" "10UF"
 			(at 87.63 68.5799 0)
 			(effects
@@
 			)
 		)
-		(property "Value" "C"
+		(property "Value" "10UF"
 			(at 43.18 55.8799 0)
 			(effects

Commit message: lots small updates
Parts:
- C1017, C1018: footprint Capacitor_SMD:C_0603_1608Metric -> Capacitor_SMD:C_0402_1005Metric
- J1001, J1004: footprint 001_download:CONN_142-0701-201_CIN -> CONN_142-0701-201_CIN; symbol 001_symbol:142-0701-201 -> 001_symbol:142-0701-201_GH
Connections:
- net GND: now also J1001.2, J1001.3, J1001.4, J1001.5, J1004.2, J1004.3, J1004.4, J1004.5
Changed lines of the file:
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@@
 	)
 	(symbol
+		(lib_id "power:GND")
+		(at 20.32 110.49 0)
+		(unit 1)
+		(exclude_from_sim no)
+		(in_bom yes)
+		(on_board yes)
+		(dnp no)
+		(fields_autoplaced yes)
+		(property "Reference" "#PWR01027"
+			(at 20.32 116.84 0)
+			(effects
+				(font
+					(size 1.27 1.27)
+				)
+				(hide yes)
+			)
+		)
+		(property "Value" "GND"
+			(at 20.32 115.57 0)
+			(effects
+				(font
+					(size 1.27 1.27)
+				)
+			)
+		)
+		(property "Footprint" ""
+			(at 20.32 110.49 0)
+			(effects
+				(font
+					(size 1.27 1.27)
+				)
+				(hide yes)
+			)
+		)
+		(property "Datasheet" ""
+			(at 20.32 110.49 0)
+			(effects
+				(font
+					(size 1.27 1.27)
+				)
+				(hide yes)
+			)
+		)
+		(property "Description" "Power symbol creates a global label with name \"GND\" , ground"
+			(at 20.32 110.49 0)
+			(effects
+				(font
+					(size 1.27 1.27)
+				)
+				(hide yes)
+			)
+		)
+		(pin "1"
+		)
+		(instances
+			(project "kdigitizer"
+				(path "/00000000-0000-0000-0000-000000000003/00000000-0000-0000-0000-000000000015"
+					(reference "#PWR01027")
+					(unit 1)
+				)
+			)
+		)
+	)
+	(symbol
 		(lib_id "001_symbol:U.FL-R-SMT10_1")
 		(at 142.24 71.12 0)
@@
 			)
 		)
-		(property "Footprint" "Capacitor_SMD:C_0603_1608Metric"
+		(property "Footprint" "Capacitor_SMD:C_0402_1005Metric"
 			(at 274.32 32.0548 0)
 			(effects
@@
 	)
 	(symbol
-		(lib_id "001_symbol:142-0701-201")
+		(lib_id "001_symbol:142-0701-201_GH")
 		(at 213.36 149.86 0)
 		(mirror x)
@@
 			)
 		)
-		(property "Footprint" "001_download:CONN_142-0701-201_CIN"
+		(property "Footprint" "CONN_142-0701-201_CIN"
 			(at 213.36 149.86 0)
 			(effects
@@
 		(pin "1"
 		)
+		(pin "2"
+		)
+		(pin "3"
+		)
+		(pin "4"
+		)
+		(pin "5"
+		)
 		(instances
 			(project "kdigitizer"
@@
 	)
 	(symbol
+		(lib_id "power:GND")
+		(at 228.6 149.86 0)
+		(mirror y)
+		(unit 1)
+		(exclude_from_sim no)
+		(in_bom yes)
+		(on_board yes)
+		(dnp no)
+		(property "Reference" "#PWR01028"
+			(at 228.6 156.21 0)
+			(effects
+				(font
+					(size 1.27 1.27)
+				)
+				(hide yes)
+			)
+		)
+		(property "Value" "GND"
+			(at 228.6001 153.67 90)
+			(effects
+				(font
+					(size 1.27 1.27)
+				)
+				(justify right)
+			)
+		)
+		(property "Footprint" ""
+			(at 228.6 149.86 0)
+			(effects
+				(font
+					(size 1.27 1.27)
+				)
+				(hide yes)
+			)
+		)
+		(property "Datasheet" ""
+			(at 228.6 149.86 0)
+			(effects
+				(font
+					(size 1.27 1.27)
+				)
+				(hide yes)
+			)
+		)
+		(property "Description" "Power symbol creates a global label with name \"GND\" , ground"
+			(at 228.6 149.86 0)
+			(effects
+				(font
+					(size 1.27 1.27)
+				)
+				(hide yes)
+			)
+		)
+		(pin "1"
+		)
+		(instances
+			(project "kdigitizer"
+				(path "/00000000-0000-0000-0000-000000000003/00000000-0000-0000-0000-000000000015"
+					(reference "#PWR01028")
+					(unit 1)
+				)
+			)
+		)
+	)
+	(symbol
 		(lib_id "Device:FerriteBead")
 		(at 55.88 33.02 90)
@@
 			)
 		)
-		(property "Footprint" "Capacitor_SMD:C_0603_1608Metric"
+		(property "Footprint" "Capacitor_SMD:C_0402_1005Metric"
 			(at 269.24 126.0348 0)
 			(effects
@@
 	)
 	(symbol
-		(lib_id "001_symbol:142-0701-201")
+		(lib_id "001_symbol:142-0701-201_GH")
 		(at 35.56 110.49 180)
 		(unit 1)
@@
 			)
 		)
-		(property "Footprint" "001_download:CONN_142-0701-201_CIN"
+		(property "Footprint" "CONN_142-0701-201_CIN"
 			(at 35.56 110.49 0)
 			(effects
@@
 		(pin "1"
 		)
+		(pin "5"
+		)
+		(pin "2"
+		)
+		(pin "4"
+		)
+		(pin "3"
+		)
 		(instances
