File: se_diff.kicad_sch (KiCad schematic)
At the start: 12 parts

Commit message: fields
Parts:
- C2101, C2102, C2103, C2104, L2101, R2101, R2102, R2103, R2104, R2105, R2106: gfootprint 0603 -> (none)
Changed lines of the file:
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@@
-			)
-		)
-		(property "gfootprint" "0603"
-			(at 300.99 -143.51 0)
-			(effects
-				(font
-					(size 1.27 1.27)
-				)
-				(hide yes)
 			)
 		)
@@
 		(property "Description" "Inductor"
 			(at 217.17 80.01 0)
-			(effects
-				(font
-					(size 1.27 1.27)
-				)
-				(hide yes)
-			)
-		)
-		(property "gfootprint" "0603"
-			(at 0 160.02 0)
 			(effects
 				(font
@@
 			)
 		)
-		(property "gfootprint" "0603"
-			(at 170.18 -12.7 0)
-			(effects
-				(font
-					(size 1.27 1.27)
-				)
-				(hide yes)
-			)
-		)
 		(pin "2"
 		)
@@
 		(property "Description" "Unpolarized capacitor"
 			(at 93.98 76.2 0)
-			(effects
-				(font
-					(size 1.27 1.27)
-				)
-				(hide yes)
-			)
-		)
-		(property "gfootprint" "0603"
-			(at 175.26 170.18 0)
 			(effects
 				(font
@@
 			)
 		)
-		(property "gfootprint" "0603"
-			(at 0 157.48 0)
-			(effects
-				(font
-					(size 1.27 1.27)
-				)
-				(hide yes)
-			)
-		)
 		(pin "2"
 		)
@@
 		(property "Description" "Resistor"
 			(at 185.42 73.66 0)
-			(effects
-				(font
-					(size 1.27 1.27)
-				)
-				(hide yes)
-			)
-		)
-		(property "gfootprint" "0603"
-			(at 269.24 259.08 0)
 			(effects
 				(font
@@
 			)
 		)
-		(property "gfootprint" "0603"
-			(at 259.08 -101.6 0)
-			(effects
-				(font
-					(size 1.27 1.27)
-				)
-				(hide yes)
-			)
-		)
 		(pin "2"
 		)
@@
 			)
 		)
-		(property "gfootprint" "0603"
-			(at 0 157.48 0)
-			(effects
-				(font
-					(size 1.27 1.27)
-				)
-				(hide yes)
-			)
-		)
 		(pin "2"
 		)
@@
 			)
 		)
-		(property "gfootprint" "0603"
-			(at 0 0 0)
-			(effects
-				(font
-					(size 1.27 1.27)
-				)
-				(hide yes)
-			)
-		)
 		(pin "2"
 		)
@@
 			)
 		)
-		(property "gfootprint" "0603"
-			(at 311.15 -153.67 0)
-			(effects
-				(font
-					(size 1.27 1.27)
-				)
-				(hide yes)
-			)
-		)
 		(pin "2"
 		)
@@
 			(effects
 				(font
-					(size 1.27 1.27)
-				)
-				(hide yes)
-			)
-		)
-		(property "gfootprint" "0603"
-			(at 295.91 -114.3 0)
-			(effects
-				(font

Commit message: vendor info
Parts:
- C2101, C2102, C2103: Vendor (none) -> digikey:445-2664-1-ND
- C2104: Vendor (none) -> digikey:1276-2244-1-ND
- R2101, R2102: Vendor (none) -> digikey:P0.0GCT-ND
- R2103, R2104: Vendor (none) -> digikey:RR08P200DCT-ND
- R2105, R2106: Vendor (none) -> digikey:311-4.99HRCT-ND
- XMER2101: Vendor (none) -> digikey:TCM4-19+
Changed lines of the file:
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@@
+			)
+		)
+		(property "Vendor" "digikey:311-4.99HRCT-ND"
+			(at 311.15 -143.51 0)
+			(effects
+				(font
+					(size 1.27 1.27)
+				)
+				(hide yes)
 			)
 		)
@@
 			)
 		)
+		(property "Vendor" "digikey:TCM4-19+"
+			(at 347.98 152.4 0)
+			(effects
+				(font
+					(size 1.27 1.27)
+				)
+				(hide yes)
+			)
+		)
 		(pin "4"
 		)
@@
 			)
 		)
+		(property "Vendor" "digikey:445-2664-1-ND"
+			(at 175.26 -12.7 0)
+			(effects
+				(font
+					(size 1.27 1.27)
+				)
+				(hide yes)
+			)
+		)
 		(pin "2"
 		)
@@
 		(property "Description" "Unpolarized capacitor"
 			(at 93.98 76.2 0)
+			(effects
+				(font
+					(size 1.27 1.27)
+				)
+				(hide yes)
+			)
+		)
+		(property "Vendor" "digikey:445-2664-1-ND"
+			(at 170.18 170.18 0)
 			(effects
 				(font
@@
 			)
 		)
+		(property "Vendor" "digikey:RR08P200DCT-ND"
+			(at 0 157.48 0)
+			(effects
+				(font
+					(size 1.27 1.27)
+				)
+				(hide yes)
+			)
+		)
 		(pin "2"
 		)
@@
 		(property "Description" "Resistor"
 			(at 185.42 73.66 0)
+			(effects
+				(font
+					(size 1.27 1.27)
+				)
+				(hide yes)
+			)
+		)
+		(property "Vendor" "digikey:P0.0GCT-ND"
+			(at 259.08 259.08 0)
 			(effects
 				(font
@@
 			)
 		)
+		(property "Vendor" "digikey:P0.0GCT-ND"
+			(at 269.24 -101.6 0)
+			(effects
+				(font
+					(size 1.27 1.27)
+				)
+				(hide yes)
+			)
+		)
 		(pin "2"
 		)
@@
 			)
 		)
+		(property "Vendor" "digikey:1276-2244-1-ND"
+			(at 0 157.48 0)
+			(effects
+				(font
+					(size 1.27 1.27)
+				)
+				(hide yes)
+			)
+		)
 		(pin "2"
 		)
@@
 			)
 		)
+		(property "Vendor" "digikey:445-2664-1-ND"
+			(at 0 0 0)
+			(effects
+				(font
+					(size 1.27 1.27)
+				)
+				(hide yes)
+			)
+		)
 		(pin "2"
 		)
@@
 			)
 		)
+		(property "Vendor" "digikey:311-4.99HRCT-ND"
+			(at 300.99 -153.67 0)
+			(effects
+				(font
+					(size 1.27 1.27)
+				)
+				(hide yes)
+			)
+		)
 		(pin "2"
 		)
@@
 			(effects
 				(font
+					(size 1.27 1.27)
+				)
+				(hide yes)
+			)
+		)
+		(property "Vendor" "digikey:RR08P200DCT-ND"
+			(at 295.91 -113.03 0)
+			(effects
+				(font

Commit message: update value
Parts:
- C2101, C2102, C2103: value C -> 10000PF
- C2104: value C -> 25PF
- R2101, R2102: value R -> 0
- R2103, R2104: value R -> 200
- R2105, R2106: value R -> 4.99
Changed lines of the file:
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@@
 			)
 		)
-		(property "Value" "R"
+		(property "Value" "4.99"
 			(at 227.33 87.63 90)
 			(effects
@@
 			)
 		)
-		(property "Value" "C"
+		(property "Value" "10000PF"
 			(at 93.98 86.36 90)
 			(effects
@@
 			)
 		)
-		(property "Value" "C"
+		(property "Value" "10000PF"
 			(at 93.98 71.12 90)
 			(effects
@@
 			)
 		)
-		(property "Value" "R"
+		(property "Value" "200"
 			(at 198.12 80.0099 0)
 			(effects
@@
 			)
 		)
-		(property "Value" "R"
+		(property "Value" "0"
 			(at 185.42 69.85 90)
 			(effects
@@
 			)
 		)
-		(property "Value" "R"
+		(property "Value" "0"
 			(at 185.42 87.63 90)
 			(effects
@@
 			)
 		)
-		(property "Value" "C"
+		(property "Value" "25PF"
 			(at 210.82 80.0099 0)
 			(effects
@@
 			)
 		)
-		(property "Value" "C"
+		(property "Value" "10000PF"
 			(at 182.88 96.5201 0)
 			(effects
@@
 			)
 		)
-		(property "Value" "R"
+		(property "Value" "4.99"
 			(at 227.33 77.47 90)
 			(effects
@@
 			)
 		)
-		(property "Value" "R"
+		(property "Value" "200"
 			(at 204.47 95.25 90)
 			(effects

Commit message: lots small updates
Parts:
- L2101: value L -> DNP
Changed lines of the file:
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@@
 			)
 		)
-		(property "Value" "L"
+		(property "Value" "DNP"
 			(at 218.44 81.2799 0)
 			(effects
