File: slowmon.kicad_sch (KiCad schematic)
At the start: 20 parts, among them J801 20021121-00020C4LF, J802 20021121-00020C4LF

Commit message: fields
Parts:
- C801: gfootprint 0402 -> (none)
- C802, C803, C804, C805, C806, R801, R802, R803, R804, R805, R806, R807, R808, R809, R810, R811: gfootprint 0603 -> (none)
- J801, J802: MANUFACTURER AMPHENOL -> (none); PARTREV N -> (none); STANDARD Manufacturer Recommendations -> (none)
Changed lines of the file:
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@@
-			)
-		)
-		(property "Sim.Device" "D"
-			(at 163.83 64.77 0)
-			(effects
-				(font
-					(size 1.27 1.27)
-				)
-				(hide yes)
-			)
-		)
-		(property "Sim.Pins" "1=K 2=A"
-			(at 163.83 64.77 0)
-			(effects
-				(font
-					(size 1.27 1.27)
-				)
-				(hide yes)
 			)
 		)
@@
 			)
 		)
-		(property "PARTREV" "N"
-			(at 205.74 92.71 0)
-			(effects
-				(font
-					(size 1.27 1.27)
-				)
-				(justify bottom)
-				(hide yes)
-			)
-		)
-		(property "STANDARD" "Manufacturer Recommendations"
-			(at 205.74 92.71 0)
-			(effects
-				(font
-					(size 1.27 1.27)
-				)
-				(justify bottom)
-				(hide yes)
-			)
-		)
-		(property "MANUFACTURER" "AMPHENOL"
-			(at 205.74 92.71 0)
-			(effects
-				(font
-					(size 1.27 1.27)
-				)
-				(justify bottom)
-				(hide yes)
-			)
-		)
 		(pin "18"
 		)
@@
 			)
 		)
-		(property "gfootprint" "0603"
-			(at 0 0 0)
-			(effects
-				(font
-					(size 1.27 1.27)
-				)
-				(hide yes)
-			)
-		)
 		(pin "1"
 		)
@@
 			)
 		)
-		(property "gfootprint" "0603"
-			(at 0 0 0)
-			(effects
-				(font
-					(size 1.27 1.27)
-				)
-				(hide yes)
-			)
-		)
 		(pin "1"
 		)
@@
 			)
 		)
-		(property "gfootprint" "0603"
-			(at 96.52 107.95 0)
-			(effects
-				(font
-					(size 1.27 1.27)
-				)
-				(hide yes)
-			)
-		)
 		(pin "2"
 		)
@@
 			)
 		)
-		(property "gfootprint" "0603"
-			(at 10.16 -24.13 0)
-			(effects
-				(font
-					(size 1.27 1.27)
-				)
-				(hide yes)
-			)
-		)
 		(pin "2"
 		)
@@
 			)
 		)
-		(property "gfootprint" "0603"
-			(at 0 0 0)
-			(effects
-				(font
-					(size 1.27 1.27)
-				)
-				(hide yes)
-			)
-		)
 		(pin "1"
 		)
@@
 			)
 		)
-		(property "gfootprint" "0603"
-			(at 0 204.47 0)
-			(effects
-				(font
-					(size 1.27 1.27)
-				)
-				(hide yes)
-			)
-		)
 		(pin "1"
 		)
@@
 			)
 		)
-		(property "gfootprint" "0603"
-			(at 0 213.36 0)
-			(effects
-				(font
-					(size 1.27 1.27)
-				)
-				(hide yes)
-			)
-		)
 		(pin "1"
 		)
@@
 			)
 		)
-		(property "gfootprint" "0603"
-			(at 0 213.36 0)
-			(effects
-				(font
-					(size 1.27 1.27)
-				)
-				(hide yes)
-			)
-		)
 		(pin "1"
 		)
@@
 			)
 		)
-		(property "gfootprint" "0402"
-			(at 10.16 -36.83 0)
-			(effects
-				(font
-					(size 1.27 1.27)
-				)
-				(hide yes)
-			)
-		)
 		(pin "1"
 		)
@@
 			)
 		)
-		(property "gfootprint" "0603"
-			(at 0 201.93 0)
-			(effects
-				(font
-					(size 1.27 1.27)
-				)
-				(hide yes)
-			)
-		)
 		(pin "1"
 		)
@@
 			)
 		)
-		(property "gfootprint" "0603"
-			(at 0 144.78 0)
-			(effects
-				(font
-					(size 1.27 1.27)
-				)
-				(hide yes)
-			)
-		)
 		(pin "2"
 		)
@@
 			)
 		)
-		(property "gfootprint" "0603"
-			(at 0 0 0)
-			(effects
-				(font
-					(size 1.27 1.27)
-				)
-				(hide yes)
-			)
-		)
 		(pin "1"
 		)
@@
 			)
 		)
-		(property "gfootprint" "0603"
-			(at 96.52 217.17 0)
-			(effects
-				(font
-					(size 1.27 1.27)
-				)
-				(hide yes)
-			)
-		)
 		(pin "2"
 		)
@@
 			)
 		)
-		(property "gfootprint" "0603"
-			(at 0 0 0)
-			(effects
-				(font
-					(size 1.27 1.27)
-				)
-				(hide yes)
-			)
-		)
 		(pin "1"
 		)
@@
 			)
 		)
-		(property "gfootprint" "0603"
-			(at -12.7 12.7 0)
-			(effects
-				(font
-					(size 1.27 1.27)
-				)
-				(hide yes)
-			)
-		)
 		(pin "2"
 		)
@@
 			)
 		)
-		(property "gfootprint" "0603"
-			(at 0 223.52 0)
-			(effects
-				(font
-					(size 1.27 1.27)
-				)
-				(hide yes)
-			)
-		)
 		(pin "1"
 		)
@@
 			)
 		)
-		(property "PARTREV" "N"
-			(at 116.84 92.71 0)
-			(effects
-				(font
-					(size 1.27 1.27)
-				)
-				(justify bottom)
-				(hide yes)
-			)
-		)
-		(property "STANDARD" "Manufacturer Recommendations"
-			(at 116.84 92.71 0)
-			(effects
-				(font
-					(size 1.27 1.27)
-				)
-				(justify bottom)
-				(hide yes)
-			)
-		)
-		(property "MANUFACTURER" "AMPHENOL"
-			(at 116.84 92.71 0)
-			(effects
-				(font
-					(size 1.27 1.27)
-				)
-				(justify bottom)
-				(hide yes)
-			)
-		)
 		(pin "18"
 		)
@@
 			(effects
 				(font
-					(size 1.27 1.27)
-				)
-				(hide yes)
-			)
-		)
-		(property "gfootprint" "0603"
-			(at 10.16 -36.83 0)
-			(effects
-				(font

Commit message: vendor info
Parts:
- C801: Vendor (none) -> digikey:490-1293-1-ND
- C802, C803, C804, C805, C806: Vendor (none) -> digikey:1276-1280-1-ND
- D801: Vendor (none) -> digikey:754-1116-1-ND
- J801, J802: Vendor (none) -> digikey:609-3698-1-ND
- R801, R802, R804: Vendor (none) -> digikey:311-4.75KHRCT-ND
- R803, R807, R808, R809, R810, R811: Vendor (none) -> digikey:311-22.0KHRCT-ND
- R806: Vendor (none) -> digikey:311-150HRCT-ND
Changed lines of the file:
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@@
+			)
+		)
+		(property "Vendor" "digikey:754-1116-1-ND"
+			(at 228.6 228.6 0)
+			(effects
+				(font
+					(size 1.27 1.27)
+				)
+				(hide yes)
 			)
 		)
@@
 			)
 		)
+		(property "Vendor" "digikey:609-3698-1-ND"
+			(at 0 185.42 0)
+			(effects
+				(font
+					(size 1.27 1.27)
+				)
+				(hide yes)
+			)
+		)
 		(pin "18"
 		)
@@
 			)
 		)
+		(property "Vendor" "digikey:311-22.0KHRCT-ND"
+			(at 0 0 0)
+			(effects
+				(font
+					(size 1.27 1.27)
+				)
+				(hide yes)
+			)
+		)
 		(pin "1"
 		)
@@
 			)
 		)
+		(property "Vendor" "digikey:311-22.0KHRCT-ND"
+			(at 0 0 0)
+			(effects
+				(font
+					(size 1.27 1.27)
+				)
+				(hide yes)
+			)
+		)
 		(pin "1"
 		)
@@
 			)
 		)
+		(property "Vendor" "digikey:311-4.75KHRCT-ND"
+			(at 106.68 71.12 0)
+			(effects
+				(font
+					(size 1.27 1.27)
+				)
+				(hide yes)
+			)
+		)
 		(pin "2"
 		)
@@
 			)
 		)
+		(property "Vendor" "digikey:311-22.0KHRCT-ND"
+			(at 0 0 0)
+			(effects
+				(font
+					(size 1.27 1.27)
+				)
+				(hide yes)
+			)
+		)
 		(pin "2"
 		)
@@
 			)
 		)
+		(property "Vendor" "digikey:311-22.0KHRCT-ND"
+			(at 0 0 0)
+			(effects
+				(font
+					(size 1.27 1.27)
+				)
+				(hide yes)
+			)
+		)
 		(pin "1"
 		)
@@
 			)
 		)
+		(property "Vendor" "digikey:1276-1280-1-ND"
+			(at 0 233.68 0)
+			(effects
+				(font
+					(size 1.27 1.27)
+				)
+				(hide yes)
+			)
+		)
 		(pin "1"
 		)
@@
 			)
 		)
+		(property "Vendor" "digikey:1276-1280-1-ND"
+			(at 0 233.68 0)
+			(effects
+				(font
+					(size 1.27 1.27)
+				)
+				(hide yes)
+			)
+		)
 		(pin "1"
 		)
@@
 			)
 		)
+		(property "Vendor" "digikey:1276-1280-1-ND"
+			(at 0 223.52 0)
+			(effects
+				(font
+					(size 1.27 1.27)
+				)
+				(hide yes)
+			)
+		)
 		(pin "1"
 		)
@@
 			)
 		)
+		(property "Vendor" "digikey:490-1293-1-ND"
+			(at 0 0 0)
+			(effects
+				(font
+					(size 1.27 1.27)
+				)
+				(hide yes)
+			)
+		)
 		(pin "1"
 		)
@@
 			)
 		)
+		(property "Vendor" "digikey:1276-1280-1-ND"
+			(at 0 220.98 0)
+			(effects
+				(font
+					(size 1.27 1.27)
+				)
+				(hide yes)
+			)
+		)
 		(pin "1"
 		)
@@
 			)
 		)
+		(property "Vendor" "digikey:311-150HRCT-ND"
+			(at 0 144.78 0)
+			(effects
+				(font
+					(size 1.27 1.27)
+				)
+				(hide yes)
+			)
+		)
 		(pin "2"
 		)
@@
 			)
 		)
+		(property "Vendor" "digikey:311-22.0KHRCT-ND"
+			(at 0 0 0)
+			(effects
+				(font
+					(size 1.27 1.27)
+				)
+				(hide yes)
+			)
+		)
 		(pin "1"
 		)
@@
 			)
 		)
+		(property "Vendor" "digikey:311-4.75KHRCT-ND"
+			(at 106.68 193.04 0)
+			(effects
+				(font
+					(size 1.27 1.27)
+				)
+				(hide yes)
+			)
+		)
 		(pin "2"
 		)
@@
 			)
 		)
+		(property "Vendor" "digikey:311-22.0KHRCT-ND"
+			(at 0 0 0)
+			(effects
+				(font
+					(size 1.27 1.27)
+				)
+				(hide yes)
+			)
+		)
 		(pin "1"
 		)
@@
 			)
 		)
+		(property "Vendor" "digikey:1276-1280-1-ND"
+			(at 0 233.68 0)
+			(effects
+				(font
+					(size 1.27 1.27)
+				)
+				(hide yes)
+			)
+		)
 		(pin "1"
 		)
@@
 			)
 		)
+		(property "Vendor" "digikey:609-3698-1-ND"
+			(at 0 185.42 0)
+			(effects
+				(font
+					(size 1.27 1.27)
+				)
+				(hide yes)
+			)
+		)
 		(pin "18"
 		)
@@
 			(effects
 				(font
+					(size 1.27 1.27)
+				)
+				(hide yes)
+			)
+		)
+		(property "Vendor" "digikey:311-4.75KHRCT-ND"
+			(at 0 0 0)
+			(effects
+				(font

Commit message: update value
Parts:
- C801: value C -> 220PF
- C802, C803, C804, C805, C806: value C -> 150PF
- D801: value D -> APT1608CGCK
- R801, R802, R804: value R -> 4.75K
- R803, R807, R808, R809, R810, R811: value R -> 22K
- R806: value R -> 150
Changed lines of the file:
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@@
 			)
 		)
-		(property "Value" "D"
+		(property "Value" "APT1608CGCK"
 			(at 160.02 64.77 0)
 			(effects
@@
 			)
 		)
-		(property "Value" "R"
+		(property "Value" "22K"
 			(at 186.69 55.8801 0)
 			(effects
@@
 			)
 		)
-		(property "Value" "R"
+		(property "Value" "22K"
 			(at 179.07 66.0401 0)
 			(effects
@@
 			)
 		)
-		(property "Value" "R"
+		(property "Value" "4.75K"
 			(at 50.8 36.8299 0)
 			(effects
@@
 			)
 		)
-		(property "Value" "R"
+		(property "Value" "22K"
 			(at 50.8 90.1699 0)
 			(effects
@@
 			)
 		)
-		(property "Value" "R"
+		(property "Value" "22K"
 			(at 182.88 60.9601 0)
 			(effects
@@
 			)
 		)
-		(property "Value" "C"
+		(property "Value" "150PF"
 			(at 78.74 118.1099 0)
 			(effects
@@
 			)
 		)
-		(property "Value" "C"
+		(property "Value" "150PF"
 			(at 90.17 118.1099 0)
 			(effects
@@
 			)
 		)
-		(property "Value" "C"
+		(property "Value" "150PF"
 			(at 96.52 113.0299 0)
 			(effects
@@
 			)
 		)
-		(property "Value" "C"
+		(property "Value" "220PF"
 			(at 49.53 53.3399 0)
 			(effects
@@
 			)
 		)
-		(property "Value" "C"
+		(property "Value" "150PF"
 			(at 83.82 111.7599 0)
 			(effects
@@
 			)
 		)
-		(property "Value" "R"
+		(property "Value" "150"
 			(at 166.37 73.6599 0)
 			(effects
@@
 			)
 		)
-		(property "Value" "R"
+		(property "Value" "22K"
 			(at 191.77 52.0701 0)
 			(effects
@@
 			)
 		)
-		(property "Value" "R"
+		(property "Value" "4.75K"
 			(at 50.8 97.7899 0)
 			(effects
@@
 			)
 		)
-		(property "Value" "R"
+		(property "Value" "22K"
 			(at 172.72 68.5801 0)
 			(effects
@@
 			)
 		)
-		(property "Value" "C"
+		(property "Value" "150PF"
 			(at 104.14 118.1099 0)
 			(effects
@@
 			)
 		)
-		(property "Value" "R"
+		(property "Value" "4.75K"
 			(at 50.8 29.2099 0)
 			(effects

Commit message: lots small updates
Parts:
- R805: value R -> DNP
Changed lines of the file:
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@@
 			)
 		)
-		(property "Value" "R"
+		(property "Value" "DNP"
 			(at 69.85 78.74 90)
 			(effects
