File: spu0410.kicad_sch (KiCad schematic)
At the start: 10 parts, among them U1601 LT6233CS6TRMPBF

Commit message: fields
Parts:
- C1601, C1602, R1601, R1602, R1603, R1604, R1605, TP1: gfootprint 0603 -> (none)
- U1601: Availability In Stock -> (none); COPYRIGHT Copyright C 2016 Accelerated Designs. All rights reserved -> (none); Check_prices https://www.snapeda.com/parts/LT6233CS6%23TRMPBF/Analog+Dev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 -> (none); DIGIKEY_PART_NUMBER LT6233CS6#TRMPBFTRND -> (none); Description_1 General Purpose Amplifier 1 Circuit Rail-to-Rail TSOT-23-6 -> (none); MANUFACTURER_PART_NUMBER LT6233CS6#TRMPBF -> (none); MF Analog Devices -> (none); MP LT6233CS6#TRMPBF -> (none); Package SOT-23-6 Linear Technology -> (none); Price None -> (none); Purchase-URL https://www.snapeda.com/api/url_track_click_mouser/?unipart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 -> (none); SnapEDA_Link https://www.snapeda.com/parts/LT6233CS6%23TRMPBF/Analog+Dev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 -> (none); VENDOR Linear Technology -> (none)
Changed lines of the file:
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@@
-			)
-		)
-		(property "gfootprint" "0603"
-			(at 144.78 -144.78 0)
-			(effects
-				(font
-					(size 1.27 1.27)
-				)
-				(hide yes)
 			)
 		)
@@
 		(property "Description" "Resistor"
 			(at 176.53 54.61 0)
-			(effects
-				(font
-					(size 1.27 1.27)
-				)
-				(hide yes)
-			)
-		)
-		(property "gfootprint" "0603"
-			(at 121.92 -121.92 0)
 			(effects
 				(font
@@
 			)
 		)
-		(property "gfootprint" "0603"
-			(at 307.34 -111.76 0)
-			(effects
-				(font
-					(size 1.27 1.27)
-				)
-				(hide yes)
-			)
-		)
 		(pin "2"
 		)
@@
 			)
 		)
-		(property "gfootprint" "0603"
-			(at 285.75 285.75 0)
-			(effects
-				(font
-					(size 1.27 1.27)
-				)
-				(hide yes)
-			)
-		)
 		(pin "1"
 		)
@@
 			)
 		)
-		(property "gfootprint" "0603"
-			(at 41.91 -41.91 0)
-			(effects
-				(font
-					(size 1.27 1.27)
-				)
-				(hide yes)
-			)
-		)
 		(pin "2"
 		)
@@
 			)
 		)
-		(property "gfootprint" "0603"
-			(at 0 119.38 0)
-			(effects
-				(font
-					(size 1.27 1.27)
-				)
-				(hide yes)
-			)
-		)
 		(pin "1"
 		)
@@
 		(property "Description" "Resistor"
 			(at 125.73 76.2 0)
-			(effects
-				(font
-					(size 1.27 1.27)
-				)
-				(hide yes)
-			)
-		)
-		(property "gfootprint" "0603"
-			(at 49.53 -49.53 0)
 			(effects
 				(font
@@
 			)
 		)
-		(property "DIGIKEY_PART_NUMBER" "LT6233CS6#TRMPBFTRND"
-			(at 204.47 71.12 0)
-			(effects
-				(font
-					(size 1.27 1.27)
-				)
-				(justify bottom)
-				(hide yes)
-			)
-		)
-		(property "MF" "Analog Devices"
-			(at 204.47 71.12 0)
-			(effects
-				(font
-					(size 1.27 1.27)
-				)
-				(justify bottom)
-				(hide yes)
-			)
-		)
-		(property "VENDOR" "Linear Technology"
-			(at 204.47 71.12 0)
-			(effects
-				(font
-					(size 1.27 1.27)
-				)
-				(justify bottom)
-				(hide yes)
-			)
-		)
-		(property "Description_1" "\nGeneral Purpose Amplifier 1 Circuit Rail-to-Rail TSOT-23-6\n"
-			(at 204.47 71.12 0)
-			(effects
-				(font
-					(size 1.27 1.27)
-				)
-				(justify bottom)
-				(hide yes)
-			)
-		)
-		(property "COPYRIGHT" "Copyright C 2016 Accelerated Designs. All rights reserved"
-			(at 204.47 71.12 0)
-			(effects
-				(font
-					(size 1.27 1.27)
-				)
-				(justify bottom)
-				(hide yes)
-			)
-		)
-		(property "Package" "SOT-23-6 Linear Technology"
-			(at 204.47 71.12 0)
-			(effects
-				(font
-					(size 1.27 1.27)
-				)
-				(justify bottom)
-				(hide yes)
-			)
-		)
-		(property "Price" "None"
-			(at 204.47 71.12 0)
-			(effects
-				(font
-					(size 1.27 1.27)
-				)
-				(justify bottom)
-				(hide yes)
-			)
-		)
-		(property "Check_prices" "https://www.snapeda.com/parts/LT6233CS6%23TRMPBF/Analog+Devices/view-part/?ref=eda"
-			(at 204.47 71.12 0)
-			(effects
-				(font
-					(size 1.27 1.27)
-				)
-				(justify bottom)
-				(hide yes)
-			)
-		)
-		(property "SnapEDA_Link" "https://www.snapeda.com/parts/LT6233CS6%23TRMPBF/Analog+Devices/view-part/?ref=snap"
-			(at 204.47 71.12 0)
-			(effects
-				(font
-					(size 1.27 1.27)
-				)
-				(justify bottom)
-				(hide yes)
-			)
-		)
-		(property "MP" "LT6233CS6#TRMPBF"
-			(at 204.47 71.12 0)
-			(effects
-				(font
-					(size 1.27 1.27)
-				)
-				(justify bottom)
-				(hide yes)
-			)
-		)
-		(property "Purchase-URL" "https://www.snapeda.com/api/url_track_click_mouser/?unipart_id=491320&manufacturer=Analog Devices&part_name=LT6233CS6#TRMPBF&search_term=lt6233cs6#trmpbf"
-			(at 204.47 71.12 0)
-			(effects
-				(font
-					(size 1.27 1.27)
-				)
-				(justify bottom)
-				(hide yes)
-			)
-		)
-		(property "Availability" "In Stock"
-			(at 204.47 71.12 0)
-			(effects
-				(font
-					(size 1.27 1.27)
-				)
-				(justify bottom)
-				(hide yes)
-			)
-		)
-		(property "MANUFACTURER_PART_NUMBER" "LT6233CS6#TRMPBF"
-			(at 204.47 71.12 0)
-			(effects
-				(font
-					(size 1.27 1.27)
-				)
-				(justify bottom)
-				(hide yes)
-			)
-		)
 		(pin "2"
 		)
@@
 			(effects
 				(font
-					(size 1.27 1.27)
-				)
-				(hide yes)
-			)
-		)
-		(property "gfootprint" "0603"
-			(at 299.72 299.72 0)
-			(effects
-				(font

Commit message: vendor info
Parts:
- C1601, C1602: Vendor (none) -> digikey:490-3897-1-ND
- MIC1601: Vendor (none) -> digikey:423-1138-1-ND
- R1601, R1603, R1604: Vendor (none) -> digikey:311-4.75KHRCT-ND
- R1602: Vendor (none) -> digikey:311-220KHRCT-ND
- R1605: Vendor (none) -> digikey:P0.0GCT-ND
- U1601: Vendor (none) -> digikey:LT6233CS6#TRMPBFCT-ND
Changed lines of the file:
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@@
+			)
+		)
+		(property "Vendor" "digikey:P0.0GCT-ND"
+			(at 144.78 -144.78 0)
+			(effects
+				(font
+					(size 1.27 1.27)
+				)
+				(hide yes)
 			)
 		)
@@
 		(property "Description" "Resistor"
 			(at 176.53 54.61 0)
+			(effects
+				(font
+					(size 1.27 1.27)
+				)
+				(hide yes)
+			)
+		)
+		(property "Vendor" "digikey:311-220KHRCT-ND"
+			(at 121.92 -121.92 0)
 			(effects
 				(font
@@
 			)
 		)
+		(property "Vendor" "digikey:490-3897-1-ND"
+			(at 307.34 -111.76 0)
+			(effects
+				(font
+					(size 1.27 1.27)
+				)
+				(hide yes)
+			)
+		)
 		(pin "2"
 		)
@@
 			)
 		)
+		(property "Vendor" "digikey:311-4.75KHRCT-ND"
+			(at 285.75 285.75 0)
+			(effects
+				(font
+					(size 1.27 1.27)
+				)
+				(hide yes)
+			)
+		)
 		(pin "1"
 		)
@@
 			)
 		)
+		(property "Vendor" "digikey:490-3897-1-ND"
+			(at 41.91 -41.91 0)
+			(effects
+				(font
+					(size 1.27 1.27)
+				)
+				(hide yes)
+			)
+		)
 		(pin "2"
 		)
@@
 		(property "Description" "Resistor"
 			(at 125.73 76.2 0)
+			(effects
+				(font
+					(size 1.27 1.27)
+				)
+				(hide yes)
+			)
+		)
+		(property "Vendor" "digikey:311-4.75KHRCT-ND"
+			(at 49.53 -49.53 0)
 			(effects
 				(font
@@
 			)
 		)
+		(property "Vendor" "digikey:LT6233CS6#TRMPBFCT-ND"
+			(at 408.94 142.24 0)
+			(effects
+				(font
+					(size 1.27 1.27)
+				)
+				(hide yes)
+			)
+		)
 		(pin "2"
 		)
@@
 			)
 		)
+		(property "Vendor" "digikey:423-1138-1-ND"
+			(at 0 152.4 0)
+			(effects
+				(font
+					(size 1.27 1.27)
+				)
+				(hide yes)
+			)
+		)
 		(pin "4"
 		)
@@
 			(effects
 				(font
+					(size 1.27 1.27)
+				)
+				(hide yes)
+			)
+		)
+		(property "Vendor" "digikey:311-4.75KHRCT-ND"
+			(at 299.72 299.72 0)
+			(effects
+				(font

Commit message: update value
Parts:
- C1601, C1602: value C -> 1UF
- R1601, R1603, R1604: value R -> 4.75K
- R1602: value R -> 220K
- R1605: value R -> 0
- U1601: value LT6233CS6TRMPBF -> LT6233CS6#TRMPBF
Changed lines of the file:
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@@
 			)
 		)
-		(property "Value" "R"
+		(property "Value" "0"
 			(at 215.9 67.31 90)
 			(effects
@@
 			)
 		)
-		(property "Value" "R"
+		(property "Value" "220K"
 			(at 176.53 50.8 90)
 			(effects
@@
 			)
 		)
-		(property "Value" "C"
+		(property "Value" "1UF"
 			(at 209.55 102.87 90)
 			(effects
@@
 			)
 		)
-		(property "Value" "R"
+		(property "Value" "4.75K"
 			(at 195.58 86.36 90)
 			(effects
@@
 			)
 		)
-		(property "Value" "C"
+		(property "Value" "1UF"
 			(at 118.11 71.12 90)
 			(effects
@@
 			)
 		)
-		(property "Value" "R"
+		(property "Value" "4.75K"
 			(at 125.73 72.39 90)
 			(effects
@@
 			)
 		)
-		(property "Value" "LT6233CS6TRMPBF"
+		(property "Value" "LT6233CS6#TRMPBF"
 			(at 181.61 63.5 0)
 			(effects
@@
 			)
 		)
-		(property "Value" "R"
+		(property "Value" "4.75K"
 			(at 209.55 86.36 90)
 			(effects

Commit message: lots small updates
Parts:
- TP1: now left out of the parts list
Changed lines of the file:
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@@
 		(unit 1)
 		(exclude_from_sim no)
-		(in_bom yes)
+		(in_bom no)
 		(on_board yes)
 		(dnp no)
