File: fmclpc.kicad_sch (KiCad schematic)
At the start: 3 parts, among them J1401 ASP-134604-01, J1402 ASP-134604-01

Commit message: fields
Parts:
- J1401, J1402: MANUFACTURER SAMTEC -> (none); PARTREV S -> (none); STANDARD Manufacturer recommendations -> (none)
- TP22: gfootprint 0603 -> (none)
Changed lines of the file:
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@@
-			)
-		)
-		(property "PARTREV" "S"
-			(at 144.78 133.35 0)
-			(effects
-				(font
-					(size 1.27 1.27)
-				)
-				(justify bottom)
-				(hide yes)
-			)
-		)
-		(property "STANDARD" "Manufacturer recommendations"
-			(at 144.78 133.35 0)
-			(effects
-				(font
-					(size 1.27 1.27)
-				)
-				(justify bottom)
-				(hide yes)
-			)
-		)
-		(property "MANUFACTURER" "SAMTEC"
-			(at 144.78 133.35 0)
-			(effects
-				(font
-					(size 1.27 1.27)
-				)
-				(justify bottom)
-				(hide yes)
 			)
 		)
@@
 			)
 		)
-		(property "gfootprint" "0603"
-			(at 127 -154.94 0)
-			(effects
-				(font
-					(size 1.27 1.27)
-				)
-				(hide yes)
-			)
-		)
 		(pin "1"
 		)
@@
 				(hide yes)
 			)
-		)
-		(property "PARTREV" "S"
-			(at 71.12 139.7 0)
-			(effects
-				(font
-					(size 1.27 1.27)
-				)
-				(justify bottom)
-				(hide yes)
-			)
-		)
-		(property "STANDARD" "Manufacturer recommendations"
-			(at 71.12 139.7 0)
-			(effects
-				(font
-					(size 1.27 1.27)
-				)
-				(justify bottom)
-				(hide yes)
-			)
-		)
-		(property "MANUFACTURER" "SAMTEC"
-			(at 71.12 139.7 0)
-			(effects
-				(font
-					(size 1.27 1.27)
-				)
-				(justify bottom)
-				(hide yes)
-			)

Commit message: vendor info
Parts:
- J1401, J1402: Vendor (none) -> digikey:79X1317@Newark
Changed lines of the file:
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@@
+			)
+		)
+		(property "Vendor" "digikey:79X1317@Newark"
+			(at 289.56 0 0)
+			(effects
+				(font
+					(size 1.27 1.27)
+				)
+				(hide yes)
 			)
 		)
@@
 			(effects
 				(font
+					(size 1.27 1.27)
+				)
+				(hide yes)
+			)
+		)
+		(property "Vendor" "digikey:79X1317@Newark"
+			(at 142.24 0 0)
+			(effects
+				(font

Commit message: lots small updates
Parts:
- TP22: now left out of the parts list
Changed lines of the file:
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@@
 		(unit 1)
 		(exclude_from_sim no)
-		(in_bom yes)
+		(in_bom no)
 		(on_board yes)
 		(dnp no)

Commit message: 3/105
Parts:
- J1401, J1402: Vendor digikey:79X1317@Newark -> newark:79X1317
Changed lines of the file:
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@@
 			)
 		)
-		(property "Vendor" "digikey:79X1317@Newark"
+		(property "Vendor" "newark:79X1317"
 			(at 289.56 0 0)
 			(effects
@@
 			)
 		)
-		(property "Vendor" "digikey:79X1317@Newark"
+		(property "Vendor" "newark:79X1317"
 			(at 142.24 0 0)
 			(effects
