File: fmclpc.kicad_sch (KiCad schematic)
At the start: 3 parts, among them J1401 ASP-134604-01, J1402 ASP-134604-01

Commit message: Further Project cleanup
-Added BOM and fabrication files
-updated all documentation files
- Added suggested DC blocking cap at DAC outputs

-Set DRC to 5mil trace and space and fixed various violations detailed below
- Removed various small tracks overlapping IC pads on U2701,U2901,U3101,U3201
- Spaced vias 5 mil apart around U701, U201, 1201
- Moved LMK_CLKout3 pair on In4 layer away from PMOD1_1 pin
- adjusted track into pin47 on U701 to clear pin 48
- adjusted trace under U903 to give more room from ground pads/vias
- spaced out vias around pins45/46 of U201

-Many tweak to trace to go through the center of pad throughout the design
-An example is the trace around C3005
Parts:
- J1401, J1402: Manufacturer (none) -> Samtec; Manufacturer Part Number (none) -> ASP-134604-01; Vendor newark:79X1317 -> digikey:612-ASP-134604-01CT-ND
Changed lines of the file:
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@@
 			)
 		)
-		(property "Description" ""
+		(property "Description" "ASP-134604-01"
 			(at 143.51 134.62 0)
 			(effects
@@
 			)
 		)
-		(property "Vendor" "newark:79X1317"
+		(property "Vendor" "digikey:612-ASP-134604-01CT-ND"
 			(at -1.27 1.27 0)
 			(effects
@@
 			)
 		)
-		(property "Manufacturer" ""
+		(property "Manufacturer" "Samtec"
 			(at 143.51 134.62 0)
 			(effects
@@
 			)
 		)
-		(property "Manufacturer Part Number" ""
+		(property "Manufacturer Part Number" "ASP-134604-01"
 			(at 143.51 134.62 0)
 			(effects
@@
 			)
 		)
-		(property "Description" ""
+		(property "Description" "ASP-134604-01"
 			(at 69.85 36.83 0)
 			(effects
@@
 			)
 		)
-		(property "Vendor" "newark:79X1317"
+		(property "Vendor" "digikey:612-ASP-134604-01CT-ND"
 			(at -1.27 -102.87 0)
 			(effects
@@
 			)
 		)
-		(property "Manufacturer" ""
+		(property "Manufacturer" "Samtec"
 			(at 69.85 36.83 0)
 			(effects
@@
 			)
 		)
-		(property "Manufacturer Part Number" ""
+		(property "Manufacturer Part Number" "ASP-134604-01"
 			(at 69.85 36.83 0)
 			(effects
@@
 			)
 		)
-		(property "Description" ""
+		(property "Description" "ASP-134604-01"
 			(at 146.05 30.48 0)
 			(effects
@@
 			)
 		)
-		(property "Vendor" "newark:79X1317"
+		(property "Vendor" "digikey:612-ASP-134604-01CT-ND"
 			(at 290.83 -102.87 0)
 			(effects
@@
 			)
 		)
-		(property "Manufacturer" ""
+		(property "Manufacturer" "Samtec"
 			(at 146.05 30.48 0)
 			(effects
@@
 			)
 		)
-		(property "Manufacturer Part Number" ""
+		(property "Manufacturer Part Number" "ASP-134604-01"
 			(at 146.05 30.48 0)
 			(effects
@@
 			)
 		)
-		(property "Description" ""
+		(property "Description" "ASP-134604-01"
 			(at 72.39 36.83 0)
 			(effects
@@
 			)
 		)
-		(property "Vendor" "newark:79X1317"
+		(property "Vendor" "digikey:612-ASP-134604-01CT-ND"
 			(at 143.51 -102.87 0)
 			(effects
@@
 			)
 		)
-		(property "Manufacturer" ""
+		(property "Manufacturer" "Samtec"
 			(at 72.39 36.83 0)
 			(effects
@@
 			)
 		)
-		(property "Manufacturer Part Number" ""
+		(property "Manufacturer Part Number" "ASP-134604-01"
 			(at 72.39 36.83 0)
 			(effects
@@
 			)
 		)
-		(property "Description" ""
+		(property "Description" "ASP-134604-01"
 			(at 72.39 140.97 0)
 			(effects
@@
 			)
 		)
-		(property "Vendor" "newark:79X1317"
+		(property "Vendor" "digikey:612-ASP-134604-01CT-ND"
 			(at 143.51 1.27 0)
 			(effects
@@
 			)
 		)
-		(property "Manufacturer" ""
+		(property "Manufacturer" "Samtec"
 			(at 72.39 140.97 0)
 			(effects
@@
 			)
 		)
-		(property "Manufacturer Part Number" ""
+		(property "Manufacturer Part Number" "ASP-134604-01"
 			(at 72.39 140.97 0)
 			(effects
@@
 			)
 		)
-		(property "Description" ""
+		(property "Description" "ASP-134604-01"
 			(at 143.51 30.48 0)
 			(effects
@@
 			)
 		)
-		(property "Vendor" "newark:79X1317"
+		(property "Vendor" "digikey:612-ASP-134604-01CT-ND"
 			(at -1.27 -102.87 0)
 			(effects
@@
 			)
 		)
-		(property "Manufacturer" ""
+		(property "Manufacturer" "Samtec"
 			(at 143.51 30.48 0)
 			(effects
@@
 			)
 		)
-		(property "Manufacturer Part Number" ""
+		(property "Manufacturer Part Number" "ASP-134604-01"
 			(at 143.51 30.48 0)
 			(effects
@@
 			)
 		)
-		(property "Description" ""
+		(property "Description" "ASP-134604-01"
 			(at 146.05 134.62 0)
 			(effects
@@
 			)
 		)
-		(property "Vendor" "newark:79X1317"
+		(property "Vendor" "digikey:612-ASP-134604-01CT-ND"
 			(at 290.83 1.27 0)
 			(effects
@@
 			)
 		)
-		(property "Manufacturer" ""
+		(property "Manufacturer" "Samtec"
 			(at 146.05 134.62 0)
 			(effects
@@
 			)
 		)
-		(property "Manufacturer Part Number" ""
+		(property "Manufacturer Part Number" "ASP-134604-01"
 			(at 146.05 134.62 0)
 			(effects
@@
 			)
 		)
-		(property "Description" ""
+		(property "Description" "ASP-134604-01"
 			(at 69.85 140.97 0)
 			(effects
@@
 			)
 		)
-		(property "Vendor" "newark:79X1317"
+		(property "Vendor" "digikey:612-ASP-134604-01CT-ND"
 			(at -1.27 1.27 0)
 			(effects
@@
 			)
 		)
-		(property "Manufacturer" ""
+		(property "Manufacturer" "Samtec"
 			(at 69.85 140.97 0)
 			(effects
@@
 			)
 		)
-		(property "Manufacturer Part Number" ""
+		(property "Manufacturer Part Number" "ASP-134604-01"
 			(at 69.85 140.97 0)
 			(effects
