File: TPS62110_2v2.kicad_sch (KiCad schematic)
At the start: 13 parts, among them U2901 TPS62110RSAR

Commit message: fields
Parts:
- C2901, C2904, R2901, R2902, R2903, R2904, R2905: gfootprint 0603 -> (none)
- C2902, C2903, C2905: gfootprint 1206 -> (none)
- FB2901: gfootprint 0805 -> (none)
Changed lines of the file:
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@@
-			)
-		)
-		(property "gfootprint" "1206"
-			(at 0 0 0)
-			(effects
-				(font
-					(size 1.27 1.27)
-				)
-				(hide yes)
 			)
 		)
@@
 			)
 		)
-		(property "gfootprint" "0603"
-			(at 276.86 -81.28 0)
-			(effects
-				(font
-					(size 1.27 1.27)
-				)
-				(hide yes)
-			)
-		)
 		(pin "1"
 		)
@@
 			)
 		)
-		(property "gfootprint" "1206"
-			(at 0 0 0)
-			(effects
-				(font
-					(size 1.27 1.27)
-				)
-				(hide yes)
-			)
-		)
 		(pin "1"
 		)
@@
 			)
 		)
-		(property "gfootprint" "0603"
-			(at 0 0 0)
-			(effects
-				(font
-					(size 1.27 1.27)
-				)
-				(hide yes)
-			)
-		)
 		(pin "1"
 		)
@@
 			)
 		)
-		(property "gfootprint" "0603"
-			(at 0 0 0)
-			(effects
-				(font
-					(size 1.27 1.27)
-				)
-				(hide yes)
-			)
-		)
 		(pin "1"
 		)
@@
 			)
 		)
-		(property "gfootprint" "0603"
-			(at 0 0 0)
-			(effects
-				(font
-					(size 1.27 1.27)
-				)
-				(hide yes)
-			)
-		)
 		(pin "1"
 		)
@@
 			)
 		)
-		(property "gfootprint" "0603"
-			(at 0 0 0)
-			(effects
-				(font
-					(size 1.27 1.27)
-				)
-				(hide yes)
-			)
-		)
 		(pin "1"
 		)
@@
 			)
 		)
-		(property "gfootprint" "0603"
-			(at 0 0 0)
-			(effects
-				(font
-					(size 1.27 1.27)
-				)
-				(hide yes)
-			)
-		)
 		(pin "1"
 		)
@@
 			)
 		)
-		(property "gfootprint" "0805"
-			(at -31.75 135.89 0)
-			(effects
-				(font
-					(size 1.27 1.27)
-				)
-				(hide yes)
-			)
-		)
 		(pin "2"
 		)
@@
 			)
 		)
-		(property "gfootprint" "0603"
-			(at 203.2 0 0)
-			(effects
-				(font
-					(size 1.27 1.27)
-				)
-				(hide yes)
-			)
-		)
 		(pin "1"
 		)
@@
 			(effects
 				(font
-					(size 1.27 1.27)
-				)
-				(hide yes)
-			)
-		)
-		(property "gfootprint" "1206"
-			(at 408.94 187.96 0)
-			(effects
-				(font

Commit message: vendor info
Parts:
- C2901: Vendor (none) -> digikey:490-3897-1-ND
- C2902, C2903: Vendor (none) -> digikey:490-5527-1-ND
- C2904: Vendor (none) -> digikey:490-1403-1-ND
- C2905: Vendor (none) -> digikey:490-5528-1-ND
- FB2901: Vendor (none) -> digikey:732-1620-1-ND
- L2901: Vendor (none) -> digikey:732-1200-1-ND
- R2901, R2902: Vendor (none) -> digikey:311-11.5KHRCT-ND
- R2903, R2904, R2905: Vendor (none) -> digikey:311-422KHRCT-ND
- U2901: Vendor (none) -> digikey:296-24839-1-ND
Changed lines of the file:
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@@
+			)
+		)
+		(property "Vendor" "digikey:490-5527-1-ND"
+			(at 0 0 0)
+			(effects
+				(font
+					(size 1.27 1.27)
+				)
+				(hide yes)
 			)
 		)
@@
 			)
 		)
+		(property "Vendor" "digikey:311-422KHRCT-ND"
+			(at 276.86 -81.28 0)
+			(effects
+				(font
+					(size 1.27 1.27)
+				)
+				(hide yes)
+			)
+		)
 		(pin "1"
 		)
@@
 			)
 		)
+		(property "Vendor" "digikey:732-1200-1-ND"
+			(at 284.48 -83.82 0)
+			(effects
+				(font
+					(size 1.27 1.27)
+				)
+				(hide yes)
+			)
+		)
 		(pin "2"
 		)
@@
 			)
 		)
+		(property "Vendor" "digikey:490-5527-1-ND"
+			(at 0 0 0)
+			(effects
+				(font
+					(size 1.27 1.27)
+				)
+				(hide yes)
+			)
+		)
 		(pin "1"
 		)
@@
 			)
 		)
+		(property "Vendor" "digikey:311-11.5KHRCT-ND"
+			(at 0 0 0)
+			(effects
+				(font
+					(size 1.27 1.27)
+				)
+				(hide yes)
+			)
+		)
 		(pin "1"
 		)
@@
 			)
 		)
+		(property "Vendor" "digikey:490-3897-1-ND"
+			(at 0 0 0)
+			(effects
+				(font
+					(size 1.27 1.27)
+				)
+				(hide yes)
+			)
+		)
 		(pin "1"
 		)
@@
 			)
 		)
+		(property "Vendor" "digikey:311-422KHRCT-ND"
+			(at 0 0 0)
+			(effects
+				(font
+					(size 1.27 1.27)
+				)
+				(hide yes)
+			)
+		)
 		(pin "1"
 		)
@@
 			)
 		)
+		(property "Vendor" "digikey:311-422KHRCT-ND"
+			(at 0 0 0)
+			(effects
+				(font
+					(size 1.27 1.27)
+				)
+				(hide yes)
+			)
+		)
 		(pin "1"
 		)
@@
 			)
 		)
+		(property "Vendor" "digikey:490-1403-1-ND"
+			(at 0 0 0)
+			(effects
+				(font
+					(size 1.27 1.27)
+				)
+				(hide yes)
+			)
+		)
 		(pin "1"
 		)
@@
 			)
 		)
+		(property "Vendor" "digikey:732-1620-1-ND"
+			(at -31.75 135.89 0)
+			(effects
+				(font
+					(size 1.27 1.27)
+				)
+				(hide yes)
+			)
+		)
 		(pin "2"
 		)
@@
 			)
 		)
+		(property "Vendor" "digikey:311-11.5KHRCT-ND"
+			(at 203.2 0 0)
+			(effects
+				(font
+					(size 1.27 1.27)
+				)
+				(hide yes)
+			)
+		)
 		(pin "1"
 		)
@@
 			)
 		)
+		(property "Vendor" "digikey:296-24839-1-ND"
+			(at 0 0 0)
+			(effects
+				(font
+					(size 1.27 1.27)
+				)
+				(hide yes)
+			)
+		)
 		(pin "10"
 		)
@@
 			(effects
 				(font
+					(size 1.27 1.27)
+				)
+				(hide yes)
+			)
+		)
+		(property "Vendor" "digikey:490-5528-1-ND"
+			(at 408.94 187.96 0)
+			(effects
+				(font

Commit message: update value
Parts:
- C2901: value C -> 1UF
- C2902, C2903: value C -> 22UF
- C2904: value C -> 10PF
- C2905: value C -> 47UF
- FB2901: value FerriteBead -> 742792040
- L2901: value L -> 74477710
- R2901, R2902: value R -> 11.5K
- R2903, R2904, R2905: value R -> 422K
Changed lines of the file:
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@@
 			)
 		)
-		(property "Value" "C"
+		(property "Value" "22UF"
 			(at 76.2 97.7901 0)
 			(effects
@@
 			)
 		)
-		(property "Value" "R"
+		(property "Value" "422K"
 			(at 179.324 97.536 90)
 			(effects
@@
 			)
 		)
-		(property "Value" "L"
+		(property "Value" "74477710"
 			(at 184.15 102.87 90)
 			(effects
@@
 			)
 		)
-		(property "Value" "C"
+		(property "Value" "22UF"
 			(at 71.12 92.7101 0)
 			(effects
@@
 			)
 		)
-		(property "Value" "R"
+		(property "Value" "11.5K"
 			(at 98.044 88.138 90)
 			(effects
@@
 			)
 		)
-		(property "Value" "C"
+		(property "Value" "1UF"
 			(at 66.04 87.6301 0)
 			(effects
@@
 			)
 		)
-		(property "Value" "R"
+		(property "Value" "422K"
 			(at 186.69 88.9001 0)
 			(effects
@@
 			)
 		)
-		(property "Value" "R"
+		(property "Value" "422K"
 			(at 186.69 81.2801 0)
 			(effects
@@
 			)
 		)
-		(property "Value" "C"
+		(property "Value" "10PF"
 			(at 196.85 88.9001 0)
 			(effects
@@
 			)
 		)
-		(property "Value" "FerriteBead"
+		(property "Value" "742792040"
 			(at 52.1208 78.74 90)
 			(effects
@@
 			)
 		)
-		(property "Value" "R"
+		(property "Value" "11.5K"
 			(at 101.6 87.63 90)
 			(effects
@@
 			)
 		)
-		(property "Value" "C"
+		(property "Value" "47UF"
 			(at 208.28 95.2499 0)
 			(effects

Commit message: direction
Connections:
- net GND: now also U2901.1 (PGND)
Changed lines of the file:
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@@
+	)
+	(symbol
+		(lib_id "power:GND")
+		(at 110.49 107.95 0)
+		(mirror y)
+		(unit 1)
+		(exclude_from_sim no)
+		(in_bom yes)
+		(on_board yes)
+		(dnp no)
+		(fields_autoplaced yes)
+		(property "Reference" "#PWR02907"
+			(at 110.49 114.3 0)
+			(effects
+				(font
+					(size 1.27 1.27)
+				)
+				(hide yes)
+			)
+		)
+		(property "Value" "GND"
+			(at 110.49 113.03 0)
+			(effects
+				(font
+					(size 1.27 1.27)
+				)
+			)
+		)
+		(property "Footprint" ""
+			(at 110.49 107.95 0)
+			(effects
+				(font
+					(size 1.27 1.27)
+				)
+				(hide yes)
+			)
+		)
+		(property "Datasheet" ""
+			(at 110.49 107.95 0)
+			(effects
+				(font
+					(size 1.27 1.27)
+				)
+				(hide yes)
+			)
+		)
+		(property "Description" "Power symbol creates a global label with name \"GND\" , ground"
+			(at 110.49 107.95 0)
+			(effects
+				(font
+					(size 1.27 1.27)
+				)
+				(hide yes)
+			)
+		)
+		(pin "1"
+		)
+		(instances
+			(project "kdigitizer"
+				(path "/00000000-0000-0000-0000-000000000003/00000000-0000-0000-0000-000000000002/5fad0ac0-b30a-4219-89b7-8d138bce3826"
+					(reference "#PWR02907")
+					(unit 1)
+				)
+			)
+		)
 	)
 	(symbol
