File: level_shift.kicad_sch (KiCad schematic)
At the start: 37 parts, among them U1701 SN74LVC8T245PWR, U1702 SN74LVC8T245PWR, U1703 SN74LVC8T245PWR, U1704 SN74AVC4T245PWR, U1705 SN74AVC4T245PWR

Commit message: fields
Parts:
- C1701, C1702, C1703, C1704, C1705, C1706, C1707, C1708, C1709, C1710: gfootprint 0402 -> (none)
- R1701, R1702, R1703, R1704, R1705, R1706, TP10, TP14, TP15, TP16, TP20, TP21, TP23, TP24, TP25, TP26, TP27, TP3, TP4, TP7, TP8, TP9: gfootprint 0603 -> (none)

Commit message: vendor info
Parts:
- C1701, C1702, C1703, C1704, C1705, C1706, C1707, C1708, C1709, C1710: Vendor (none) -> digikey:490-1318-1-ND
- R1701, R1702, R1703, R1704, R1705, R1706: Vendor (none) -> digikey:311-4.75KHRCT-ND
- U1701, U1702, U1703: Vendor (none) -> digikey:296-18593-1-ND
- U1704, U1705: Vendor (none) -> digikey:296-18056-1-ND
Changed lines of the file:
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@@
 			)
 		)
+		(property "Vendor" "digikey:296-18056-1-ND"
+			(at 0 220.98 0)
+			(effects
+				(font
+					(size 1.27 1.27)
+				)
+				(hide yes)
+			)
+		)
 		(pin "9"
 		)
@@
 			)
 		)
+		(property "Vendor" "digikey:311-4.75KHRCT-ND"
+			(at 64.77 -64.77 0)
+			(effects
+				(font
+					(size 1.27 1.27)
+				)
+				(hide yes)
+			)
+		)
 		(pin "1"
 		)
@@
 			)
 		)
+		(property "Vendor" "digikey:490-1318-1-ND"
+			(at 0 81.28 0)
+			(effects
+				(font
+					(size 1.27 1.27)
+				)
+				(hide yes)
+			)
+		)
 		(pin "1"
 		)
@@
 			)
 		)
+		(property "Vendor" "digikey:311-4.75KHRCT-ND"
+			(at 193.04 193.04 0)
+			(effects
+				(font
+					(size 1.27 1.27)
+				)
+				(hide yes)
+			)
+		)
 		(pin "2"
 		)
@@
 			)
 		)
+		(property "Vendor" "digikey:490-1318-1-ND"
+			(at 0 228.6 0)
+			(effects
+				(font
+					(size 1.27 1.27)
+				)
+				(hide yes)
+			)
+		)
 		(pin "1"
 		)
@@
 			)
 		)
+		(property "Vendor" "digikey:490-1318-1-ND"
+			(at 99.06 0 0)
+			(effects
+				(font
+					(size 1.27 1.27)
+				)
+				(hide yes)
+			)
+		)
 		(pin "1"
 		)
@@
 			)
 		)
+		(property "Vendor" "digikey:490-1318-1-ND"
+			(at 0 228.6 0)
+			(effects
+				(font
+					(size 1.27 1.27)
+				)
+				(hide yes)
+			)
+		)
 		(pin "1"
 		)
@@
 			)
 		)
+		(property "Vendor" "digikey:490-1318-1-ND"
+			(at 0 190.5 0)
+			(effects
+				(font
+					(size 1.27 1.27)
+				)
+				(hide yes)
+			)
+		)
 		(pin "1"
 		)
@@
 			)
 		)
+		(property "Vendor" "digikey:311-4.75KHRCT-ND"
+			(at 62.23 -62.23 0)
+			(effects
+				(font
+					(size 1.27 1.27)
+				)
+				(hide yes)
+			)
+		)
 		(pin "1"
 		)
@@
 			)
 		)
+		(property "Vendor" "digikey:490-1318-1-ND"
+			(at 601.98 0 0)
+			(effects
+				(font
+					(size 1.27 1.27)
+				)
+				(hide yes)
+			)
+		)
 		(pin "1"
 		)
@@
 			)
 		)
+		(property "Vendor" "digikey:490-1318-1-ND"
+			(at 0 304.8 0)
+			(effects
+				(font
+					(size 1.27 1.27)
+				)
+				(hide yes)
+			)
+		)
 		(pin "1"
 		)
@@
 			)
 		)
+		(property "Vendor" "digikey:311-4.75KHRCT-ND"
+			(at 116.84 116.84 0)
+			(effects
+				(font
+					(size 1.27 1.27)
+				)
+				(hide yes)
+			)
+		)
 		(pin "2"
 		)
@@
 			)
 		)
+		(property "Vendor" "digikey:296-18593-1-ND"
+			(at 0 111.76 0)
+			(effects
+				(font
+					(size 1.27 1.27)
+				)
+				(hide yes)
+			)
+		)
 		(pin "2"
 		)
@@
 			)
 		)
+		(property "Vendor" "digikey:311-4.75KHRCT-ND"
+			(at 118.11 -118.11 0)
+			(effects
+				(font
+					(size 1.27 1.27)
+				)
+				(hide yes)
+			)
+		)
 		(pin "1"
 		)
@@
 			)
 		)
+		(property "Vendor" "digikey:490-1318-1-ND"
+			(at 109.22 0 0)
+			(effects
+				(font
+					(size 1.27 1.27)
+				)
+				(hide yes)
+			)
+		)
 		(pin "1"
 		)
@@
 			)
 		)
+		(property "Vendor" "digikey:490-1318-1-ND"
+			(at 599.44 0 0)
+			(effects
+				(font
+					(size 1.27 1.27)
+				)
+				(hide yes)
+			)
+		)
 		(pin "1"
 		)
@@
 			)
 		)
+		(property "Vendor" "digikey:311-4.75KHRCT-ND"
+			(at 276.86 276.86 0)
+			(effects
+				(font
+					(size 1.27 1.27)
+				)
+				(hide yes)
+			)
+		)
 		(pin "2"
 		)
@@
 			)
 		)
+		(property "Vendor" "digikey:296-18056-1-ND"
+			(at 0 335.28 0)
+			(effects
+				(font
+					(size 1.27 1.27)
+				)
+				(hide yes)
+			)
+		)
 		(pin "9"
 		)
@@
 			)
 		)
+		(property "Vendor" "digikey:296-18593-1-ND"
+			(at 0 421.64 0)
+			(effects
+				(font
+					(size 1.27 1.27)
+				)
+				(hide yes)
+			)
+		)
 		(pin "2"
 		)
@@
 			)
 		)
+		(property "Vendor" "digikey:296-18593-1-ND"
+			(at 0 259.08 0)
+			(effects
+				(font
+					(size 1.27 1.27)
+				)
+				(hide yes)
+			)
+		)
 		(pin "2"
 		)
@@
 			(effects
 				(font
+					(size 1.27 1.27)
+				)
+				(hide yes)
+			)
+		)
+		(property "Vendor" "digikey:490-1318-1-ND"
+			(at 0 391.16 0)
+			(effects
+				(font

Commit message: update value
Parts:
- C1701, C1702, C1703, C1704, C1705, C1706, C1707, C1708, C1709, C1710: value C -> 0.1UF
- R1701, R1702, R1703, R1704, R1705, R1706: value R -> 4.75K
Changed lines of the file:
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@@
 			)
 		)
-		(property "Value" "R"
+		(property "Value" "4.75K"
 			(at 234.95 166.37 90)
 			(effects
@@
 			)
 		)
-		(property "Value" "C"
+		(property "Value" "0.1UF"
 			(at 128.27 41.9099 0)
 			(effects
@@
 			)
 		)
-		(property "Value" "R"
+		(property "Value" "4.75K"
 			(at 60.96 128.27 90)
 			(effects
@@
 			)
 		)
-		(property "Value" "C"
+		(property "Value" "0.1UF"
 			(at 55.88 115.5699 0)
 			(effects
@@
 			)
 		)
-		(property "Value" "C"
+		(property "Value" "0.1UF"
 			(at 53.34 41.9099 0)
 			(effects
@@
 			)
 		)
-		(property "Value" "C"
+		(property "Value" "0.1UF"
 			(at 130.81 115.5699 0)
 			(effects
@@
 			)
 		)
-		(property "Value" "C"
+		(property "Value" "0.1UF"
 			(at 228.6 96.5199 0)
 			(effects
@@
 			)
 		)
-		(property "Value" "R"
+		(property "Value" "4.75K"
 			(at 234.95 168.91 90)
 			(effects
@@
 			)
 		)
-		(property "Value" "C"
+		(property "Value" "0.1UF"
 			(at 304.8 153.6699 0)
 			(effects
@@
 			)
 		)
-		(property "Value" "C"
+		(property "Value" "0.1UF"
 			(at 229.87 153.6699 0)
 			(effects
@@
 			)
 		)
-		(property "Value" "R"
+		(property "Value" "4.75K"
 			(at 58.42 54.61 90)
 			(effects
@@
 			)
 		)
-		(property "Value" "R"
+		(property "Value" "4.75K"
 			(at 233.68 111.76 90)
 			(effects
@@
 			)
 		)
-		(property "Value" "C"
+		(property "Value" "0.1UF"
 			(at 58.42 196.8499 0)
 			(effects
@@
 			)
 		)
-		(property "Value" "C"
+		(property "Value" "0.1UF"
 			(at 303.53 96.5199 0)
 			(effects
@@
 			)
 		)
-		(property "Value" "R"
+		(property "Value" "4.75K"
 			(at 63.5 209.55 90)
 			(effects
@@
 			)
 		)
-		(property "Value" "C"
+		(property "Value" "0.1UF"
 			(at 133.35 196.8499 0)
 			(effects

Commit message: lots small updates
Parts:
- TP10, TP14, TP15, TP16, TP20, TP21, TP23, TP24, TP25, TP26, TP27, TP3, TP4, TP7, TP8, TP9: now left out of the parts list
Changed lines of the file:
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@@
 		(unit 1)
 		(exclude_from_sim no)
-		(in_bom yes)
+		(in_bom no)
 		(on_board yes)
 		(dnp no)
@@
 		(unit 1)
 		(exclude_from_sim no)
-		(in_bom yes)
+		(in_bom no)
 		(on_board yes)
 		(dnp no)
@@
 		(unit 1)
 		(exclude_from_sim no)
-		(in_bom yes)
+		(in_bom no)
 		(on_board yes)
 		(dnp no)
@@
 		(unit 1)
 		(exclude_from_sim no)
-		(in_bom yes)
+		(in_bom no)
 		(on_board yes)
 		(dnp no)
@@
 		(unit 1)
 		(exclude_from_sim no)
-		(in_bom yes)
+		(in_bom no)
 		(on_board yes)
 		(dnp no)
@@
 		(unit 1)
 		(exclude_from_sim no)
-		(in_bom yes)
+		(in_bom no)
 		(on_board yes)
 		(dnp no)
@@
 		(unit 1)
 		(exclude_from_sim no)
-		(in_bom yes)
+		(in_bom no)
 		(on_board yes)
 		(dnp no)
@@
 		(unit 1)
 		(exclude_from_sim no)
-		(in_bom yes)
+		(in_bom no)
 		(on_board yes)
 		(dnp no)
@@
 		(unit 1)
 		(exclude_from_sim no)
-		(in_bom yes)
+		(in_bom no)
 		(on_board yes)
 		(dnp no)
@@
 		(unit 1)
 		(exclude_from_sim no)
-		(in_bom yes)
+		(in_bom no)
 		(on_board yes)
 		(dnp no)
@@
 		(unit 1)
 		(exclude_from_sim no)
-		(in_bom yes)
+		(in_bom no)
 		(on_board yes)
 		(dnp no)
@@
 		(unit 1)
 		(exclude_from_sim no)
-		(in_bom yes)
+		(in_bom no)
 		(on_board yes)
 		(dnp no)
@@
 		(unit 1)
 		(exclude_from_sim no)
-		(in_bom yes)
+		(in_bom no)
 		(on_board yes)
 		(dnp no)
@@
 		(unit 1)
 		(exclude_from_sim no)
-		(in_bom yes)
+		(in_bom no)
 		(on_board yes)
 		(dnp no)
@@
 		(unit 1)
 		(exclude_from_sim no)
-		(in_bom yes)
+		(in_bom no)
 		(on_board yes)
 		(dnp no)
@@
 		(unit 1)
 		(exclude_from_sim no)
-		(in_bom yes)
+		(in_bom no)
 		(on_board yes)
 		(dnp no)

Commit message: direction
Connections:
- net GND: now also C1702.1; no longer C1702.2
- net P2_VADJ: now also C1702.2; no longer C1702.1
Other:
- moved on the sheet: C1702
Changed lines of the file:
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@@
 	)
 	(junction
-		(at 153.67 142.24)
+		(at 52.07 110.49)
 		(diameter 0)
 		(color 0 0 0 0)
 	)
 	(junction
-		(at 299.72 170.18)
+		(at 153.67 142.24)
 		(diameter 0)
 		(color 0 0 0 0)
 	)
 	(junction
-		(at 59.69 191.77)
+		(at 299.72 170.18)
 		(diameter 0)
 		(color 0 0 0 0)
 	)
 	(junction
-		(at 52.07 110.49)
+		(at 59.69 191.77)
 		(diameter 0)
 		(color 0 0 0 0)
@@
 	(wire
 		(pts
+			(xy 52.07 110.49) (xy 57.15 110.49)
+		)
+		(stroke
+			(width 0)
+			(type default)
+		)
+	)
+	(wire
+		(pts
 			(xy 128.27 215.9) (xy 172.72 215.9)
 		)
@@
 	(wire
 		(pts
-			(xy 52.07 110.49) (xy 57.15 110.49)
-		)
-		(stroke
-			(width 0)
-			(type default)
-		)
-	)
-	(wire
-		(pts
 			(xy 41.91 134.62) (xy 64.77 134.62)
 		)
@@
 	(symbol
 		(lib_id "Device:C")
-		(at 52.07 114.3 0)
+		(at 52.07 114.3 180)
 		(unit 1)
 		(exclude_from_sim no)
@@
 					(size 1.27 1.27)
 				)
-				(justify left)
+				(justify right)
 			)
 		)
@@
 					(size 1.27 1.27)
 				)
-				(justify left)
+				(justify right)
 			)
 		)
 		(property "Footprint" "Capacitor_SMD:C_0402_1005Metric"
-			(at 53.0352 118.11 0)
+			(at 51.1048 110.49 0)
 			(effects
 				(font
@@
 		)
 		(property "Vendor" "digikey:490-1318-1-ND"
-			(at 0 228.6 0)
+			(at 104.14 0 0)
 			(effects
 				(font
