File: zest.kicad_pcb (KiCad board)
At the start: 8 copper layers, 110 x 181.8 mm, 443 parts, among them J1001 142-0701-201, J1002 U.FL-R-SMT(10), J1003 U.FL-R-SMT(10), J1004 142-0701-201, J1005 U.FL-R-SMT(10), J1201 142-0701-201, J1202 142-0701-201, J1401 ASP-134604-01, J1402 ASP-134604-01, J1501 10029449-111RLF, J1502 PPPC072LJBN-RC, J1503 PPPC072LJBN-RC, J1901 961102-6404-AR, J201 142-0701-201, J202 142-0701-201, J203 142-0701-201, J204 142-0701-201, J701 142-0701-201, J702 142-0701-201, J703 142-0701-201, J704 142-0701-201, J801 20021121-00020C4LF, J802 20021121-00020C4LF, J901 U.FL-R-SMT(10), J902 U.FL-R-SMT(10), J903 U.FL-R-SMT(10), J904 U.FL-R-SMT(10), J905 U.FL-R-SMT(10), J906 U.FL-R-SMT(10), Q1501 FDN335N, Q1502 FDN335N, T1001 TCM2-43X+, T1002 TCM2-43X+, U1001 TCP-2-33W+, U1002 LMK01801BISQE/NOPB, U1101 AD7794BRUZ, U1201 AD9781BCPZ, U1301 AMC7823IRTAT, U1601 LT6233CS6#TRMPBF, U1701 SN74LVC8T245PWR, U1702 SN74LVC8T245PWR, U1703 SN74LVC8T245PWR, U1704 SN74AVC4T245PWR, U1705 SN74AVC4T245PWR, U1801 ADL5501AKSZ-R7, U1901 AT24C64D-SSHM-T, U2001 KX023-1025-FR, U201 AD9653BCPZ-125, U2701 TPS62110RSAR, U2801 LTC6655CHLS8-2.5#PBF, U2901 TPS62110RSAR, U3001 LT6233CS6#TRMPBF, U3002 PBSS4230T,215, U3101 LT1763IDE-3.3#PBF, U3201 LT1763IDE-1.8#PBF, U701 AD9653BCPZ-125, U901 BAT54W-7-F, U902 ZXCT1009QFTA, U903 LT6233CS6#TRMPBF

Commit message: Schematic Changes
Added Manufacturer/MPN/Description Fields to parts
Added libraries to project
Modified FMC schematic to use new symbol
Parts:
- R1001: value 475 -> 475R
- R1002, R202, R702: value 100 -> 100R
- R1003, R1004, R1005, R1006, R1007, R1008, R1009, R1010, R1505, R1506, R2103, R2104, R2203, R2204, R2303, R2304, R2403, R2404, R2501, R2601, R3003, R303, R304, R403, R404, R503, R504, R603, R604: value 200 -> 200R
- R1101, R1102, R1501, R1502, R1503, R1504, R1605, R1901, R1902, R2101, R2102, R2201, R2202, R2301, R2302, R2401, R2402, R301, R302, R401, R402, R501, R502, R601, R602, R901, R902, R903: value 0 -> 0R
- R1201, R1202: value 49.9 -> 49.9R
- R1204: value 287 -> 287R
- R1801: value 221 -> 221R
- R2105, R2106, R2205, R2206, R2305, R2306, R2405, R2406, R305, R306, R405, R406, R505, R506, R605, R606: value 4.99 -> 4.99R
- R806, R913, R914: value 150 -> 150R
- R905: value 0.1 -> 0.1R
