File: zest.kicad_pcb (KiCad board)
At the start: 8 copper layers, 110 x 181.8 mm, 443 parts, among them J1001 142-0701-201, J1002 U.FL-R-SMT(10), J1003 U.FL-R-SMT(10), J1004 142-0701-201, J1005 U.FL-R-SMT(10), J1201 142-0701-201, J1202 142-0701-201, J1401 ASP-134604-01, J1402 ASP-134604-01, J1501 10029449-111RLF, J1502 PPPC072LJBN-RC, J1503 PPPC072LJBN-RC, J1901 961102-6404-AR, J201 142-0701-201, J202 142-0701-201, J203 142-0701-201, J204 142-0701-201, J701 142-0701-201, J702 142-0701-201, J703 142-0701-201, J704 142-0701-201, J801 20021121-00020C4LF, J802 20021121-00020C4LF, J901 U.FL-R-SMT(10), J902 U.FL-R-SMT(10), J903 U.FL-R-SMT(10), J904 U.FL-R-SMT(10), J905 U.FL-R-SMT(10), J906 U.FL-R-SMT(10), Q1501 FDN335N, Q1502 FDN335N, T1001 TCM2-43X+, T1002 TCM2-43X+, U1001 TCP-2-33W+, U1002 LMK01801BISQE/NOPB, U1101 AD7794BRUZ, U1201 AD9781BCPZ, U1301 AMC7823IRTAT, U1601 LT6233CS6#TRMPBF, U1701 SN74LVC8T245PWR, U1702 SN74LVC8T245PWR, U1703 SN74LVC8T245PWR, U1704 SN74AVC4T245PWR, U1705 SN74AVC4T245PWR, U1801 ADL5501AKSZ-R7, U1901 AT24C64D-SSHM-T, U2001 KX023-1025-FR, U201 AD9653BCPZ-125, U2701 TPS62110RSAR, U2801 LTC6655CHLS8-2.5#PBF, U2901 TPS62110RSAR, U3001 LT6233CS6#TRMPBF, U3002 PBSS4230T,215, U3101 LT1763IDE-3.3#PBF, U3201 LT1763IDE-1.8#PBF, U701 AD9653BCPZ-125, U901 BAT54W-7-F, U902 ZXCT1009QFTA, U903 LT6233CS6#TRMPBF

Commit message: Updated some Schematics
- updated slowmon schematic
- updated diff to se schematic
- cleaned up DRC/ERC errors
No changes were made that effected the PCB layout
Parts:
- D1501, D1502, D801, D901, D902, D903: value APT1608CGCK -> Green LED
- J801, J802: value 20021121-00020C4LF -> 20pin 50mil Header
- L2501, L2601: value MLF1608D47NMTA00 -> 47nH
Changed lines of the file:
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@@
 	(net 105 "/ad9781/diff2se_0/DIFF-")
 	(net 106 "Net-(C2502-Pad2)")
-	(net 107 "Net-(XMER2501-PRIMARY_DOT)")
+	(net 107 "Net-(C2503-Pad2)")
 	(net 108 "/ad9781/diff2se_0/SE+")
-	(net 109 "Net-(XMER2501-PRIMARY)")
+	(net 109 "Net-(C2504-Pad2)")
 	(net 110 "/ad9781/diff2se_1/DIFF+")
 	(net 111 "/ad9781/diff2se_1/DIFF-")
 	(net 112 "Net-(C2602-Pad2)")
-	(net 113 "Net-(XMER2601-PRIMARY_DOT)")
-	(net 114 "Net-(XMER2601-PRIMARY)")
+	(net 113 "Net-(C2603-Pad2)")
+	(net 114 "Net-(C2604-Pad2)")
 	(net 115 "/ad9781/diff2se_1/SE-")
 	(net 116 "Net-(U2701-VINA)")
@@
 	(net 512 "unconnected-(XMER2301-NC-Pad5)")
 	(net 513 "unconnected-(XMER2401-NC-Pad5)")
-	(net 514 "unconnected-(XMER2501-NOT_USED-Pad5)")
-	(net 515 "unconnected-(XMER2601-NOT_USED-Pad5)")
+	(net 514 "unconnected-(XMER2501-NC-Pad5)")
+	(net 515 "unconnected-(XMER2601-NC-Pad5)")
 	(net 516 "/ADC0/ADC01_SDIO")
 	(net 517 "/ADC0/ADC01_PDWN")
@@
 			)
 		)
-		(property "Value" "APT1608CGCK"
+		(property "Value" "Green LED"
 			(at 0 1.43 90)
 			(layer "F.Fab")
@@
 			(layers "F.Cu" "F.Paste" "F.Mask")
 			(roundrect_rratio 0.25)
-			(net 107 "Net-(XMER2501-PRIMARY_DOT)")
+			(net 107 "Net-(C2503-Pad2)")
 			(pintype "passive")
 		)
@@
 			)
 		)
-		(property "Value" "APT1608CGCK"
+		(property "Value" "Green LED"
 			(at 0 1.43 180)
 			(layer "F.Fab")
@@
 			)
 		)
-		(property "Value" "MLF1608D47NMTA00"
+		(property "Value" "47nH"
 			(at 0 1.43 180)
 			(layer "F.Fab")
@@
 			)
 		)
-		(property ki_fp_filters "DB714_MNC")
 		(sheetname "diff2se_0")
 		(sheetfile "diff_se.kicad_sch")
@@
 			(layers "F.Cu" "F.Paste" "F.Mask")
 			(net 105 "/ad9781/diff2se_0/DIFF-")
-			(pinfunction "SECONDARY")
 			(pintype "unspecified")
 		)
@@
 			(layers "F.Cu" "F.Paste" "F.Mask")
 			(net 1 "GND")
-			(pinfunction "SECONDARY_CT")
 			(pintype "unspecified")
 		)
@@
 			(layers "F.Cu" "F.Paste" "F.Mask")
 			(net 104 "/ad9781/diff2se_0/DIFF+")
-			(pinfunction "SECONDARY_DOT")
 			(pintype "unspecified")
 		)
@@
 			(size 1.4478 0.6604)
 			(layers "F.Cu" "F.Paste" "F.Mask")
-			(net 109 "Net-(XMER2501-PRIMARY)")
-			(pinfunction "PRIMARY")
+			(net 109 "Net-(C2504-Pad2)")
 			(pintype "unspecified")
 		)
@@
 			(size 1.4478 0.6604)
 			(layers "F.Cu" "F.Paste" "F.Mask")
-			(net 514 "unconnected-(XMER2501-NOT_USED-Pad5)")
-			(pinfunction "NOT_USED")
-			(pintype "unspecified+no_connect")
+			(net 514 "unconnected-(XMER2501-NC-Pad5)")
+			(pinfunction "NC")
+			(pintype "no_connect")
 		)
 		(pad "6" smd rect
@@
 			(size 1.4478 0.6604)
 			(layers "F.Cu" "F.Paste" "F.Mask")
-			(net 107 "Net-(XMER2501-PRIMARY_DOT)")
-			(pinfunction "PRIMARY_DOT")
+			(net 107 "Net-(C2503-Pad2)")
 			(pintype "unspecified")
 		)
@@
 			)
 		)
-		(property "Value" "20021121-00020C4LF"
+		(property "Value" "20pin 50mil Header"
 			(at 7.573618 7.094366 -90)
 			(layer "F.Fab")
@@
 			)
 		)
-		(property "Value" "APT1608CGCK"
+		(property "Value" "Green LED"
 			(at 0 1.43 0)
 			(layer "F.Fab")
@@
 			)
 		)
-		(property "Value" "APT1608CGCK"
+		(property "Value" "Green LED"
 			(at 0 1.43 180)
 			(layer "F.Fab")
@@
 			(layers "F.Cu" "F.Paste" "F.Mask")
 			(roundrect_rratio 0.25)
-			(net 113 "Net-(XMER2601-PRIMARY_DOT)")
+			(net 113 "Net-(C2603-Pad2)")
 			(pintype "passive")
 		)
@@
 			)
 		)
-		(property ki_fp_filters "DB714_MNC")
 		(sheetname "diff2se_1")
 		(sheetfile "diff_se.kicad_sch")
@@
 			(layers "F.Cu" "F.Paste" "F.Mask")
 			(net 111 "/ad9781/diff2se_1/DIFF-")
-			(pinfunction "SECONDARY")
 			(pintype "unspecified")
 		)
@@
 			(layers "F.Cu" "F.Paste" "F.Mask")
 			(net 1 "GND")
-			(pinfunction "SECONDARY_CT")
 			(pintype "unspecified")
 		)
@@
 			(layers "F.Cu" "F.Paste" "F.Mask")
 			(net 110 "/ad9781/diff2se_1/DIFF+")
-			(pinfunction "SECONDARY_DOT")
 			(pintype "unspecified")
 		)
@@
 			(size 1.4478 0.6604)
 			(layers "F.Cu" "F.Paste" "F.Mask")
-			(net 114 "Net-(XMER2601-PRIMARY)")
-			(pinfunction "PRIMARY")
+			(net 114 "Net-(C2604-Pad2)")
 			(pintype "unspecified")
 		)
@@
 			(size 1.4478 0.6604)
 			(layers "F.Cu" "F.Paste" "F.Mask")
-			(net 515 "unconnected-(XMER2601-NOT_USED-Pad5)")
-			(pinfunction "NOT_USED")
-			(pintype "unspecified+no_connect")
+			(net 515 "unconnected-(XMER2601-NC-Pad5)")
+			(pinfunction "NC")
+			(pintype "no_connect")
 		)
 		(pad "6" smd rect
@@
 			(size 1.4478 0.6604)
 			(layers "F.Cu" "F.Paste" "F.Mask")
-			(net 113 "Net-(XMER2601-PRIMARY_DOT)")
-			(pinfunction "PRIMARY_DOT")
+			(net 113 "Net-(C2603-Pad2)")
 			(pintype "unspecified")
 		)
@@
 			(layers "F.Cu" "F.Paste" "F.Mask")
 			(roundrect_rratio 0.25)
-			(net 114 "Net-(XMER2601-PRIMARY)")
+			(net 114 "Net-(C2604-Pad2)")
 			(pintype "passive")
 		)
@@
 			)
 		)
-		(property "Value" "APT1608CGCK"
+		(property "Value" "Green LED"
 			(at 0 1.43 90)
 			(layer "F.Fab")
@@
 			(layers "F.Cu" "F.Paste" "F.Mask")
 			(roundrect_rratio 0.25)
-			(net 109 "Net-(XMER2501-PRIMARY)")
+			(net 109 "Net-(C2504-Pad2)")
 			(pintype "passive")
 		)
@@
 			)
 		)
-		(property "Value" "20021121-00020C4LF"
+		(property "Value" "20pin 50mil Header"
 			(at 7.573618 7.094366 -90)
 			(layer "F.Fab")
@@
 			)
 		)
-		(property "Value" "APT1608CGCK"
+		(property "Value" "Green LED"
 			(at 0 1.43 -90)
 			(layer "F.Fab")
@@
 			)
 		)
-		(property ki_fp_filters "TO-???* *_Diode_* *SingleDiode* D_*")
+		(property ki_fp_filters "LED* LED_SMD:* LED_THT:*")
 		(sheetname "slowmon")
 		(sheetfile "slowmon.kicad_sch")
@@
 			)
 		)
-		(property "Value" "MLF1608D47NMTA00"
+		(property "Value" "47nH"
 			(at 0 1.43 180)
 			(layer "F.Fab")
